File: electrical/master_board/rev_a/nucleo_144.sch (KiCad schematic (older format))
At the start: 0 parts

Commit message: Starting to check in electrical directory.
Parts:
- added U? (x10): F767ZI;NUCLEO144, symbol F767ZI_NUCLEO144:F767ZI;NUCLEO144
Changed lines of the file:
@@
 $Descr A4 11693 8268
 encoding utf-8
-Sheet 1 9
+Sheet 3 9
 Title ""
 Date ""
@@
 Comment4 ""
 $EndDescr
+$Comp
+L F767ZI_NUCLEO144:F767ZI;NUCLEO144 U?
+U 1 1 5E75C3F5
+P 1500 1350
+F 0 "U?" H 2306 1640 60  0000 C CNN
+F 1 "F767ZI;NUCLEO144" H 2306 1534 60  0000 C CNN
+F 2 "" H 1500 1350 50  0001 C CNN
+F 3 "" H 1500 1350 50  0001 C CNN
+	1    1500 1350
+	1    0    0    -1
+$EndComp
+$Comp
+L F767ZI_NUCLEO144:F767ZI;NUCLEO144 U?
+U 2 1 5E761191
+P 1600 3400
+F 0 "U?" H 2506 3690 60  0000 C CNN
+F 1 "F767ZI;NUCLEO144" H 2506 3584 60  0000 C CNN
+F 2 "" H 1600 3400 50  0001 C CNN
+F 3 "" H 1600 3400 50  0001 C CNN
+	2    1600 3400
+	1    0    0    -1
+$EndComp
+$Comp
+L F767ZI_NUCLEO144:F767ZI;NUCLEO144 U?
+U 3 1 5E7669F5
+P 1550 5550
+F 0 "U?" H 2556 5840 60  0000 C CNN
+F 1 "F767ZI;NUCLEO144" H 2556 5734 60  0000 C CNN
+F 2 "" H 1550 5550 50  0001 C CNN
+F 3 "" H 1550 5550 50  0001 C CNN
+	3    1550 5550
+	1    0    0    -1
+$EndComp
+$Comp
+L F767ZI_NUCLEO144:F767ZI;NUCLEO144 U?
+U 4 1 5E76D4F3
+P 3450 1200
+F 0 "U?" H 4156 1490 60  0000 C CNN
+F 1 "F767ZI;NUCLEO144" H 4156 1384 60  0000 C CNN
+F 2 "" H 3450 1200 50  0001 C CNN
+F 3 "" H 3450 1200 50  0001 C CNN
+	4    3450 1200
+	1    0    0    -1
+$EndComp
+$Comp
+L F767ZI_NUCLEO144:F767ZI;NUCLEO144 U?
+U 5 1 5E771671
+P 3700 3350
+F 0 "U?" H 4406 3640 60  0000 C CNN
+F 1 "F767ZI;NUCLEO144" H 4406 3534 60  0000 C CNN
+F 2 "" H 3700 3350 50  0001 C CNN
+F 3 "" H 3700 3350 50  0001 C CNN
+	5    3700 3350
+	1    0    0    -1
+$EndComp
+$Comp
+L F767ZI_NUCLEO144:F767ZI;NUCLEO144 U?
+U 6 1 5E7752BB
+P 3800 5550
+F 0 "U?" H 4556 5840 60  0000 C CNN
+F 1 "F767ZI;NUCLEO144" H 4556 5734 60  0000 C CNN
+F 2 "" H 3800 5550 50  0001 C CNN
+F 3 "" H 3800 5550 50  0001 C CNN
+	6    3800 5550
+	1    0    0    -1
+$EndComp
+$Comp
+L F767ZI_NUCLEO144:F767ZI;NUCLEO144 U?
+U 7 1 5E7773F6
+P 5300 1150
+F 0 "U?" H 6206 1440 60  0000 C CNN
+F 1 "F767ZI;NUCLEO144" H 6206 1334 60  0000 C CNN
+F 2 "" H 5300 1150 50  0001 C CNN
+F 3 "" H 5300 1150 50  0001 C CNN
+	7    5300 1150
+	1    0    0    -1
+$EndComp
+$Comp
+L F767ZI_NUCLEO144:F767ZI;NUCLEO144 U?
+U 8 1 5E77BCA3
+P 5350 3450
+F 0 "U?" H 6256 3740 60  0000 C CNN
+F 1 "F767ZI;NUCLEO144" H 6256 3634 60  0000 C CNN
+F 2 "" H 5350 3450 50  0001 C CNN
+F 3 "" H 5350 3450 50  0001 C CNN
+	8    5350 3450
+	1    0    0    -1
+$EndComp
+$Comp
+L F767ZI_NUCLEO144:F767ZI;NUCLEO144 U?
+U 9 1 5E77F676
+P 5300 4050
+F 0 "U?" H 5806 4340 60  0000 C CNN
+F 1 "F767ZI;NUCLEO144" H 5806 4234 60  0000 C CNN
+F 2 "" H 5300 4050 50  0001 C CNN
+F 3 "" H 5300 4050 50  0001 C CNN
+	9    5300 4050
+	1    0    0    -1
+$EndComp
+$Comp
+L F767ZI_NUCLEO144:F767ZI;NUCLEO144 U?
+U 10 1 5E782D7F
+P 5350 5100
+F 0 "U?" H 6100 5390 60  0000 C CNN
+F 1 "F767ZI;NUCLEO144" H 6100 5284 60  0000 C CNN
+F 2 "" H 5350 5100 50  0001 C CNN
+F 3 "" H 5350 5100 50  0001 C CNN
+	10   5350 5100
+	1    0    0    -1
+$EndComp
 $EndSCHEMATC
