File: electrical/master_board/rev_a/nucleo_144.sch (KiCad schematic (older format))
At the start: 10 parts

Commit message: Updated nucleo_144.sch to use the correct symbol for the F767ZI;NUCLEO144 .
Parts:
- removed U? (x10): F767ZI;NUCLEO144, symbol F767ZI_NUCLEO144:F767ZI;NUCLEO144
- added CN? (x10): F767ZI;NUCLEO144, NUCLEO144, symbol master_board:F767ZI;NUCLEO144
Changed lines of the file:
@@
 $EndDescr
 $Comp
-L F767ZI_NUCLEO144:F767ZI;NUCLEO144 U?
-U 1 1 5E75C3F5
-P 1500 1350
-F 0 "U?" H 2306 1640 60  0000 C CNN
-F 1 "F767ZI;NUCLEO144" H 2306 1534 60  0000 C CNN
-F 2 "" H 1500 1350 50  0001 C CNN
-F 3 "" H 1500 1350 50  0001 C CNN
-	1    1500 1350
+L master_board:F767ZI;NUCLEO144 CN?
+U 1 1 5EA6C86E
+P 950 1050
+F 0 "CN?" H 1756 1340 60  0000 C CNN
+F 1 "F767ZI;NUCLEO144" H 1756 1234 60  0000 C CNN
+F 2 "NUCLEO144" H 1150 1100 60  0001 L CNN
+F 3 "https://www.st.com/resource/en/user_manual/dm00244518-stm32-nucleo144-boards-stmicroelectronics.pdf" H 1150 900 60  0001 L CNN
+F 4 "https://www.st.com/resource/en/user_manual/dm00244518-stm32-nucleo144-boards-stmicroelectronics.pdf" H 1150 1000 60  0001 L CNN "manf#"
+F 5 "NUCLEO144-F767ZI;Nucleo144 STM32F767ZI" H 1150 800 60  0001 L CNN "Field5"
+	1    950  1050
 	1    0    0    -1
 $EndComp
 $Comp
-L F767ZI_NUCLEO144:F767ZI;NUCLEO144 U?
-U 2 1 5E761191
-P 1600 3400
-F 0 "U?" H 2506 3690 60  0000 C CNN
-F 1 "F767ZI;NUCLEO144" H 2506 3584 60  0000 C CNN
-F 2 "" H 1600 3400 50  0001 C CNN
-F 3 "" H 1600 3400 50  0001 C CNN
-	2    1600 3400
+L master_board:F767ZI;NUCLEO144 CN?
+U 2 1 5EA70BAD
+P 750 3050
+F 0 "CN?" H 1656 3340 60  0000 C CNN
+F 1 "F767ZI;NUCLEO144" H 1656 3234 60  0000 C CNN
+F 2 "NUCLEO144" H 950 3100 60  0001 L CNN
+F 3 "https://www.st.com/resource/en/user_manual/dm00244518-stm32-nucleo144-boards-stmicroelectronics.pdf" H 950 2900 60  0001 L CNN
+F 4 "https://www.st.com/resource/en/user_manual/dm00244518-stm32-nucleo144-boards-stmicroelectronics.pdf" H 950 3000 60  0001 L CNN "manf#"
+F 5 "NUCLEO144-F767ZI;Nucleo144 STM32F767ZI" H 950 2800 60  0001 L CNN "Field5"
+	2    750  3050
 	1    0    0    -1
 $EndComp
 $Comp
-L F767ZI_NUCLEO144:F767ZI;NUCLEO144 U?
-U 3 1 5E7669F5
-P 1550 5550
-F 0 "U?" H 2556 5840 60  0000 C CNN
-F 1 "F767ZI;NUCLEO144" H 2556 5734 60  0000 C CNN
-F 2 "" H 1550 5550 50  0001 C CNN
-F 3 "" H 1550 5550 50  0001 C CNN
-	3    1550 5550
+L master_board:F767ZI;NUCLEO144 CN?
+U 3 1 5EA7C999
+P 750 5050
+F 0 "CN?" H 1756 5340 60  0000 C CNN
+F 1 "F767ZI;NUCLEO144" H 1756 5234 60  0000 C CNN
+F 2 "NUCLEO144" H 950 5100 60  0001 L CNN
+F 3 "https://www.st.com/resource/en/user_manual/dm00244518-stm32-nucleo144-boards-stmicroelectronics.pdf" H 950 4900 60  0001 L CNN
+F 4 "https://www.st.com/resource/en/user_manual/dm00244518-stm32-nucleo144-boards-stmicroelectronics.pdf" H 950 5000 60  0001 L CNN "manf#"
+F 5 "NUCLEO144-F767ZI;Nucleo144 STM32F767ZI" H 950 4800 60  0001 L CNN "Field5"
+	3    750  5050
 	1    0    0    -1
 $EndComp
 $Comp
-L F767ZI_NUCLEO144:F767ZI;NUCLEO144 U?
-U 4 1 5E76D4F3
-P 3450 1200
-F 0 "U?" H 4156 1490 60  0000 C CNN
-F 1 "F767ZI;NUCLEO144" H 4156 1384 60  0000 C CNN
-F 2 "" H 3450 1200 50  0001 C CNN
-F 3 "" H 3450 1200 50  0001 C CNN
-	4    3450 1200
+L master_board:F767ZI;NUCLEO144 CN?
+U 4 1 5EA803E6
+P 3050 1050
+F 0 "CN?" H 3756 1340 60  0000 C CNN
+F 1 "F767ZI;NUCLEO144" H 3756 1234 60  0000 C CNN
+F 2 "NUCLEO144" H 3250 1100 60  0001 L CNN
+F 3 "https://www.st.com/resource/en/user_manual/dm00244518-stm32-nucleo144-boards-stmicroelectronics.pdf" H 3250 900 60  0001 L CNN
+F 4 "https://www.st.com/resource/en/user_manual/dm00244518-stm32-nucleo144-boards-stmicroelectronics.pdf" H 3250 1000 60  0001 L CNN "manf#"
+F 5 "NUCLEO144-F767ZI;Nucleo144 STM32F767ZI" H 3250 800 60  0001 L CNN "Field5"
+	4    3050 1050
 	1    0    0    -1
 $EndComp
 $Comp
-L F767ZI_NUCLEO144:F767ZI;NUCLEO144 U?
-U 5 1 5E771671
-P 3700 3350
-F 0 "U?" H 4406 3640 60  0000 C CNN
-F 1 "F767ZI;NUCLEO144" H 4406 3534 60  0000 C CNN
-F 2 "" H 3700 3350 50  0001 C CNN
-F 3 "" H 3700 3350 50  0001 C CNN
-	5    3700 3350
+L master_board:F767ZI;NUCLEO144 CN?
+U 5 1 5EA869E7
+P 3050 3100
+F 0 "CN?" H 3756 3390 60  0000 C CNN
+F 1 "F767ZI;NUCLEO144" H 3756 3284 60  0000 C CNN
+F 2 "NUCLEO144" H 3250 3150 60  0001 L CNN
+F 3 "https://www.st.com/resource/en/user_manual/dm00244518-stm32-nucleo144-boards-stmicroelectronics.pdf" H 3250 2950 60  0001 L CNN
+F 4 "https://www.st.com/resource/en/user_manual/dm00244518-stm32-nucleo144-boards-stmicroelectronics.pdf" H 3250 3050 60  0001 L CNN "manf#"
+F 5 "NUCLEO144-F767ZI;Nucleo144 STM32F767ZI" H 3250 2850 60  0001 L CNN "Field5"
+	5    3050 3100
 	1    0    0    -1
 $EndComp
 $Comp
-L F767ZI_NUCLEO144:F767ZI;NUCLEO144 U?
-U 6 1 5E7752BB
-P 3800 5550
-F 0 "U?" H 4556 5840 60  0000 C CNN
-F 1 "F767ZI;NUCLEO144" H 4556 5734 60  0000 C CNN
-F 2 "" H 3800 5550 50  0001 C CNN
-F 3 "" H 3800 5550 50  0001 C CNN
-	6    3800 5550
+L master_board:F767ZI;NUCLEO144 CN?
+U 6 1 5EA8B5AE
+P 3050 5150
+F 0 "CN?" H 3806 5440 60  0000 C CNN
+F 1 "F767ZI;NUCLEO144" H 3806 5334 60  0000 C CNN
+F 2 "NUCLEO144" H 3250 5200 60  0001 L CNN
+F 3 "https://www.st.com/resource/en/user_manual/dm00244518-stm32-nucleo144-boards-stmicroelectronics.pdf" H 3250 5000 60  0001 L CNN
+F 4 "https://www.st.com/resource/en/user_manual/dm00244518-stm32-nucleo144-boards-stmicroelectronics.pdf" H 3250 5100 60  0001 L CNN "manf#"
+F 5 "NUCLEO144-F767ZI;Nucleo144 STM32F767ZI" H 3250 4900 60  0001 L CNN "Field5"
+	6    3050 5150
 	1    0    0    -1
 $EndComp
 $Comp
-L F767ZI_NUCLEO144:F767ZI;NUCLEO144 U?
-U 7 1 5E7773F6
-P 5300 1150
-F 0 "U?" H 6206 1440 60  0000 C CNN
-F 1 "F767ZI;NUCLEO144" H 6206 1334 60  0000 C CNN
-F 2 "" H 5300 1150 50  0001 C CNN
-F 3 "" H 5300 1150 50  0001 C CNN
-	7    5300 1150
+L master_board:F767ZI;NUCLEO144 CN?
+U 7 1 5EA96891
+P 4800 1000
+F 0 "CN?" H 5706 1290 60  0000 C CNN
+F 1 "F767ZI;NUCLEO144" H 5706 1184 60  0000 C CNN
+F 2 "NUCLEO144" H 5000 1050 60  0001 L CNN
+F 3 "https://www.st.com/resource/en/user_manual/dm00244518-stm32-nucleo144-boards-stmicroelectronics.pdf" H 5000 850 60  0001 L CNN
+F 4 "https://www.st.com/resource/en/user_manual/dm00244518-stm32-nucleo144-boards-stmicroelectronics.pdf" H 5000 950 60  0001 L CNN "manf#"
+F 5 "NUCLEO144-F767ZI;Nucleo144 STM32F767ZI" H 5000 750 60  0001 L CNN "Field5"
+	7    4800 1000
 	1    0    0    -1
 $EndComp
 $Comp
-L F767ZI_NUCLEO144:F767ZI;NUCLEO144 U?
-U 8 1 5E77BCA3
-P 5350 3450
-F 0 "U?" H 6256 3740 60  0000 C CNN
-F 1 "F767ZI;NUCLEO144" H 6256 3634 60  0000 C CNN
-F 2 "" H 5350 3450 50  0001 C CNN
-F 3 "" H 5350 3450 50  0001 C CNN
-	8    5350 3450
+L master_board:F767ZI;NUCLEO144 CN?
+U 8 1 5EA99BA4
+P 4800 3100
+F 0 "CN?" H 5706 3390 60  0000 C CNN
+F 1 "F767ZI;NUCLEO144" H 5706 3284 60  0000 C CNN
+F 2 "NUCLEO144" H 5000 3150 60  0001 L CNN
+F 3 "https://www.st.com/resource/en/user_manual/dm00244518-stm32-nucleo144-boards-stmicroelectronics.pdf" H 5000 2950 60  0001 L CNN
+F 4 "https://www.st.com/resource/en/user_manual/dm00244518-stm32-nucleo144-boards-stmicroelectronics.pdf" H 5000 3050 60  0001 L CNN "manf#"
+F 5 "NUCLEO144-F767ZI;Nucleo144 STM32F767ZI" H 5000 2850 60  0001 L CNN "Field5"
+	8    4800 3100
 	1    0    0    -1
 $EndComp
 $Comp
-L F767ZI_NUCLEO144:F767ZI;NUCLEO144 U?
-U 9 1 5E77F676
-P 5300 4050
-F 0 "U?" H 5806 4340 60  0000 C CNN
-F 1 "F767ZI;NUCLEO144" H 5806 4234 60  0000 C CNN
-F 2 "" H 5300 4050 50  0001 C CNN
-F 3 "" H 5300 4050 50  0001 C CNN
-	9    5300 4050
+L master_board:F767ZI;NUCLEO144 CN?
+U 9 1 5EA9E01B
+P 4850 3700
+F 0 "CN?" H 5356 3990 60  0000 C CNN
+F 1 "F767ZI;NUCLEO144" H 5356 3884 60  0000 C CNN
+F 2 "NUCLEO144" H 5050 3750 60  0001 L CNN
+F 3 "https://www.st.com/resource/en/user_manual/dm00244518-stm32-nucleo144-boards-stmicroelectronics.pdf" H 5050 3550 60  0001 L CNN
+F 4 "https://www.st.com/resource/en/user_manual/dm00244518-stm32-nucleo144-boards-stmicroelectronics.pdf" H 5050 3650 60  0001 L CNN "manf#"
+F 5 "NUCLEO144-F767ZI;Nucleo144 STM32F767ZI" H 5050 3450 60  0001 L CNN "Field5"
+	9    4850 3700
 	1    0    0    -1
 $EndComp
 $Comp
-L F767ZI_NUCLEO144:F767ZI;NUCLEO144 U?
-U 10 1 5E782D7F
-P 5350 5100
-F 0 "U?" H 6100 5390 60  0000 C CNN
-F 1 "F767ZI;NUCLEO144" H 6100 5284 60  0000 C CNN
-F 2 "" H 5350 5100 50  0001 C CNN
-F 3 "" H 5350 5100 50  0001 C CNN
-	10   5350 5100
+L master_board:F767ZI;NUCLEO144 CN?
+U 10 1 5EAA521F
+P 4850 4750
+F 0 "CN?" H 5600 5040 60  0000 C CNN
+F 1 "F767ZI;NUCLEO144" H 5600 4934 60  0000 C CNN
+F 2 "NUCLEO144" H 5050 4800 60  0001 L CNN
+F 3 "https://www.st.com/resource/en/user_manual/dm00244518-stm32-nucleo144-boards-stmicroelectronics.pdf" H 5050 4600 60  0001 L CNN
+F 4 "https://www.st.com/resource/en/user_manual/dm00244518-stm32-nucleo144-boards-stmicroelectronics.pdf" H 5050 4700 60  0001 L CNN "manf#"
+F 5 "NUCLEO144-F767ZI;Nucleo144 STM32F767ZI" H 5050 4500 60  0001 L CNN "Field5"
+	10   4850 4750
 	1    0    0    -1
 $EndComp
