File: electrical/master_board/rev_a/master.kicad_pcb (KiCad board)
At the start: 2 copper layers, 0 parts

Commit message: Inject the PCB outlines into master/center/ne/nw/se/sw PCB's.
Other:
- board outline added: 144.3 x 156 mm
