File: electrical/master_board/rev_a/sonars_leds.sch (KiCad schematic (older format))
At the start: 35 parts, among them CN101 BRIDGE_NE_INNER;3xM1x1+M1x5, CN102 BRIDGE_NW_INNER;M1x2+M2x5, CN103 BRIDGE_SE_INNER;M1x8, CN104 BRIDGE_SW_INNER;M1x8, CN4 SERVO;M1x3, CN5 SERVO;M1x3, CN50 HCSR04;F1X4, CN51 HCSR04LP;F1X4, CN52 HCSR04LP;F1X4, CN53 HCSR04LP;F1X4, CN54 HCSR04LP;F1X4, CN6 SERVO;M1x3, CN7 SERVO;M1x3, U4 SN74HCS595;TTSOP16, U5 SN74HCS595;TTSOP16, U6 CD450B;TTSOP16, U7 CD450B;TTSOP16

Commit message: Reworked Sonars, Servers, and LED's schematics.
Parts:
- removed C13: 10pF;1608, symbol Device:C
- removed CN101: BRIDGE_NE_INNER;3xM1x1+M1x5, HR2:BRIDGE_NE_INNER_3xM1x1+M1x5, symbol HR2:BRIDGE_NE_INNER;3xM1x1+M1x5
- removed CN102: BRIDGE_NW_INNER;M1x2+M2x5, HR2:BRIDGE_NW_INNER_M1x2+M2x5, symbol HR2:BRIDGE_NW_INNER;M1x2+M2x5
- removed CN103: BRIDGE_SE_INNER;M1x8, HR2:BRIDGE_SE_INNER_M1x8, symbol HR2:BRIDGE_SE_INNER;M1x8
- removed CN104: BRIDGE_SW_INNER;M1x8, HR2:BRIDGE_SW_INNER_M1x8, symbol HR2:BRIDGE_SW_INNER;M1x8
- removed CN4, CN5, CN6, CN7: SERVO;M1x3, Connector_PinHeader_2.54mm:PinHeader_1x03_P2.54mm_Vertical, symbol HR2:SERVO;M1x3
- removed CN50: HCSR04;F1X4, HR2:HCSR04_F1x4, symbol HR2:HCSR04;F1X4
- removed R23, R24, R25, R26, R27, R33: 33KΩ;1608, symbol Device:R_US
- removed R28, R29, R30, R31, R32, R34: 22KΩ;1608, symbol Device:R_US
- removed U4, U5: SN74HCS595;TTSOP16, Package_SO:TSSOP-16_4.4x5mm_P0.65mm, symbol HR2:SN74HCS595;TTSOP16
- added CN4, CN5, CN6, CN7: SERVO;F1x3, Connector_PinHeader_2.54mm:PinHeader_1x03_P2.54mm_Vertical, symbol HR2:SERVO;F1x3
- added CN50, CN60, CN70: HCSR04LP;F1X4, HR2:HCSR04_F1x4LP, symbol HR2:HCSR04LP;F1X4
- added R48, R50, R52, R54, R56, R58: 22KΩ;1608, symbol Device:R_US
- added R49, R51, R53, R55, R57, R59: 33KΩ;1608, symbol Device:R_US
- added U9: SN74HCS595;TTSOP16, Package_SO:TSSOP-16_4.4x5mm_P0.65mm, symbol HR2:SN74HCS595;TTSOP16
Connections:
- net labels added: DIO_NSS, MISC_MOSI, MISC_SCK, P5V, SONAR_SER
- net labels removed: 9V, LED1, LED10, LED11, LED12, LED13, LED14, LED15, LED16, LED2, LED3, LED4, LED5, LED6, LED7, LED8, LED9, LED_MOSI, LED_NSS, LED_SCLK
- wire segments 232 -> 219
- no-connect marks 11 -> 4
Other:
- note added: "3.3V to 5V Level Shifter"
- note added: "8-Bit Serial to\nParallel Shift\nRegister."
- note added: "Note:\nQH is temp. No Connect."
- note added: "Notes:\n1. The Sonars are HC04's that operate off of 5V.\n2. The trigger signals are provided by a serial shift register.\n3. A level shifter is used to shift trigger signals from 3.3V to 5V.\n4. A resistor voltage divider is used to convert the echo from 5V to 3.3V.\n5. Most hobby servers operate off of approximately 5V - 6V.\n6. The 4.8V supply is a 5V supply that is used for servos and LED's.\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"
- note added: "Servos"
- note added: "Sonar Connectors"
- note removed: "16-Bit SPI LED Shift Register"
- note removed: "3.3V to 5V Level Shifters"
- note removed: "LED Bus"
- note removed: "NE Quadrant Connector"
- note removed: "NW Quadrant Connector"
- note removed: "Notes:\n1. The LED's are on seperate PCB's that fit the Bantam Tools\n PCB blank restriction of 4in x 5in. There are 4 of them,\n and they are imaginatively called NE, NW, SE, and SW and\n they are connected to by CN101, CN102, CN103, and CN104.\n2. The LED's are controlled by a 16-bit shift regester that is\n filled using an SPI controller. The 3.3V outputs are fed into\n FET's that drive the LE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"
- note removed: "SE Quadrant Connector"
- note removed: "SW Quadrant Connector"
- note removed: "Servo Bus"
- note removed: "Servo\nConnectors"
- note removed: "Sonar Bus"
- note removed: "Sonar\nBus"
- note removed: "TO DO:\n1. Add 2 buttons to both the SE and SW connectors."
- moved on the sheet: C10, C11, C12, CN51, R21, R22, U6, U7
