File: electrical/master_board/rev_a/sw.sch (KiCad schematic (older format))
At the start: 27 parts

Commit message: Reworked Sonars, Servers, and LED's schematics.
Parts:
- removed CN?: BRIDGE_SW_OUTER;M1x8, HR2:BRIDGE_SW_OUTER_M1x8, symbol HR2:BRIDGE_SW_OUTER;M1x8
- gave numbers to parts that had none: 26
Connections:
- wire segments 97 -> 95
- no-connect marks 1 -> 0
Changed lines of the file:
@@
 $Descr A 11000 8500
 encoding utf-8
-Sheet 11 12
-Title "HR2 SW PCB"
-Date "2020-06-13"
+Sheet 11 13
+Title "HR2 Master Board"
+Date "2020-10-03"
 Rev "A"
-Comp "Homebrew Robotics Club"
-Comment1 ""
-Comment2 ""
+Comp "HomeBrew Robotics Club"
+Comment1 "Copyright © 2020 by HomeBrew Robotics Club "
+Comment2 "MIT License"
 Comment3 ""
 Comment4 ""
 $EndDescr
 $Comp
-L HR2:HOLE;M2.5 H?
+L HR2:HOLE;M2.5 H4
 U 1 1 5F2F7A6B
 P 2650 4450
-F 0 "H?" H 2600 4500 50  0000 L CNN
+F 0 "H4" H 2600 4500 50  0000 L CNN
 F 1 "HOLE;M2.5" H 2450 4400 50  0000 L CNN
 F 2 "MountingHole:MountingHole_2.7mm_M2.5" H 2850 4500 60  0001 L CNN
@@
 $EndComp
 $Comp
-L Device:LED D?
+L Device:LED D11
 U 1 1 5F30CB7A
 P 5400 4150
-F 0 "D?" V 5500 4250 50  0000 R CNN
+F 0 "D11" V 5500 4250 50  0000 R CNN
 F 1 "LED;GRNRA" V 5300 4600 50  0000 R CNN
 F 2 "HR2:LED_GRNRA" H 5400 4150 50  0001 C CNN
@@
 $EndComp
 $Comp
-L Device:LED D?
+L Device:LED D13
 U 1 1 5F30CF92
 P 7200 4150
-F 0 "D?" V 7300 4300 50  0000 R CNN
+F 0 "D13" V 7300 4300 50  0000 R CNN
 F 1 "LED;GRNRA" V 7100 4600 50  0000 R CNN
 F 2 "HR2:LED_GRNRA" H 7200 4150 50  0001 C CNN
@@
 $EndComp
 $Comp
-L Device:LED D?
+L Device:LED D14
 U 1 1 5F30EB24
 P 8100 4150
-F 0 "D?" V 8200 4300 50  0000 R CNN
+F 0 "D14" V 8200 4300 50  0000 R CNN
 F 1 "LED;GRNRA" V 8000 4600 50  0000 R CNN
 F 2 "HR2:LED_GRNRA" H 8100 4150 50  0001 C CNN
@@
 	0    -1   -1   0
 $EndComp
-$Comp
-L HR2:BRIDGE_SW_OUTER;M1x8 CN?
-U 1 1 5F387C15
-P 2500 3000
-F 0 "CN?" H 2850 2150 50  0000 C CNN
-F 1 "BRIDGE_SW_OUTER;M1x8" H 2850 3150 50  0000 C CNN
-F 2 "HR2:BRIDGE_SW_OUTER_M1x8" H 2700 3050 60  0001 L CNN
-F 3 "" H 2700 2850 60  0001 L CNN
-F 4 "SW Outer Bridge Connector" H 2700 2750 60  0001 L CNN "Field5"
-	1    2500 3000
-	1    0    0    1
-$EndComp
-NoConn ~ 3300 2300
 Wire Wire Line
 	8100 4900 8100 4800
-Text Label 3750 4900 0    50   ~ 0
+Text Label 6000 4900 0    50   ~ 0
 GND
 $Comp
-L Transistor_FET:2N7000 Q?
+L Transistor_FET:2N7000 Q16
 U 1 1 5F39F103
 P 8000 4600
-F 0 "Q?" H 7850 4750 50  0000 L CNN
+F 0 "Q16" H 7850 4750 50  0000 L CNN
 F 1 "2N7000;SOT23" H 7400 4550 50  0000 L CNN
 F 2 "Package_TO_SOT_SMD:SOT-23" H 8200 4525 50  0001 L CIN
@@
 $EndComp
 $Comp
-L Device:R_US R?
+L Device:R_US R72
 U 1 1 5F3A3A4B
 P 7850 3500
-F 0 "R?" V 7750 3400 50  0000 L CNN
+F 0 "R72" V 7750 3400 50  0000 L CNN
 F 1 "330Ω;1608" V 7950 3300 50  0000 L CNN
 F 2 "Resistor_SMD:R_0603_1608Metric" V 7890 3490 50  0001 C CNN
@@
 	8100 4400 8100 4300
 $Comp
-L Device:R_US R?
+L Device:R_US R71
 U 1 1 5F3A820E
 P 7850 3200
-F 0 "R?" V 7750 3100 50  0000 L CNN
+F 0 "R71" V 7750 3100 50  0000 L CNN
 F 1 "330Ω;1608" V 7950 3000 50  0000 L CNN
 F 2 "Resistor_SMD:R_0603_1608Metric" V 7890 3190 50  0001 C CNN
@@
 $EndComp
 $Comp
-L Device:R_US R?
+L Device:R_US R73
 U 1 1 5F3A878F
 P 7850 3800
-F 0 "R?" V 7750 3700 50  0000 L CNN
+F 0 "R73" V 7750 3700 50  0000 L CNN
 F 1 "330Ω;1608" V 7950 3600 50  0000 L CNN
 F 2 "Resistor_SMD:R_0603_1608Metric" V 7890 3790 50  0001 C CNN
@@
 	7200 4900 7200 4800
 $Comp
-L Transistor_FET:2N7000 Q?
+L Transistor_FET:2N7000 Q15
 U 1 1 5F3B5AC4
 P 7100 4600
-F 0 "Q?" H 6950 4750 50  0000 L CNN
+F 0 "Q15" H 6950 4750 50  0000 L CNN
 F 1 "2N7000;SOT23" H 6500 4550 50  0000 L CNN
 F 2 "Package_TO_SOT_SMD:SOT-23" H 7300 4525 50  0001 L CIN
@@
 $EndComp
 $Comp
-L Device:R_US R?
+L Device:R_US R69
 U 1 1 5F3B5ACE
 P 6950 3500
-F 0 "R?" V 6850 3400 50  0000 L CNN
+F 0 "R69" V 6850 3400 50  0000 L CNN
 F 1 "330Ω;1608" V 7050 3300 50  0000 L CNN
 F 2 "Resistor_SMD:R_0603_1608Metric" V 6990 3490 50  0001 C CNN
@@
 	7200 4400 7200 4300
 $Comp
-L Device:R_US R?
+L Device:R_US R68
 U 1 1 5F3B5AD9
 P 6950 3200
-F 0 "R?" V 6850 3100 50  0000 L CNN
+F 0 "R68" V 6850 3100 50  0000 L CNN
 F 1 "330Ω;1608" V 7050 3000 50  0000 L CNN
 F 2 "Resistor_SMD:R_0603_1608Metric" V 6990 3190 50  0001 C CNN
@@
 $EndComp
 $Comp
-L Device:R_US R?
+L Device:R_US R70
 U 1 1 5F3B5AE3
 P 6950 3800
-F 0 "R?" V 6850 3700 50  0000 L CNN
+F 0 "R70" V 6850 3700 50  0000 L CNN
 F 1 "330Ω;1608" V 7050 3600 50  0000 L CNN
 F 2 "Resistor_SMD:R_0603_1608Metric" V 6990 3790 50  0001 C CNN
@@
 	5400 4900 5400 4800
 $Comp
-L Transistor_FET:2N7000 Q?
+L Transistor_FET:2N7000 Q13
 U 1 1 5F3B8D4A
 P 5300 4600
-F 0 "Q?" H 5150 4750 50  0000 L CNN
+F 0 "Q13" H 5150 4750 50  0000 L CNN
 F 1 "2N7000;SOT23" H 4700 4550 50  0000 L CNN
 F 2 "Package_TO_SOT_SMD:SOT-23" H 5500 4525 50  0001 L CIN
@@
 $EndComp
 $Comp
-L Device:R_US R?
+L Device:R_US R63
 U 1 1 5F3B8D54
 P 5150 3500
-F 0 "R?" V 5050 3400 50  0000 L CNN
+F 0 "R63" V 5050 3400 50  0000 L CNN
 F 1 "330Ω;1608" V 5250 3300 50  0000 L CNN
 F 2 "Resistor_SMD:R_0603_1608Metric" V 5190 3490 50  0001 C CNN
@@
 	5400 4400 5400 4300
 $Comp
-L Device:R_US R?
+L Device:R_US R62
 U 1 1 5F3B8D5F
 P 5150 3200
-F 0 "R?" V 5050 3100 50  0000 L CNN
+F 0 "R62" V 5050 3100 50  0000 L CNN
 F 1 "330Ω;1608" V 5250 3000 50  0000 L CNN
 F 2 "Resistor_SMD:R_0603_1608Metric" V 5190 3190 50  0001 C CNN
@@
 $EndComp
 $Comp
-L Device:R_US R?
+L Device:R_US R64
 U 1 1 5F3B8D69
 P 5150 3800
-F 0 "R?" V 5050 3700 50  0000 L CNN
+F 0 "R64" V 5050 3700 50  0000 L CNN
 F 1 "330Ω;1608" V 5250 3600 50  0000 L CNN
 F 2 "Resistor_SMD:R_0603_1608Metric" V 5190 3790 50  0001 C CNN
@@
 	4500 4900 4500 4800
 $Comp
-L Transistor_FET:2N7000 Q?
+L Transistor_FET:2N7000 Q12
 U 1 1 5F3BEA19
 P 4400 4600
-F 0 "Q?" H 4250 4750 50  0000 L CNN
+F 0 "Q12" H 4250 4750 50  0000 L CNN
 F 1 "2N7000;SOT23" H 3800 4550 50  0000 L CNN
 F 2 "Package_TO_SOT_SMD:SOT-23" H 4600 4525 50  0001 L CIN
@@
 $EndComp
 $Comp
-L Device:R_US R?
+L Device:R_US R60
 U 1 1 5F3BEA23
 P 4250 3500
-F 0 "R?" V 4150 3400 50  0000 L CNN
+F 0 "R60" V 4150 3400 50  0000 L CNN
 F 1 "330Ω;1608" V 4350 3300 50  0000 L CNN
 F 2 "Resistor_SMD:R_0603_1608Metric" V 4290 3490 50  0001 C CNN
@@
 $EndComp
 $Comp
-L Device:R_US R?
+L Device:R_US R59
 U 1 1 5F3BEA2E
 P 4250 3200
-F 0 "R?" V 4150 3100 50  0000 L CNN
+F 0 "R59" V 4150 3100 50  0000 L CNN
 F 1 "330Ω;1608" V 4350 3000 50  0000 L CNN
 F 2 "Resistor_SMD:R_0603_1608Metric" V 4290 3190 50  0001 C CNN
@@
 $EndComp
 $Comp
-L Device:R_US R?
+L Device:R_US R61
 U 1 1 5F3BEA38
 P 4250 3800
-F 0 "R?" V 4150 3700 50  0000 L CNN
+F 0 "R61" V 4150 3700 50  0000 L CNN
 F 1 "330Ω;1608" V 4350 3600 50  0000 L CNN
 F 2 "Resistor_SMD:R_0603_1608Metric" V 4290 3790 50  0001 C CNN
@@
 	3300 2800 3900 2800
 Wire Wire Line
-	3300 3000 3600 3000
-Wire Wire Line
 	8100 4900 7200 4900
 Wire Wire Line
@@
 	4500 4000 4500 3800
 $Comp
-L Device:LED D?
+L Device:LED D10
 U 1 1 5F30BFB1
 P 4500 4150
-F 0 "D?" V 4600 4250 50  0000 R CNN
+F 0 "D10" V 4600 4250 50  0000 R CNN
 F 1 "LED;GRNRA" V 4400 4600 50  0000 R CNN
 F 2 "HR2:LED_GRNRA" H 4500 4150 50  0001 C CNN
@@
 	6200 3800 6300 3800
 $Comp
-L Device:R_US R?
+L Device:R_US R67
 U 1 1 5F3B8D25
 P 6050 3800
-F 0 "R?" V 5950 3700 50  0000 L CNN
+F 0 "R67" V 5950 3700 50  0000 L CNN
 F 1 "330Ω;1608" V 6150 3600 50  0000 L CNN
 F 2 "Resistor_SMD:R_0603_1608Metric" V 6090 3790 50  0001 C CNN
@@
 $EndComp
 $Comp
-L Device:R_US R?
+L Device:R_US R65
 U 1 1 5F3B8D1B
 P 6050 3200
-F 0 "R?" V 5950 3100 50  0000 L CNN
+F 0 "R65" V 5950 3100 50  0000 L CNN
 F 1 "330Ω;1608" V 6150 3000 50  0000 L CNN
 F 2 "Resistor_SMD:R_0603_1608Metric" V 6090 3190 50  0001 C CNN
@@
 	6300 4400 6300 4300
 $Comp
-L Device:R_US R?
+L Device:R_US R66
 U 1 1 5F3B8D10
 P 6050 3500
-F 0 "R?" V 5950 3400 50  0000 L CNN
+F 0 "R66" V 5950 3400 50  0000 L CNN
 F 1 "330Ω;1608" V 6150 3300 50  0000 L CNN
 F 2 "Resistor_SMD:R_0603_1608Metric" V 6090 3490 50  0001 C CNN
@@
 $EndComp
 $Comp
-L Transistor_FET:2N7000 Q?
+L Transistor_FET:2N7000 Q14
 U 1 1 5F3B8D06
 P 6200 4600
-F 0 "Q?" H 6050 4750 50  0000 L CNN
+F 0 "Q14" H 6050 4750 50  0000 L CNN
 F 1 "2N7000;SOT23" H 5600 4550 50  0000 L CNN
 F 2 "Package_TO_SOT_SMD:SOT-23" H 6400 4525 50  0001 L CIN
@@
 	6300 4900 6300 4800
 $Comp
-L Device:LED D?
+L Device:LED D12
 U 1 1 5F30CF88
 P 6300 4150
-F 0 "D?" V 6400 4250 50  0000 R CNN
+F 0 "D12" V 6400 4250 50  0000 R CNN
 F 1 "LED;GRNRA" V 6200 4600 50  0000 R CNN
 F 2 "HR2:LED_GRNRA" H 6300 4150 50  0001 C CNN
@@
 Wire Wire Line
 	3300 2400 7500 2400
-Wire Wire Line
-	4500 4900 3600 4900
-Wire Wire Line
-	3600 4900 3600 3000
 Connection ~ 4500 4900
 Connection ~ 5400 4900
@@
 Connection ~ 7200 4900
 Wire Wire Line
-	3300 2900 4000 2900
-Wire Wire Line
-	4000 2900 4000 3200
+	3300 2200 4000 2200
+Wire Wire Line
+	4000 2200 4000 3200
 Connection ~ 4000 3200
 Wire Wire Line
-	4000 2900 4900 2900
-Wire Wire Line
-	4900 2900 4900 3200
-Connection ~ 4000 2900
+	4000 2200 4900 2200
+Wire Wire Line
+	4900 2200 4900 3200
+Connection ~ 4000 2200
 Connection ~ 4900 3200
 Wire Wire Line
-	4900 2900 5800 2900
-Wire Wire Line
-	5800 2900 5800 3200
-Connection ~ 4900 2900
+	4900 2200 5800 2200
+Wire Wire Line
+	5800 2200 5800 3200
+Connection ~ 4900 2200
 Connection ~ 5800 3200
 Wire Wire Line
-	5800 2900 6700 2900
-Wire Wire Line
-	6700 2900 6700 3200
-Connection ~ 5800 2900
+	5800 2200 6700 2200
+Wire Wire Line
+	6700 2200 6700 3200
+Connection ~ 5800 2200
 Connection ~ 6700 3200
 Wire Wire Line
-	6700 2900 7600 2900
-Wire Wire Line
-	7600 2900 7600 3200
-Connection ~ 6700 2900
+	6700 2200 7600 2200
+Wire Wire Line
+	7600 2200 7600 3200
+Connection ~ 6700 2200
 Connection ~ 7600 3200
 Text Label 3950 4600 0    50   ~ 0
@@
 Text Label 7550 4600 0    50   ~ 0
 LED11
-Text Label 3350 3000 0    50   ~ 0
-GND
-Text Label 3650 2900 0    50   ~ 0
+Text Label 6000 2200 0    50   ~ 0
 9V
 Text Notes 2150 4250 0    50   ~ 0
@@
 Wire Wire Line
 	4200 4600 3900 4600
+Wire Wire Line
+	3300 4900 4500 4900
+Text HLabel 3300 4900 0    50   Input ~ 0
+GND
+Text HLabel 3300 2200 0    50   Input ~ 0
+9V
+Text HLabel 3300 2400 0    50   Input ~ 0
+LED11
+Text HLabel 3300 2500 0    50   Input ~ 0
+LED10
+Text HLabel 3300 2600 0    50   Input ~ 0
+LED9
+Text HLabel 3300 2700 0    50   Input ~ 0
+LED8
+Text HLabel 3300 2800 0    50   Input ~ 0
+LED7
 $EndSCHEMATC
