File: electrical/master_board/rev_a/sonars_servos.sch (KiCad schematic (older format))
At the start: 31 parts, among them CN4 SERVO;F1x3, CN5 SERVO;F1x3, CN50 HCSR04LP;F1X4, CN51 HCSR04LP;F1X4, CN52 HCSR04LP;F1X4, CN53 HCSR04LP;F1X4, CN54 HCSR04LP;F1X4, CN6 SERVO;F1x3, CN60 HCSR04LP;F1X4, CN7 SERVO;F1x3, CN70 HCSR04LP;F1X4, U6 CD450B;TTSOP16, U7 CD450B;TTSOP16, U9 SN74HCS595;TTSOP16

Commit message: Lot's schematic work.
Connections:
- net labels added: MISC_NSS, SER_OUT
- net labels removed: DIO_NSS, SONAR_SER
- no-connect marks 4 -> 3
Changed lines of the file:
@@
 $Descr A 11000 8500
 encoding utf-8
-Sheet 9 9
+Sheet 6 9
 Title "HR2 Servos and Sonars"
 Date "2020-10-03"
@@
 MISC_MOSI
 Text HLabel 1000 4000 0    50   Output ~ 0
-SONAR_SER
+SER_OUT
 Text HLabel 1000 1200 0    50   Input ~ 0
 MISC_SCK
@@
 Wire Wire Line
 	1600 4000 1000 4000
-NoConn ~ 1200 2700
 Text Label 1700 2600 2    50   ~ 0
 3.3V
@@
 	1200 2800 1700 2800
 Text HLabel 1000 1300 0    50   Input ~ 0
-DIO_NSS
+MISC_NSS
 Wire Wire Line
 	1200 2400 1400 2400
@@
 Text Label 1900 3700 0    50   ~ 0
 GND
-NoConn ~ 1200 2900
 Text Notes 500  3900 0    50   ~ 0
 Note:\nQH is temp. No Connect.
+NoConn ~ 1200 2700
 Wire Bus Line
 	5000 2000 5000 2350

Commit message: Cleaned up schematics some.
Connections:
- net labels added: SER_IO, ~NRST
- wire segments 219 -> 213
Other:
- note added: "5 Volt Trigger Bus"
- note added: "Notes:\n1. The Sonars are HC04's that operate off of 5V.\n2. The trigger signals are provided by a serial shift register.\n3. A level shifter is used to shift trigger signals from 3.3V to 5V.\n4. A resistor voltage divider is used to convert the echo from 5V to 3.3V.\n5. Most hobby servers operate off of approximately 5V - 6V.\n6. The P5V supply is a 5V supply that is used for servos and LED's.\n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"
- note removed: "Note:\nQH is temp. No Connect."
- note removed: "Notes:\n1. The Sonars are HC04's that operate off of 5V.\n2. The trigger signals are provided by a serial shift register.\n3. A level shifter is used to shift trigger signals from 3.3V to 5V.\n4. A resistor voltage divider is used to convert the echo from 5V to 3.3V.\n5. Most hobby servers operate off of approximately 5V - 6V.\n6. The 4.8V supply is a 5V supply that is used for servos and LED's.\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"
- moved on the sheet: C10, C11, C12, U6, U7

Commit message: Bound signals to Morpho pins.
Connections:
- net labels added: DIO_MOSI, DIO_SCK, ~DIO_NSS
- net labels removed: MISC_MOSI, MISC_NSS, MISC_SCK
Changed lines of the file:
@@
 $Descr A 11000 8500
 encoding utf-8
-Sheet 6 10
+Sheet 3 10
 Title "HR2 Servos and Sonars"
 Date "2020-10-17"
@@
 	3800 3200 4750 3200
 Text HLabel 1300 2900 0    50   Input ~ 0
-MISC_MOSI
+DIO_MOSI
 Text HLabel 1300 3900 0    50   Output ~ 0
 SER_OUT
 Text HLabel 1300 3000 0    50   Input ~ 0
-MISC_SCK
+DIO_SCK
 Text HLabel 1300 3100 0    50   Input ~ 0
-MISC_NSS
+~DIO_NSS
 Text Notes 4900 1100 0    50   ~ 0
 3.3V to 5V Level Shifter
@@
 	1300 3900 3900 3900
 Text Label 1300 2900 0    50   ~ 0
-MISC_MOSI
+DIO_MOSI
 Text Label 1300 3000 0    50   ~ 0
-MISC_SCK
+DIO_SCK
 Text Label 1300 3100 0    50   ~ 0
-MISC_NSS
+~DIO_NSS
 Text Label 1300 3900 0    50   ~ 0
 SER_IO
@@
 Wire Wire Line
 	2000 5200 2000 5900
-Text Label 2000 5200 0    50   ~ 0
+Text Label 1300 5900 0    50   ~ 0
 ECHO1
 Text Label 3200 5200 0    50   ~ 0
@@
 Wire Bus Line
 	1800 2250 1800 5700
+Text Label 2000 5200 0    50   ~ 0
+ECHO1
+Text Label 1300 6000 0    50   ~ 0
+ECHO2
+Text Label 1300 6500 0    50   ~ 0
+ECHO7
+Text Label 1300 6400 0    50   ~ 0
+ECHO6
+Text Label 1300 6300 0    50   ~ 0
+ECHO5
+Text Label 1300 6200 0    50   ~ 0
+ECHO4
+Text Label 1300 6100 0    50   ~ 0
+ECHO3
 $EndSCHEMATC

Commit message: Minor tweaks prior to reannotate.
Changed lines of the file:
@@
 $Descr A 11000 8500
 encoding utf-8
-Sheet 3 10
+Sheet 8 10
 Title "HR2 Servos and Sonars"
 Date "2020-10-17"
@@
 	6550 650  6550 1300
 Wire Bus Line
-	2250 4000 6500 4000
+	2300 4000 6500 4000
 Wire Bus Line
 	6500 4000 9500 4000

Commit message: Reannoted. Postioned components are in the 80-99 reference range.
Parts:
- renumbered C10 to C17, C11 to C18, C12 to C19, CN4 to CN6, CN5 to CN7, CN6 to CN8, CN60 to CN81, CN70 to CN82, CN50 to CN83, CN51 to CN84, CN52 to CN85, CN53 to CN86, CN54 to CN87, CN7 to CN9, R48 to R23, R49 to R24, R50 to R25, R51 to R26, R52 to R27, R53 to R28, R21 to R29, R22 to R30, R54 to R31, R55 to R32, R56 to R33, R57 to R34, R58 to R35, R59 to R36, U6 to U10, U9 to U8, U7 to U9
Changed lines of the file:
@@
 $EndDescr
 $Comp
-L HR2:CD450B;TTSOP16 U6
+L HR2:CD450B;TTSOP16 U10
 U 1 1 5F56033D
 P 4750 2600
-F 0 "U6" H 5000 2750 50  0000 C CNN
+F 0 "U10" H 5000 2750 50  0000 C CNN
 F 1 "CD450B;TTSOP16" H 5300 1750 50  0000 C CNN
 F 2 "Package_SO:TSSOP-16_4.4x5mm_P0.65mm" H 4950 2650 60  0001 L CNN
@@
 Notes:\n1. The Sonars are HC04's that operate off of 5V.\n2. The trigger signals are provided by a serial shift register.\n3. A level shifter is used to shift trigger signals from 3.3V to 5V.\n4. A resistor voltage divider is used to convert the echo from 5V to 3.3V.\n5. Most hobby servers operate off of approximately 5V - 6V.\n6. The P5V supply is a 5V supply that is used for servos and LED's.\n   This supply can be noisy due to changing current draw.\n7. The servo PWM signals are level shifted from 3.3V to 5v.\n8. The servos are manually labeled to support mechanical\n   automatic positioned derived from the mechanical model.\n9. The echo signals are fed to external interrupt pins on the Nucleo PCB.
 $Comp
-L Device:C C10
+L Device:C C17
 U 1 1 5F7FE24F
 P 2350 1050
-F 0 "C10" H 2150 1150 50  0000 L CNN
+F 0 "C17" H 2150 1150 50  0000 L CNN
 F 1 "10pF;1608" H 2400 950 50  0000 L CNN
 F 2 "" H 2388 900 50  0001 C CNN
@@
 	1900 1300 1800 1200
 $Comp
-L Device:C C11
+L Device:C C18
 U 1 1 5F8B3EAF
 P 2950 1050
-F 0 "C11" H 2750 1150 50  0000 L CNN
+F 0 "C18" H 2750 1150 50  0000 L CNN
 F 1 "10pF;1608" H 3000 950 50  0000 L CNN
 F 2 "" H 2988 900 50  0001 C CNN
@@
 $EndComp
 $Comp
-L Device:C C12
+L Device:C C19
 U 1 1 5F8B4468
 P 3550 1050
-F 0 "C12" H 3350 1150 50  0000 L CNN
+F 0 "C19" H 3350 1150 50  0000 L CNN
 F 1 "10pF;1608" H 3600 950 50  0000 L CNN
 F 2 "" H 3588 900 50  0001 C CNN
@@
 SERVO4_5V
 $Comp
-L HR2:SERVO;F1x3 CN4
+L HR2:SERVO;F1x3 CN6
 U 1 1 5FB31019
 P 7550 1000
-F 0 "CN4" H 8050 1150 60  0000 R CNN
+F 0 "CN6" H 8050 1150 60  0000 R CNN
 F 1 "SERVO;F1x3" H 8200 650 60  0000 R CNN
 F 2 "Connector_PinHeader_2.54mm:PinHeader_1x03_P2.54mm_Vertical" H 7750 1050 60  0001 L CNN
@@
 $EndComp
 $Comp
-L HR2:SERVO;F1x3 CN5
+L HR2:SERVO;F1x3 CN7
 U 1 1 5FB9CF1F
 P 8550 1000
-F 0 "CN5" H 9050 1150 60  0000 R CNN
+F 0 "CN7" H 9050 1150 60  0000 R CNN
 F 1 "SERVO;F1x3" H 9200 650 60  0000 R CNN
 F 2 "Connector_PinHeader_2.54mm:PinHeader_1x03_P2.54mm_Vertical" H 8750 1050 60  0001 L CNN
@@
 $EndComp
 $Comp
-L HR2:SERVO;F1x3 CN6
+L HR2:SERVO;F1x3 CN8
 U 1 1 5FB9D556
 P 9550 1000
-F 0 "CN6" H 10050 1150 60  0000 R CNN
+F 0 "CN8" H 10050 1150 60  0000 R CNN
 F 1 "SERVO;F1x3" H 10200 650 60  0000 R CNN
 F 2 "Connector_PinHeader_2.54mm:PinHeader_1x03_P2.54mm_Vertical" H 9750 1050 60  0001 L CNN
@@
 $EndComp
 $Comp
-L HR2:SERVO;F1x3 CN7
+L HR2:SERVO;F1x3 CN9
 U 1 1 5FB9D857
 P 10500 1000
-F 0 "CN7" H 11000 1150 60  0000 R CNN
+F 0 "CN9" H 11000 1150 60  0000 R CNN
 F 1 "SERVO;F1x3" H 11150 650 60  0000 R CNN
 F 2 "Connector_PinHeader_2.54mm:PinHeader_1x03_P2.54mm_Vertical" H 10700 1050 60  0001 L CNN
@@
 	1300 1400 4750 1400
 $Comp
-L HR2:CD450B;TTSOP16 U7
+L HR2:CD450B;TTSOP16 U9
 U 1 1 5F67B87E
 P 4750 1300
-F 0 "U7" H 5000 1450 50  0000 C CNN
+F 0 "U9" H 5000 1450 50  0000 C CNN
 F 1 "CD450B;TTSOP16" H 5300 450 50  0000 C CNN
 F 2 "Package_SO:TSSOP-16_4.4x5mm_P0.65mm" H 4950 1350 60  0001 L CNN
@@
 P 3400 4400
 AR Path="/5F7F066C" Ref="CN?"  Part="1"
-AR Path="/5F48CAAD/5F7F066C" Ref="CN60"  Part="1"
-F 0 "CN60" H 3800 4550 50  0000 C CNN
+AR Path="/5F48CAAD/5F7F066C" Ref="CN81"  Part="1"
+F 0 "CN81" H 3800 4550 50  0000 C CNN
 F 1 "HCSR04LP;F1X4" H 3850 3950 50  0000 C CNN
 F 2 "HR2:HCSR04_F1x4LP" H 3600 4450 60  0001 L CNN
@@
 P 4600 4400
 AR Path="/5F7F06A3" Ref="CN?"  Part="1"
-AR Path="/5F48CAAD/5F7F06A3" Ref="CN70"  Part="1"
-F 0 "CN70" H 5000 4550 50  0000 C CNN
+AR Path="/5F48CAAD/5F7F06A3" Ref="CN82"  Part="1"
+F 0 "CN82" H 5000 4550 50  0000 C CNN
 F 1 "HCSR04LP;F1X4" H 5050 3950 50  0000 C CNN
 F 2 "HR2:HCSR04_F1x4LP" H 4800 4450 60  0001 L CNN
@@
 ECHO3_5V
 $Comp
-L Device:R_US R53
+L Device:R_US R28
 U 1 1 5F7F06EE
 P 4700 5450
-F 0 "R53" H 4750 5350 50  0000 L CNN
+F 0 "R28" H 4750 5350 50  0000 L CNN
 F 1 "33KΩ;1608" H 4250 5550 50  0000 L CNN
 F 2 "" V 4740 5440 50  0001 C CNN
@@
 $EndComp
 $Comp
-L Device:R_US R52
+L Device:R_US R27
 U 1 1 5F7F06E4
 P 4700 4950
-F 0 "R52" H 4750 4850 50  0000 L CNN
+F 0 "R27" H 4750 4850 50  0000 L CNN
 F 1 "22KΩ;1608" H 4250 5050 50  0000 L CNN
 F 2 "" V 4740 4940 50  0001 C CNN
@@
 P 5800 4400
 AR Path="/5F7F06DA" Ref="CN?"  Part="1"
-AR Path="/5F48CAAD/5F7F06DA" Ref="CN50"  Part="1"
-F 0 "CN50" H 6200 4550 50  0000 C CNN
+AR Path="/5F48CAAD/5F7F06DA" Ref="CN83"  Part="1"
+F 0 "CN83" H 6200 4550 50  0000 C CNN
 F 1 "HCSR04LP;F1X4" H 6250 3950 50  0000 C CNN
 F 2 "HR2:HCSR04_F1x4LP" H 6000 4450 60  0001 L CNN
@@
 ECHO2_5V
 $Comp
-L Device:R_US R51
+L Device:R_US R26
 U 1 1 5F7F06B7
 P 3500 5450
-F 0 "R51" H 3550 5350 50  0000 L CNN
+F 0 "R26" H 3550 5350 50  0000 L CNN
 F 1 "33KΩ;1608" H 3050 5550 50  0000 L CNN
 F 2 "" V 3540 5440 50  0001 C CNN
@@
 $EndComp
 $Comp
-L Device:R_US R50
+L Device:R_US R25
 U 1 1 5F7F06AD
 P 3500 4950
-F 0 "R50" H 3550 4850 50  0000 L CNN
+F 0 "R25" H 3550 4850 50  0000 L CNN
 F 1 "22KΩ;1608" H 3050 5050 50  0000 L CNN
 F 2 "" V 3540 4940 50  0001 C CNN
@@
 ECHO1_5V
 $Comp
-L Device:R_US R49
+L Device:R_US R24
 U 1 1 5F7F0680
 P 2300 5450
-F 0 "R49" H 2350 5350 50  0000 L CNN
+F 0 "R24" H 2350 5350 50  0000 L CNN
 F 1 "33KΩ;1608" H 1850 5550 50  0000 L CNN
 F 2 "" V 2340 5440 50  0001 C CNN
@@
 $EndComp
 $Comp
-L Device:R_US R48
+L Device:R_US R23
 U 1 1 5F7F0676
 P 2300 4950
-F 0 "R48" H 2350 4850 50  0000 L CNN
+F 0 "R23" H 2350 4850 50  0000 L CNN
 F 1 "22KΩ;1608" H 1850 5050 50  0000 L CNN
 F 2 "" V 2340 4940 50  0001 C CNN
@@
 ECHO7_5V
 $Comp
-L Device:R_US R59
+L Device:R_US R36
 U 1 1 5F7E7575
 P 9500 5450
-F 0 "R59" H 9550 5350 50  0000 L CNN
+F 0 "R36" H 9550 5350 50  0000 L CNN
 F 1 "33KΩ;1608" H 9050 5550 50  0000 L CNN
 F 2 "" V 9540 5440 50  0001 C CNN
@@
 $EndComp
 $Comp
-L Device:R_US R58
+L Device:R_US R35
 U 1 1 5F7E756B
 P 9500 4950
-F 0 "R58" H 9550 4850 50  0000 L CNN
+F 0 "R35" H 9550 4850 50  0000 L CNN
 F 1 "22KΩ;1608" H 9050 5050 50  0000 L CNN
 F 2 "" V 9540 4940 50  0001 C CNN
@@
 P 10600 4400
 AR Path="/5F7E7561" Ref="CN?"  Part="1"
-AR Path="/5F48CAAD/5F7E7561" Ref="CN54"  Part="1"
-F 0 "CN54" H 11000 4550 50  0000 C CNN
+AR Path="/5F48CAAD/5F7E7561" Ref="CN87"  Part="1"
+F 0 "CN87" H 11000 4550 50  0000 C CNN
 F 1 "HCSR04LP;F1X4" H 11050 3950 50  0000 C CNN
 F 2 "HR2:HCSR04_F1x4LP" H 10800 4450 60  0001 L CNN
@@
 ECHO6_5V
 $Comp
-L Device:R_US R57
+L Device:R_US R34
 U 1 1 5F7E753E
 P 8300 5450
-F 0 "R57" H 8350 5350 50  0000 L CNN
+F 0 "R34" H 8350 5350 50  0000 L CNN
 F 1 "33KΩ;1608" H 7850 5550 50  0000 L CNN
 F 2 "" V 8340 5440 50  0001 C CNN
@@
 $EndComp
 $Comp
-L Device:R_US R56
+L Device:R_US R33
 U 1 1 5F7E7534
 P 8300 4950
-F 0 "R56" H 8350 4850 50  0000 L CNN
+F 0 "R33" H 8350 4850 50  0000 L CNN
 F 1 "22KΩ;1608" H 7850 5050 50  0000 L CNN
 F 2 "" V 8340 4940 50  0001 C CNN
@@
 P 9400 4400
 AR Path="/5F7E752A" Ref="CN?"  Part="1"
-AR Path="/5F48CAAD/5F7E752A" Ref="CN53"  Part="1"
-F 0 "CN53" H 9800 4550 50  0000 C CNN
+AR Path="/5F48CAAD/5F7E752A" Ref="CN86"  Part="1"
+F 0 "CN86" H 9800 4550 50  0000 C CNN
 F 1 "HCSR04LP;F1X4" H 9850 3950 50  0000 C CNN
 F 2 "HR2:HCSR04_F1x4LP" H 9600 4450 60  0001 L CNN
@@
 ECHO5_5V
 $Comp
-L Device:R_US R55
+L Device:R_US R32
 U 1 1 5F7E2DCE
 P 7100 5450
-F 0 "R55" H 7150 5350 50  0000 L CNN
+F 0 "R32" H 7150 5350 50  0000 L CNN
 F 1 "33KΩ;1608" H 6650 5550 50  0000 L CNN
 F 2 "" V 7140 5440 50  0001 C CNN
@@
 $EndComp
 $Comp
-L Device:R_US R54
+L Device:R_US R31
 U 1 1 5F7E2DC4
 P 7100 4950
-F 0 "R54" H 7150 4850 50  0000 L CNN
+F 0 "R31" H 7150 4850 50  0000 L CNN
 F 1 "22KΩ;1608" H 6650 5050 50  0000 L CNN
 F 2 "" V 7140 4940 50  0001 C CNN
@@
 P 8200 4400
 AR Path="/5F7E2DBA" Ref="CN?"  Part="1"
-AR Path="/5F48CAAD/5F7E2DBA" Ref="CN52"  Part="1"
-F 0 "CN52" H 8600 4550 50  0000 C CNN
+AR Path="/5F48CAAD/5F7E2DBA" Ref="CN85"  Part="1"
+F 0 "CN85" H 8600 4550 50  0000 C CNN
 F 1 "HCSR04LP;F1X4" H 8650 3950 50  0000 C CNN
 F 2 "HR2:HCSR04_F1x4LP" H 8400 4450 60  0001 L CNN
@@
 ECHO4_5V
 $Comp
-L Device:R_US R22
+L Device:R_US R30
 U 1 1 5FADC37B
 P 5900 5450
-F 0 "R22" H 5950 5350 50  0000 L CNN
+F 0 "R30" H 5950 5350 50  0000 L CNN
 F 1 "33KΩ;1608" H 5450 5550 50  0000 L CNN
 F 2 "" V 5940 5440 50  0001 C CNN
@@
 $EndComp
 $Comp
-L Device:R_US R21
+L Device:R_US R29
 U 1 1 5FADB964
 P 5900 4950
-F 0 "R21" H 5950 4850 50  0000 L CNN
+F 0 "R29" H 5950 4850 50  0000 L CNN
 F 1 "22KΩ;1608" H 5450 5050 50  0000 L CNN
 F 2 "" V 5940 4940 50  0001 C CNN
@@
 P 7000 4400
 AR Path="/5F490633" Ref="CN?"  Part="1"
-AR Path="/5F48CAAD/5F490633" Ref="CN51"  Part="1"
-F 0 "CN51" H 7400 4550 50  0000 C CNN
+AR Path="/5F48CAAD/5F490633" Ref="CN84"  Part="1"
+F 0 "CN84" H 7400 4550 50  0000 C CNN
 F 1 "HCSR04LP;F1X4" H 7450 3950 50  0000 C CNN
 F 2 "HR2:HCSR04_F1x4LP" H 7200 4450 60  0001 L CNN
@@
 	1300 2900 2700 2900
 $Comp
-L HR2:SN74HCS595;TTSOP16 U9
+L HR2:SN74HCS595;TTSOP16 U8
 U 1 1 5FF3477F
 P 2700 2600
-F 0 "U9" H 2950 2750 60  0000 C CNN
+F 0 "U8" H 2950 2750 60  0000 C CNN
 F 1 "SN74HCS595;TTSOP16" H 3300 1450 60  0000 C CNN
 F 2 "Package_SO:TSSOP-16_4.4x5mm_P0.65mm" H 2900 2650 60  0001 L CNN

Commit message: Assigned PCB footprints.
Parts:
- C17, C18, C19: footprint (none) -> Capacitor_SMD:C_0603_1608Metric
- R23, R24, R25, R26, R27, R28, R29, R30, R31, R32, R33, R34, R35, R36: footprint (none) -> Resistor_SMD:R_0603_1608Metric
Changed lines of the file:
@@
 F 0 "C17" H 2150 1150 50  0000 L CNN
 F 1 "10pF;1608" H 2400 950 50  0000 L CNN
-F 2 "" H 2388 900 50  0001 C CNN
+F 2 "Capacitor_SMD:C_0603_1608Metric" H 2388 900 50  0001 C CNN
 F 3 "~" H 2350 1050 50  0001 C CNN
 	1    2350 1050
@@
 F 0 "C18" H 2750 1150 50  0000 L CNN
 F 1 "10pF;1608" H 3000 950 50  0000 L CNN
-F 2 "" H 2988 900 50  0001 C CNN
+F 2 "Capacitor_SMD:C_0603_1608Metric" H 2988 900 50  0001 C CNN
 F 3 "~" H 2950 1050 50  0001 C CNN
 	1    2950 1050
@@
 F 0 "C19" H 3350 1150 50  0000 L CNN
 F 1 "10pF;1608" H 3600 950 50  0000 L CNN
-F 2 "" H 3588 900 50  0001 C CNN
+F 2 "Capacitor_SMD:C_0603_1608Metric" H 3588 900 50  0001 C CNN
 F 3 "~" H 3550 1050 50  0001 C CNN
 	1    3550 1050
@@
 F 0 "R28" H 4750 5350 50  0000 L CNN
 F 1 "33KΩ;1608" H 4250 5550 50  0000 L CNN
-F 2 "" V 4740 5440 50  0001 C CNN
+F 2 "Resistor_SMD:R_0603_1608Metric" V 4740 5440 50  0001 C CNN
 F 3 "~" H 4700 5450 50  0001 C CNN
 	1    4700 5450
@@
 F 0 "R27" H 4750 4850 50  0000 L CNN
 F 1 "22KΩ;1608" H 4250 5050 50  0000 L CNN
-F 2 "" V 4740 4940 50  0001 C CNN
+F 2 "Resistor_SMD:R_0603_1608Metric" V 4740 4940 50  0001 C CNN
 F 3 "~" H 4700 4950 50  0001 C CNN
 	1    4700 4950
@@
 F 0 "R26" H 3550 5350 50  0000 L CNN
 F 1 "33KΩ;1608" H 3050 5550 50  0000 L CNN
-F 2 "" V 3540 5440 50  0001 C CNN
+F 2 "Resistor_SMD:R_0603_1608Metric" V 3540 5440 50  0001 C CNN
 F 3 "~" H 3500 5450 50  0001 C CNN
 	1    3500 5450
@@
 F 0 "R25" H 3550 4850 50  0000 L CNN
 F 1 "22KΩ;1608" H 3050 5050 50  0000 L CNN
-F 2 "" V 3540 4940 50  0001 C CNN
+F 2 "Resistor_SMD:R_0603_1608Metric" V 3540 4940 50  0001 C CNN
 F 3 "~" H 3500 4950 50  0001 C CNN
 	1    3500 4950
@@
 F 0 "R24" H 2350 5350 50  0000 L CNN
 F 1 "33KΩ;1608" H 1850 5550 50  0000 L CNN
-F 2 "" V 2340 5440 50  0001 C CNN
+F 2 "Resistor_SMD:R_0603_1608Metric" V 2340 5440 50  0001 C CNN
 F 3 "~" H 2300 5450 50  0001 C CNN
 	1    2300 5450
@@
 F 0 "R23" H 2350 4850 50  0000 L CNN
 F 1 "22KΩ;1608" H 1850 5050 50  0000 L CNN
-F 2 "" V 2340 4940 50  0001 C CNN
+F 2 "Resistor_SMD:R_0603_1608Metric" V 2340 4940 50  0001 C CNN
 F 3 "~" H 2300 4950 50  0001 C CNN
 	1    2300 4950
@@
 F 0 "R36" H 9550 5350 50  0000 L CNN
 F 1 "33KΩ;1608" H 9050 5550 50  0000 L CNN
-F 2 "" V 9540 5440 50  0001 C CNN
+F 2 "Resistor_SMD:R_0603_1608Metric" V 9540 5440 50  0001 C CNN
 F 3 "~" H 9500 5450 50  0001 C CNN
 	1    9500 5450
@@
 F 0 "R35" H 9550 4850 50  0000 L CNN
 F 1 "22KΩ;1608" H 9050 5050 50  0000 L CNN
-F 2 "" V 9540 4940 50  0001 C CNN
+F 2 "Resistor_SMD:R_0603_1608Metric" V 9540 4940 50  0001 C CNN
 F 3 "~" H 9500 4950 50  0001 C CNN
 	1    9500 4950
@@
 F 0 "R34" H 8350 5350 50  0000 L CNN
 F 1 "33KΩ;1608" H 7850 5550 50  0000 L CNN
-F 2 "" V 8340 5440 50  0001 C CNN
+F 2 "Resistor_SMD:R_0603_1608Metric" V 8340 5440 50  0001 C CNN
 F 3 "~" H 8300 5450 50  0001 C CNN
 	1    8300 5450
@@
 F 0 "R33" H 8350 4850 50  0000 L CNN
 F 1 "22KΩ;1608" H 7850 5050 50  0000 L CNN
-F 2 "" V 8340 4940 50  0001 C CNN
+F 2 "Resistor_SMD:R_0603_1608Metric" V 8340 4940 50  0001 C CNN
 F 3 "~" H 8300 4950 50  0001 C CNN
 	1    8300 4950
@@
 F 0 "R32" H 7150 5350 50  0000 L CNN
 F 1 "33KΩ;1608" H 6650 5550 50  0000 L CNN
-F 2 "" V 7140 5440 50  0001 C CNN
+F 2 "Resistor_SMD:R_0603_1608Metric" V 7140 5440 50  0001 C CNN
 F 3 "~" H 7100 5450 50  0001 C CNN
 	1    7100 5450
@@
 F 0 "R31" H 7150 4850 50  0000 L CNN
 F 1 "22KΩ;1608" H 6650 5050 50  0000 L CNN
-F 2 "" V 7140 4940 50  0001 C CNN
+F 2 "Resistor_SMD:R_0603_1608Metric" V 7140 4940 50  0001 C CNN
 F 3 "~" H 7100 4950 50  0001 C CNN
 	1    7100 4950
@@
 F 0 "R30" H 5950 5350 50  0000 L CNN
 F 1 "33KΩ;1608" H 5450 5550 50  0000 L CNN
-F 2 "" V 5940 5440 50  0001 C CNN
+F 2 "Resistor_SMD:R_0603_1608Metric" V 5940 5440 50  0001 C CNN
 F 3 "~" H 5900 5450 50  0001 C CNN
 	1    5900 5450
@@
 F 0 "R29" H 5950 4850 50  0000 L CNN
 F 1 "22KΩ;1608" H 5450 5050 50  0000 L CNN
-F 2 "" V 5940 4940 50  0001 C CNN
+F 2 "Resistor_SMD:R_0603_1608Metric" V 5940 4940 50  0001 C CNN
 F 3 "~" H 5900 4950 50  0001 C CNN
 	1    5900 4950
