File: electrical/master_board/rev_a/sonars_servos.sch (KiCad schematic (older format))
At the start: 21 parts, among them CN6 SERVO;M1x3, CN7 SERVO;M1x3, CN8 SERVO;M1x3, CN81 HCSR04LP;F1X4, CN82 HCSR04LP;F1X4, CN83 HCSR04LP;F1X4, CN84 HCSR04LP;F1X4, CN85 HCSR04LP;F1X4, CN86 HCSR04LP;F1X4, CN87 HCSR04LP;F1X4, CN9 SERVO;M1x4, U10 CD4504B;TTSOP16, U19 ACS711;SOIC8, U8 SN74HC595;TTSOP16, U9 CD4504B;TTSOP16

Commit message: JLCPCB Footprints are both consistent and available.
Parts:
- removed U8: SN74HC595;TTSOP16, Package_SO:TSSOP-16_4.4x5mm_P0.65mm, symbol HR2:SN74HCS595;TTSOP16
- added U8: SN74HC595;HTSSOP16EP3.4x5, Package_SO:HTSSOP-16-1EP_4.4x5mm_P0.65mm_EP3.4x5mm, symbol HR2:SN74HC595;HTSSOP16EP3.4x5
Changed lines of the file:
@@
 Wire Wire Line
 	1000 2900 2400 2900
-$Comp
-L HR2:SN74HCS595;TTSOP16 U8
-U 1 1 5FF3477F
-P 2400 2600
-F 0 "U8" H 2650 2750 60  0000 C CNN
-F 1 "SN74HC595;TTSOP16" H 3000 1450 60  0000 C CNN
-F 2 "Package_SO:TSSOP-16_4.4x5mm_P0.65mm" H 2600 2650 60  0001 L CNN
-F 3 "Tri-state 8-Bit Shift Register" H 2600 2450 60  0001 L CNN
-F 4 "Tri-State 8-Bit Shift Register" H 2600 2350 60  0001 L CNN "Field5"
-	1    2400 2600
-	1    0    0    -1
-$EndComp
 Wire Wire Line
 	4100 3600 4350 3600
@@
 Wire Bus Line
 	6200 1900 6200 4000
+$Comp
+L HR2:SN74HC595;HTSSOP16EP3.4x5 U8
+U 1 1 5FE28106
+P 2400 2600
+F 0 "U8" H 2650 2750 50  0000 C CNN
+F 1 "SN74HC595;HTSSOP16EP3.4x5" H 2950 1450 50  0000 C CNN
+F 2 "Package_SO:HTSSOP-16-1EP_4.4x5mm_P0.65mm_EP3.4x5mm" H 2600 2650 60  0001 L CNN
+F 3 "Tri-state 8-Bit Shift Register" H 2600 2450 60  0001 L CNN
+F 4 "Tri-State 8-Bit Shift Register" H 2600 2350 60  0001 L CNN "desc"
+	1    2400 2600
+	1    0    0    -1
+$EndComp
 $EndSCHEMATC

Commit message: Converted '165/'595 back to TSSOP-16's.
Parts:
- removed U8: SN74HC595;HTSSOP16EP3.4x5, Package_SO:HTSSOP-16-1EP_4.4x5mm_P0.65mm_EP3.4x5mm, symbol HR2:SN74HC595;HTSSOP16EP3.4x5
- added U8: SN74HC595;TSSOP16, Package_SO:TSSOP-16_4.4x5mm_P0.65mm, symbol HR2:SN74HC595;TSSOP16
Changed lines of the file:
@@
 3.3V to 5V Level Shifter
 Text Notes 6300 3800 0    50   ~ 0
-Notes:\n1. The Sonars are HC04's that operate off of 5V.\n2. The trigger signals are provided by a serial shift register.\n3. A level shifter is used to shift trigger signals from 3.3V to 5V.\n4. The microcontroller has 5V tolerant input pins.\n5. Most hobby servers operate off of approximately 5V - 6V.\n6. The P5V supply is a 5V supply that is used for servos and LED's.\n   This supply can be noisy due to changing current draw.\n7. The servo PWM signals are level shifted from 3.3V to 5V.\n8. The servos are manually labeled to support mechanical\n   automatic positioned derived from the mechanical model.\n9. The echo signals are fed to external interrupt pins on the Nucleo PCB.
+Notes:\n1. The Sonars are HC04's that operate off of 5V.\n2. The trigger signals are provided by a serial shift register.\n3. A level shifter is used to shift trigger signals from 3.3V to 5V.\n4. The microcontroller has 5V tolerant input pins.\n5. Most hobby servers operate off of approximately 5V - 6V.\n6. The P5V supply is a 5V supply that is used for servos and LED's.\n   This supply can be noisy due to changing current draw.\n7. The servo PWM signals are level shifted from 3.3V to 5V.\n8. Some of the servos have an extra 4th wire the provides a\n    voltage that indicates servo position between 0V-5V.\n9. The echo signals are fed to external interrupt pins on the Nucleo PCB.
 Wire Wire Line
 	2050 900  2050 800
@@
 Text Label 9300 3100 0    50   ~ 0
 GND
-$Comp
-L HR2:SN74HC595;HTSSOP16EP3.4x5 U8
-U 1 1 5FE28106
+Wire Bus Line
+	4000 2000 4000 2250
+Wire Bus Line
+	6000 2250 6000 2600
+Wire Bus Line
+	4000 2250 6000 2250
+Wire Bus Line
+	4000 650  4000 1300
+Wire Bus Line
+	1500 650  1500 2250
+Wire Bus Line
+	8200 650  8200 1100
+Wire Bus Line
+	4000 2250 4000 3600
+Wire Bus Line
+	6200 4000 9200 4000
+Wire Bus Line
+	2000 4000 6200 4000
+Wire Bus Line
+	7200 650  7200 2700
+Wire Bus Line
+	6200 650  6200 1300
+Wire Bus Line
+	9200 650  9200 3100
+Wire Bus Line
+	1500 2250 1500 5050
+Wire Bus Line
+	6200 1900 6200 4000
+$Comp
+L HR2:SN74HC595;TSSOP16 U8
+U 1 1 5FEA6955
 P 2400 2600
-F 0 "U8" H 2650 2750 50  0000 C CNN
-F 1 "SN74HC595;HTSSOP16EP3.4x5" H 2950 1450 50  0000 C CNN
-F 2 "Package_SO:HTSSOP-16-1EP_4.4x5mm_P0.65mm_EP3.4x5mm" H 2600 2650 60  0001 L CNN
+F 0 "U8" H 2650 2750 60  0000 C CNN
+F 1 "SN74HC595;TSSOP16" H 2950 1450 50  0000 C CNN
+F 2 "Package_SO:TSSOP-16_4.4x5mm_P0.65mm" H 2600 2650 60  0001 L CNN
 F 3 "Tri-state 8-Bit Shift Register" H 2600 2450 60  0001 L CNN
 F 4 "Tri-State 8-Bit Shift Register" H 2600 2350 60  0001 L CNN "desc"
@@
 	1    0    0    -1
 $EndComp
-Wire Bus Line
-	4000 2000 4000 2250
-Wire Bus Line
-	6000 2250 6000 2600
-Wire Bus Line
-	4000 2250 6000 2250
-Wire Bus Line
-	4000 650  4000 1300
-Wire Bus Line
-	1500 650  1500 2250
-Wire Bus Line
-	8200 650  8200 1100
-Wire Bus Line
-	4000 2250 4000 3600
-Wire Bus Line
-	6200 4000 9200 4000
-Wire Bus Line
-	2000 4000 6200 4000
-Wire Bus Line
-	7200 650  7200 2700
-Wire Bus Line
-	6200 650  6200 1300
-Wire Bus Line
-	9200 650  9200 3100
-Wire Bus Line
-	1500 2250 1500 5050
-Wire Bus Line
-	6200 1900 6200 4000
 $EndSCHEMATC

Commit message: Servo1 volt. divider.  Added pin 1's
Parts:
- added R24: 2.2KΩ;1005, Resistor_SMD:R_0402_1005Metric, symbol Device:R_US
- added R25: 3.3KΩ;1005, Resistor_SMD:R_0402_1005Metric, symbol Device:R_US
Connections:
- wire segments 186 -> 192
Other:
- note added: "5V=>3V\nVoltage\nDivider"
Changed lines of the file:
@@
 	8350 1200 8500 1200
 Wire Wire Line
-	9300 1700 9300 1200
-Wire Wire Line
-	9300 1200 9500 1200
+	9300 1100 9500 1100
 Wire Wire Line
 	3500 3000 4450 3000
@@
 	8200 900  8300 1000
 Wire Wire Line
+	9500 900  9300 900
+Wire Wire Line
 	9500 1000 9300 1000
-Wire Wire Line
-	9500 1100 9300 1100
+Text Label 9300 900  0    50   ~ 0
+SGND
 Text Label 9300 1000 0    50   ~ 0
-SGND
-Text Label 9300 1100 0    50   ~ 0
 P5V
 Entry Wire Line
-	9300 1100 9200 1000
-Entry Wire Line
-	9200 900  9300 1000
+	9300 1000 9200 900
+Entry Wire Line
+	9200 800  9300 900
 Wire Bus Line
 	9200 650  8200 650
@@
 L HR2:SERVO;M1x4 CN9
 U 1 1 5FC1E3A4
-P 10200 1000
-F 0 "CN9" H 10650 1150 50  0000 C CNN
-F 1 "SERVO;M1x4" H 10550 550 50  0000 C CNN
-F 2 "Connector_PinHeader_2.54mm:PinHeader_1x04_P2.54mm_Vertical" H 10400 1050 60  0001 L CNN
-F 3 "Servo M1X4" H 10400 850 60  0001 L CNN
-F 4 "Servo M1X4" H 10400 750 60  0001 L CNN "Field5"
-	1    10200 1000
+P 10200 900
+F 0 "CN9" H 10650 1050 50  0000 C CNN
+F 1 "SERVO;M1x4" H 10550 450 50  0000 C CNN
+F 2 "Connector_PinHeader_2.54mm:PinHeader_1x04_P2.54mm_Vertical" H 10400 950 60  0001 L CNN
+F 3 "Servo M1X4" H 10400 750 60  0001 L CNN
+F 4 "Servo M1X4" H 10400 650 60  0001 L CNN "Field5"
+	1    10200 900
 	-1   0    0    -1
 $EndComp
@@
 3.3V
 Wire Wire Line
-	9500 1300 9400 1300
-Wire Wire Line
-	9400 1300 9400 1700
-Wire Wire Line
-	9400 1700 10400 1700
-Wire Wire Line
-	10400 1700 10400 6050
+	9500 1200 9400 1200
+Wire Wire Line
+	9400 1200 9400 1500
 Wire Wire Line
 	10400 6050 1000 6050
@@
 Text Label 9300 3100 0    50   ~ 0
 GND
-Wire Bus Line
-	4000 2000 4000 2250
-Wire Bus Line
-	6000 2250 6000 2600
-Wire Bus Line
-	4000 2250 6000 2250
-Wire Bus Line
-	4000 650  4000 1300
-Wire Bus Line
-	1500 650  1500 2250
-Wire Bus Line
-	8200 650  8200 1100
-Wire Bus Line
-	4000 2250 4000 3600
-Wire Bus Line
-	6200 4000 9200 4000
-Wire Bus Line
-	2000 4000 6200 4000
-Wire Bus Line
-	7200 650  7200 2700
-Wire Bus Line
-	6200 650  6200 1300
-Wire Bus Line
-	9200 650  9200 3100
-Wire Bus Line
-	1500 2250 1500 5050
-Wire Bus Line
-	6200 1900 6200 4000
 $Comp
 L HR2:SN74HC595;TSSOP16 U8
@@
 	1    0    0    -1
 $EndComp
+$Comp
+L Device:R_US R?
+U 1 1 5FEA8596
+P 10200 1750
+AR Path="/5F8C2F57/5FEA8596" Ref="R?"  Part="1"
+AR Path="/5F48CAAD/5FEA8596" Ref="R24"  Part="1"
+F 0 "R24" H 10050 1850 50  0000 L CNN
+F 1 "2.2KΩ;1005" H 9750 1600 50  0000 L CNN
+F 2 "Resistor_SMD:R_0402_1005Metric" V 10240 1740 50  0001 C CNN
+F 3 "~" H 10200 1750 50  0001 C CNN
+	1    10200 1750
+	1    0    0    -1
+$EndComp
+$Comp
+L Device:R_US R?
+U 1 1 5FEA8A70
+P 10200 2250
+AR Path="/5F8C2F57/5FEA8A70" Ref="R?"  Part="1"
+AR Path="/5F48CAAD/5FEA8A70" Ref="R25"  Part="1"
+F 0 "R25" H 10050 2350 50  0000 L CNN
+F 1 "3.3KΩ;1005" H 9750 2100 50  0000 L CNN
+F 2 "Resistor_SMD:R_0402_1005Metric" V 10240 2240 50  0001 C CNN
+F 3 "~" H 10200 2250 50  0001 C CNN
+	1    10200 2250
+	1    0    0    -1
+$EndComp
+Wire Wire Line
+	9900 3100 10200 3100
+Wire Wire Line
+	10200 3100 10200 2400
+Connection ~ 9900 3100
+Wire Wire Line
+	10200 2100 10200 2000
+Wire Wire Line
+	9300 1100 9300 1700
+Wire Wire Line
+	10200 1600 10200 1500
+Wire Wire Line
+	10200 1500 9400 1500
+Wire Wire Line
+	10200 2000 10400 2000
+Connection ~ 10200 2000
+Wire Wire Line
+	10200 2000 10200 1900
+Wire Wire Line
+	10400 2000 10400 6050
+Text Notes 9500 2250 0    50   ~ 0
+5V=>3V\nVoltage\nDivider
+Wire Bus Line
+	4000 2000 4000 2250
+Wire Bus Line
+	6000 2250 6000 2600
+Wire Bus Line
+	4000 2250 6000 2250
+Wire Bus Line
+	4000 650  4000 1300
+Wire Bus Line
+	1500 650  1500 2250
+Wire Bus Line
+	8200 650  8200 1100
+Wire Bus Line
+	4000 2250 4000 3600
+Wire Bus Line
+	6200 4000 9200 4000
+Wire Bus Line
+	2000 4000 6200 4000
+Wire Bus Line
+	7200 650  7200 2700
+Wire Bus Line
+	6200 650  6200 1300
+Wire Bus Line
+	9200 650  9200 3100
+Wire Bus Line
+	1500 2250 1500 5050
+Wire Bus Line
+	6200 1900 6200 4000
 $EndSCHEMATC

Commit message: Reannoated schematic symbols.
Parts:
- renumbered C17 to C13, C18 to C14, C19 to C15, C1 to C16, CN82 to CN10, CN83 to CN11, CN84 to CN12, CN6 to CN13, CN85 to CN14, CN7 to CN15, CN86 to CN16, CN8 to CN17, CN9 to CN18, CN87 to CN19, CN81 to CN9, R4 to R43, R23 to R44, R24 to R45, R25 to R46, U9 to U10, U10 to U11, U19 to U12, U8 to U9
Changed lines of the file:
@@
 $EndDescr
 $Comp
-L HR2:CD450B;TTSOP16 U10
+L HR2:CD450B;TTSOP16 U11
 U 1 1 5F56033D
 P 4450 2600
-F 0 "U10" H 4700 2750 50  0000 C CNN
+F 0 "U11" H 4700 2750 50  0000 C CNN
 F 1 "CD4504B;TTSOP16" H 5000 1750 50  0000 C CNN
 F 2 "Package_SO:TSSOP-16_4.4x5mm_P0.65mm" H 4650 2650 60  0001 L CNN
@@
 	1600 1300 1500 1200
 $Comp
-L Device:C C18
+L Device:C C14
 U 1 1 5F8B3EAF
 P 2650 1050
-F 0 "C18" H 2450 1150 50  0000 L CNN
+F 0 "C14" H 2450 1150 50  0000 L CNN
 F 1 "0.1µF;1005" H 2700 950 50  0000 L CNN
 F 2 "Capacitor_SMD:C_0402_1005Metric" H 2688 900 50  0001 C CNN
@@
 $EndComp
 $Comp
-L Device:C C19
+L Device:C C15
 U 1 1 5F8B4468
 P 3250 1050
-F 0 "C19" H 3050 1150 50  0000 L CNN
+F 0 "C15" H 3050 1150 50  0000 L CNN
 F 1 "0.1µF;1005" H 3300 950 50  0000 L CNN
 F 2 "Capacitor_SMD:C_0402_1005Metric" H 3288 900 50  0001 C CNN
@@
 	1000 1400 4450 1400
 $Comp
-L HR2:CD450B;TTSOP16 U9
+L HR2:CD450B;TTSOP16 U10
 U 1 1 5F67B87E
 P 4450 1300
-F 0 "U9" H 4700 1450 50  0000 C CNN
+F 0 "U10" H 4700 1450 50  0000 C CNN
 F 1 "CD4504B;TTSOP16" H 5000 450 50  0000 C CNN
 F 2 "Package_SO:TSSOP-16_4.4x5mm_P0.65mm" H 4650 1350 60  0001 L CNN
@@
 P 3100 4400
 AR Path="/5F7F066C" Ref="CN?"  Part="1"
-AR Path="/5F48CAAD/5F7F066C" Ref="CN81"  Part="1"
-F 0 "CN81" H 3500 4550 50  0000 C CNN
+AR Path="/5F48CAAD/5F7F066C" Ref="CN9"  Part="1"
+F 0 "CN9" H 3500 4550 50  0000 C CNN
 F 1 "HCSR04LP;F1X4" H 3550 3950 50  0000 C CNN
 F 2 "HR2:HCSR04_F1x4H" H 3300 4450 60  0001 L CNN
@@
 P 4300 4400
 AR Path="/5F7F06A3" Ref="CN?"  Part="1"
-AR Path="/5F48CAAD/5F7F06A3" Ref="CN82"  Part="1"
-F 0 "CN82" H 4700 4550 50  0000 C CNN
+AR Path="/5F48CAAD/5F7F06A3" Ref="CN10"  Part="1"
+F 0 "CN10" H 4700 4550 50  0000 C CNN
 F 1 "HCSR04LP;F1X4" H 4750 3950 50  0000 C CNN
 F 2 "HR2:HCSR04_F1x4H" H 4500 4450 60  0001 L CNN
@@
 P 5500 4400
 AR Path="/5F7F06DA" Ref="CN?"  Part="1"
-AR Path="/5F48CAAD/5F7F06DA" Ref="CN83"  Part="1"
-F 0 "CN83" H 5900 4550 50  0000 C CNN
+AR Path="/5F48CAAD/5F7F06DA" Ref="CN11"  Part="1"
+F 0 "CN11" H 5900 4550 50  0000 C CNN
 F 1 "HCSR04LP;F1X4" H 5950 3950 50  0000 C CNN
 F 2 "HR2:HCSR04_F1x4" H 5700 4450 60  0001 L CNN
@@
 P 10300 4400
 AR Path="/5F7E7561" Ref="CN?"  Part="1"
-AR Path="/5F48CAAD/5F7E7561" Ref="CN87"  Part="1"
-F 0 "CN87" H 10700 4550 50  0000 C CNN
+AR Path="/5F48CAAD/5F7E7561" Ref="CN19"  Part="1"
+F 0 "CN19" H 10700 4550 50  0000 C CNN
 F 1 "HCSR04LP;F1X4" H 10750 3950 50  0000 C CNN
 F 2 "HR2:HCSR04_F1x4" H 10500 4450 60  0001 L CNN
@@
 P 9100 4400
 AR Path="/5F7E752A" Ref="CN?"  Part="1"
-AR Path="/5F48CAAD/5F7E752A" Ref="CN86"  Part="1"
-F 0 "CN86" H 9500 4550 50  0000 C CNN
+AR Path="/5F48CAAD/5F7E752A" Ref="CN16"  Part="1"
+F 0 "CN16" H 9500 4550 50  0000 C CNN
 F 1 "HCSR04LP;F1X4" H 9550 3950 50  0000 C CNN
 F 2 "HR2:HCSR04_F1x4LP" H 9300 4450 60  0001 L CNN
@@
 P 7900 4400
 AR Path="/5F7E2DBA" Ref="CN?"  Part="1"
-AR Path="/5F48CAAD/5F7E2DBA" Ref="CN85"  Part="1"
-F 0 "CN85" H 8300 4550 50  0000 C CNN
+AR Path="/5F48CAAD/5F7E2DBA" Ref="CN14"  Part="1"
+F 0 "CN14" H 8300 4550 50  0000 C CNN
 F 1 "HCSR04LP;F1X4" H 8350 3950 50  0000 C CNN
 F 2 "HR2:HCSR04_F1x4LP" H 8100 4450 60  0001 L CNN
@@
 P 6700 4400
 AR Path="/5F490633" Ref="CN?"  Part="1"
-AR Path="/5F48CAAD/5F490633" Ref="CN84"  Part="1"
-F 0 "CN84" H 7100 4550 50  0000 C CNN
+AR Path="/5F48CAAD/5F490633" Ref="CN12"  Part="1"
+F 0 "CN12" H 7100 4550 50  0000 C CNN
 F 1 "HCSR04LP;F1X4" H 7150 3950 50  0000 C CNN
 F 2 "HR2:HCSR04_F1x4LP" H 6900 4450 60  0001 L CNN
@@
 ECHO3
 $Comp
-L HR2:ACS711;SOIC8 U19
+L HR2:ACS711;SOIC8 U12
 U 1 1 5FC1C86E
 P 7600 2400
-F 0 "U19" H 7850 2550 50  0000 C CNN
+F 0 "U12" H 7850 2550 50  0000 C CNN
 F 1 "ACS711;SOIC8" H 8100 1950 50  0000 C CNN
 F 2 "Package_SO:SOIC-8_3.9x4.9mm_P1.27mm" H 7800 2450 60  0001 L CNN
@@
 $EndComp
 $Comp
-L HR2:SERVO;M1x3 CN6
+L HR2:SERVO;M1x3 CN13
 U 1 1 5FC1D721
 P 7200 1000
-F 0 "CN6" H 7700 1150 50  0000 R CNN
+F 0 "CN13" H 7700 1150 50  0000 R CNN
 F 1 "SERVO;M1x3" H 7800 650 50  0000 R CNN
 F 2 "Connector_PinHeader_2.54mm:PinHeader_1x03_P2.54mm_Vertical" H 7400 1050 60  0001 L CNN
@@
 $EndComp
 $Comp
-L HR2:SERVO;M1x4 CN9
+L HR2:SERVO;M1x4 CN18
 U 1 1 5FC1E3A4
 P 10200 900
-F 0 "CN9" H 10650 1050 50  0000 C CNN
+F 0 "CN18" H 10650 1050 50  0000 C CNN
 F 1 "SERVO;M1x4" H 10550 450 50  0000 C CNN
 F 2 "Connector_PinHeader_2.54mm:PinHeader_1x04_P2.54mm_Vertical" H 10400 950 60  0001 L CNN
@@
 $EndComp
 $Comp
-L HR2:SERVO;M1x3 CN7
+L HR2:SERVO;M1x3 CN15
 U 1 1 5FC20D64
 P 8200 1000
-F 0 "CN7" H 8700 1150 50  0000 R CNN
+F 0 "CN15" H 8700 1150 50  0000 R CNN
 F 1 "SERVO;M1x3" H 8800 650 50  0000 R CNN
 F 2 "Connector_PinHeader_2.54mm:PinHeader_1x03_P2.54mm_Vertical" H 8400 1050 60  0001 L CNN
@@
 $EndComp
 $Comp
-L HR2:SERVO;M1x3 CN8
+L HR2:SERVO;M1x3 CN17
 U 1 1 5FC214E7
 P 9200 1000
-F 0 "CN8" H 9700 1150 50  0000 R CNN
+F 0 "CN17" H 9700 1150 50  0000 R CNN
 F 1 "SERVO;M1x3" H 9800 650 50  0000 R CNN
 F 2 "Connector_PinHeader_2.54mm:PinHeader_1x03_P2.54mm_Vertical" H 9400 1050 60  0001 L CNN
@@
 	7100 4700 7100 5050
 $Comp
-L Device:C C17
+L Device:C C13
 U 1 1 5F7FE24F
 P 2050 1050
-F 0 "C17" H 1850 1150 50  0000 L CNN
+F 0 "C13" H 1850 1150 50  0000 L CNN
 F 1 "0.1µF;1005" H 2100 950 50  0000 L CNN
 F 2 "Capacitor_SMD:C_0402_1005Metric" H 2088 900 50  0001 C CNN
@@
 P 8800 2050
 AR Path="/5F8C2F57/5FE95610" Ref="R?"  Part="1"
-AR Path="/5F48CAAD/5FE95610" Ref="R4"  Part="1"
-F 0 "R4" H 8700 2150 50  0000 L CNN
+AR Path="/5F48CAAD/5FE95610" Ref="R43"  Part="1"
+F 0 "R43" H 8700 2150 50  0000 L CNN
 F 1 "100KΩ;1005" H 8300 1900 50  0000 L CNN
 F 2 "Resistor_SMD:R_0402_1005Metric" V 8840 2040 50  0001 C CNN
@@
 P 9500 2500
 AR Path="/5F8C2F57/5FEE50CC" Ref="R?"  Part="1"
-AR Path="/5F48CAAD/5FEE50CC" Ref="R23"  Part="1"
-F 0 "R23" V 9400 2400 50  0000 L CNN
+AR Path="/5F48CAAD/5FEE50CC" Ref="R44"  Part="1"
+F 0 "R44" V 9400 2400 50  0000 L CNN
 F 1 "1KΩ;1005" V 9600 2350 50  0000 L CNN
 F 2 "Resistor_SMD:R_0402_1005Metric" V 9540 2490 50  0001 C CNN
@@
 	9650 2500 9900 2500
 $Comp
-L Device:C C1
+L Device:C C16
 U 1 1 5FEE702F
 P 9900 2850
-F 0 "C1" H 9700 2950 50  0000 L CNN
+F 0 "C16" H 9700 2950 50  0000 L CNN
 F 1 "0.01µF;1005" H 9350 2750 50  0000 L CNN
 F 2 "Capacitor_SMD:C_0402_1005Metric" H 9938 2700 50  0001 C CNN
@@
 GND
 $Comp
-L HR2:SN74HC595;TSSOP16 U8
+L HR2:SN74HC595;TSSOP16 U9
 U 1 1 5FEA6955
 P 2400 2600
-F 0 "U8" H 2650 2750 60  0000 C CNN
+F 0 "U9" H 2650 2750 60  0000 C CNN
 F 1 "SN74HC595;TSSOP16" H 2950 1450 50  0000 C CNN
 F 2 "Package_SO:TSSOP-16_4.4x5mm_P0.65mm" H 2600 2650 60  0001 L CNN
@@
 P 10200 1750
 AR Path="/5F8C2F57/5FEA8596" Ref="R?"  Part="1"
-AR Path="/5F48CAAD/5FEA8596" Ref="R24"  Part="1"
-F 0 "R24" H 10050 1850 50  0000 L CNN
+AR Path="/5F48CAAD/5FEA8596" Ref="R45"  Part="1"
+F 0 "R45" H 10050 1850 50  0000 L CNN
 F 1 "2.2KΩ;1005" H 9750 1600 50  0000 L CNN
 F 2 "Resistor_SMD:R_0402_1005Metric" V 10240 1740 50  0001 C CNN
@@
 P 10200 2250
 AR Path="/5F8C2F57/5FEA8A70" Ref="R?"  Part="1"
-AR Path="/5F48CAAD/5FEA8A70" Ref="R25"  Part="1"
-F 0 "R25" H 10050 2350 50  0000 L CNN
+AR Path="/5F48CAAD/5FEA8A70" Ref="R46"  Part="1"
+F 0 "R46" H 10050 2350 50  0000 L CNN
 F 1 "3.3KΩ;1005" H 9750 2100 50  0000 L CNN
 F 2 "Resistor_SMD:R_0402_1005Metric" V 10240 2240 50  0001 C CNN
