File: electrical/master_board/rev_a/power.sch (KiCad schematic (older format))
At the start: 21 parts, among them CN1 AMP10103594-0001LF;USB1x6H, CN2 AMP10103594-0001LF;USB1x6H, CN42 POLOLU_U3V70F9;F1x4+F1x5, Q1 2N2222;SOT23, Q2 PFET_6A_GSD;SOT23, Q3 2N2222;SOT23, SW1 PTS645SK50SMTR92 LFS;6x9.5, U4 LM66100;SOT363

Commit message: Added WOWBus Schematic Sheet.
Connections:
- wire segments 100 -> 103
Other:
- moved on the sheet: Q2
Changed lines of the file:
@@
 $Descr A 11000 8500
 encoding utf-8
-Sheet 2 9
+Sheet 2 10
 Title "HR2 Power"
-Date "2020-10-03"
+Date "2020-10-17"
 Rev "A"
 Comp "HomeBrew Robotics Club"
@@
 Text HLabel 8750 3200 2    50   Output ~ 0
 9V
-Text HLabel 8750 4300 2    50   Output ~ 0
+Text HLabel 8750 4400 2    50   Output ~ 0
 5V
 Wire Wire Line
@@
 	2950 4900 3600 4900
 Wire Wire Line
-	3600 4900 3600 4800
-Wire Wire Line
 	2950 5000 2950 4900
 Connection ~ 2950 4900
 Wire Wire Line
-	4200 4600 4200 4300
+	4200 4600 4200 4400
 Wire Wire Line
 	3250 5200 4200 5200
@@
 Connection ~ 2950 4300
 Wire Wire Line
-	4200 4300 4800 4300
-Wire Wire Line
-	4800 4300 4800 4600
-Connection ~ 4200 4300
+	4200 4400 4800 4400
+Wire Wire Line
+	4800 4400 4800 4600
+Connection ~ 4200 4400
 Wire Wire Line
 	4700 5200 5300 5200
@@
 	2950 6000 4800 6000
 Connection ~ 4800 6000
-Connection ~ 4800 4300
+Connection ~ 4800 4400
 Wire Wire Line
 	4800 5600 4800 5500
@@
 	7800 3600 7800 3500
 Wire Wire Line
-	4800 4300 6150 4300
-Wire Wire Line
-	7800 3600 7800 4300
+	4800 4400 6150 4400
+Wire Wire Line
+	7800 3600 7800 4400
 $Comp
 L HR2:AP2114HA-3.3TRG1_1A;SOT223 VR1
@@
 	1    0    0    -1
 $EndComp
-Connection ~ 7800 4300
+Connection ~ 7800 4400
 Wire Wire Line
 	8200 3100 8200 3200
@@
 Wire Wire Line
 	6150 4850 6150 4750
-Connection ~ 6150 4300
-Wire Wire Line
-	6150 4300 7800 4300
+Connection ~ 6150 4400
+Wire Wire Line
+	6150 4400 7800 4400
 Wire Wire Line
 	6300 4750 6150 4750
 Connection ~ 6150 4750
 Wire Wire Line
-	6150 4750 6150 4300
+	6150 4750 6150 4400
 Wire Wire Line
 	7800 4900 7800 4750
@@
 Text Label 8750 3200 2    50   ~ 0
 9V
-Text Label 8750 4300 2    50   ~ 0
+Text Label 8750 4400 2    50   ~ 0
 5V
 Text Label 8750 6000 2    50   ~ 0
@@
 L HR2:POWER_PFET_GSD Q2
 U 1 1 5F56BDDA
-P 3100 4300
-F 0 "Q2" H 3350 4450 50  0000 C CNN
-F 1 "PFET_6A_GSD;SOT23" H 4050 4450 50  0000 C CNN
-F 2 "HR2:" H 3300 4350 60  0001 L CNN
-F 3 "Power PFG (GSD pinout)" H 3300 4150 60  0001 L CNN
-F 4 "Power PFG (GSD pinout)" H 3300 4250 60  0001 L CNN "manf#"
-F 5 "Power PFET (GSD pinout)" H 3300 4050 60  0001 L CNN "Field5"
-	1    3100 4300
-	1    0    0    -1
-$EndComp
-Wire Wire Line
-	3100 4300 2950 4300
+P 3300 4300
+F 0 "Q2" H 3550 4450 50  0000 C CNN
+F 1 "PFET_6A_GSD;SOT23" H 3650 4050 50  0000 C CNN
+F 2 "HR2:" H 3500 4350 60  0001 L CNN
+F 3 "Power PFG (GSD pinout)" H 3500 4150 60  0001 L CNN
+F 4 "Power PFG (GSD pinout)" H 3500 4250 60  0001 L CNN "manf#"
+F 5 "Power PFET (GSD pinout)" H 3500 4050 60  0001 L CNN "Field5"
+	1    3300 4300
+	1    0    0    -1
+$EndComp
+Wire Wire Line
+	3300 4300 2950 4300
 Wire Wire Line
 	2950 4300 2950 3300
 Wire Wire Line
-	4100 4300 4200 4300
-Wire Wire Line
-	7800 4300 8750 4300
+	4100 4400 4200 4400
+Wire Wire Line
+	7800 4400 8750 4400
 Text Notes 3000 3900 0    50   ~ 0
 Note: The PFET's in the KiCAD library have passive pins\n  for design rule checks.  A PFET with Power In on the\n  Source and Power Out on the Drain is needed.\n  It was easier to do an ugly box than a pretty PFET.\n  Deal with it.
@@
 Text Label 8750 2400 2    50   ~ 0
 P5V
+Wire Wire Line
+	3300 4400 3200 4400
+Wire Wire Line
+	3200 4400 3200 4650
+Wire Wire Line
+	3200 4650 3600 4650
+Wire Wire Line
+	3600 4650 3600 4900
 $EndSCHEMATC

Commit message: Wrapped up SBC sheet.
Parts:
- SW1: value PTS645SK50SMTR92 LFS;6x9.5 -> PUSH_BUTTON;6x6x9.5H
Changed lines of the file:
@@
 P 4500 5200
 F 0 "SW1" H 4350 5300 50  0000 C CNN
-F 1 "PTS645SK50SMTR92 LFS;6x9.5" H 4150 5150 50  0000 C CNN
+F 1 "PUSH_BUTTON;6x6x9.5H" H 4300 5150 50  0000 C CNN
 F 2 "" H 4500 5400 50  0001 C CNN
 F 3 "~" H 4500 5400 50  0001 C CNN

Commit message: Schematic is basically complete.
Other:
- note added: "3.3V for miscellanious\ndevices that need it."
- note added: "9V for Motors and WOWBus\ngenerated by Pololu Boost regulator."
- note added: "Note: When the motors are running full bore\n up a hill, the current drain becomes significant.\n Use two USB connectors to maximize current\n from the USB battery pack."
- note added: "Note:\n1. The capacitor is a radial through hole electrolytic with a diameter\n of 10mm and lead pitch of 5mm. The capacitance is 1000µF at 16V.\n2. The ideal diode should keep the 5V rail clean while the P5V rail\n gets abused.\n"
- note added: "P5V is a "dirty" 5 volt supply used\nfor lighting LED's etc."
- note added: "Power On LED"
- note removed: "Note: When the motors are running full bore\n up a hill, the current drain becomes significant.\n Use to two USB connectors to maximize current\n from the USB battery pack."
- note removed: "Note:\n1. The LED's are controlled by a 16-bit shift regester that is\n filled using an SPI controller. The 3.3V outputs are fed into\n FET's that drive the LED's.\n"
- note removed: "Note:\n1. The capacitor is a radial through hole electrolytic with a diameter\n of 10mm and lead pitch of 5mm. The capacitance is 1000µF at 16V.\n2. The ideal diode should prevent accidental change...\n"
Changed lines of the file:
@@
 	1    0    0    -1
 $EndComp
-Text Notes 2000 6600 0    50   ~ 0
-Note: Power On/Off circuit is from David  Jones EEVBlog #262
+Text Notes 2800 3200 0    50   ~ 0
+Note: Power On/Off circuit is from David Jones EEVBlog #262
 $Comp
 L Device:Q_NPN_BEC Q1
@@
 Connection ~ 2950 3300
 Text Notes 950  3000 0    50   ~ 0
-Note: When the motors are running full bore\n  up a hill, the current drain becomes significant.\n  Use to two USB connectors to maximize current\n  from the USB battery pack.
-Text Notes 3250 1850 0    50   ~ 0
-Note:\n1. The LED's are controlled by a 16-bit shift regester that is\n   filled using an SPI controller.  The 3.3V outputs are fed into\n   FET's that drive the LED's.\n
+Note: When the motors are running full bore\n  up a hill, the current drain becomes significant.\n  Use two USB connectors to maximize current\n  from the USB battery pack.
 $Comp
 L Device:CP1 C?
@@
 	7800 2300 7800 1900
 Text Notes 5900 1650 0    50   ~ 0
-Note:\n1. The capacitor is a radial through hole electrolytic with a diameter\n    of 10mm and lead pitch of 5mm.  The capacitance is 1000µF at 16V.\n2. The ideal diode should prevent accidental change...\n
+Note:\n1. The capacitor is a radial through hole electrolytic with a diameter\n   of 10mm and lead pitch of 5mm.  The capacitance is 1000µF at 16V.\n2. The ideal diode should keep the 5V rail clean while the P5V rail\n   gets abused.\n
 Text Label 8750 2400 2    50   ~ 0
 P5V
@@
 Wire Wire Line
 	3600 4650 3600 4900
+Text Notes 5550 3550 0    50   ~ 0
+9V for Motors and WOWBus\ngenerated by Pololu Boost regulator.
+Text Notes 8750 2650 0    50   ~ 0
+P5V is a "dirty" 5 volt supply used\nfor lighting LED's etc.
+Text Notes 8600 5000 0    50   ~ 0
+3.3V for miscellanious\ndevices that need it.
+Text Notes 8450 5450 0    50   ~ 0
+Power On LED
 $EndSCHEMATC

Commit message: Fixed corruption of order1.lib file.
Parts:
- Q2: value PFET_6A_GSD;SOT23 -> POWER_PFET_GSD; footprint HR2: -> HR2:POWER_PFET_GSD; manf# Power PFG (GSD pinout) -> (none)
Changed lines of the file:
@@
 U 1 1 5F4D49AE
 P 6150 5000
-F 0 "C4" H 6000 5100 50  0000 L CNN
+F 0 "C4" H 6200 5100 50  0000 L CNN
 F 1 "4.7µF;1608" H 5700 4900 50  0000 L CNN
 F 2 "" H 6188 4850 50  0001 C CNN
@@
 U 1 1 5F4F1B8B
 P 8400 3450
-F 0 "C7" H 8515 3496 50  0000 L CNN
+F 0 "C7" H 8450 3550 50  0000 L CNN
 F 1 "470µF,25V;D8_P3.5" H 8450 3300 50  0000 L CNN
 F 2 "" H 8400 3450 50  0001 C CNN
@@
 U 1 1 5F50C5A8
 P 8200 3950
-F 0 "C6" H 8315 3996 50  0000 L CNN
+F 0 "C6" H 8250 4050 50  0000 L CNN
 F 1 "470µF,25V;D8_P3.5" H 8250 3800 50  0000 L CNN
 F 2 "" H 8200 3950 50  0001 C CNN
@@
 Wire Wire Line
 	8300 6000 8000 6000
-$Comp
-L HR2:POWER_PFET_GSD Q2
-U 1 1 5F56BDDA
-P 3300 4300
-F 0 "Q2" H 3550 4450 50  0000 C CNN
-F 1 "PFET_6A_GSD;SOT23" H 3650 4050 50  0000 C CNN
-F 2 "HR2:" H 3500 4350 60  0001 L CNN
-F 3 "Power PFG (GSD pinout)" H 3500 4150 60  0001 L CNN
-F 4 "Power PFG (GSD pinout)" H 3500 4250 60  0001 L CNN "manf#"
-F 5 "Power PFET (GSD pinout)" H 3500 4050 60  0001 L CNN "Field5"
-	1    3300 4300
-	1    0    0    -1
-$EndComp
 Wire Wire Line
 	3300 4300 2950 4300
@@
 Text Notes 3000 3900 0    50   ~ 0
 Note: The PFET's in the KiCAD library have passive pins\n  for design rule checks.  A PFET with Power In on the\n  Source and Power Out on the Drain is needed.\n  It was easier to do an ugly box than a pretty PFET.\n  Deal with it.
+Wire Wire Line
+	2400 3700 2500 3700
+Wire Wire Line
+	2500 3700 2500 3800
+Wire Wire Line
+	2500 5000 2000 5000
+Connection ~ 2000 5000
+Wire Wire Line
+	2400 3800 2500 3800
+Connection ~ 2500 3800
+Wire Wire Line
+	2500 3800 2500 5000
+Wire Wire Line
+	2400 3300 2950 3300
+Connection ~ 2950 3300
+Text Notes 950  3000 0    50   ~ 0
+Note: When the motors are running full bore\n  up a hill, the current drain becomes significant.\n  Use two USB connectors to maximize current\n  from the USB battery pack.
+$Comp
+L Device:CP1 C?
+U 1 1 5F7AF36B
+P 8200 2700
+AR Path="/5FA4A874/5F7AF36B" Ref="C?"  Part="1"
+AR Path="/5F52F39E/5F7AF36B" Ref="C13"  Part="1"
+F 0 "C13" H 8250 2800 50  0000 L CNN
+F 1 "1000µF@16V;D10P5" H 8250 2600 50  0000 L CNN
+F 2 "" H 8200 2700 50  0001 C CNN
+F 3 "~" H 8200 2700 50  0001 C CNN
+	1    8200 2700
+	1    0    0    -1
+$EndComp
+$Comp
+L HR2:LM66100;SOT363 U4
+U 1 1 5F7B1947
+P 6800 1900
+F 0 "U4" H 7050 2050 60  0000 C CNN
+F 1 "LM66100;SOT363" H 7150 1250 60  0000 C CNN
+F 2 "Package_TO_SOT_SMD:SOT363_SC-70-6" H 7000 1950 60  0001 L CNN
+F 3 "1.5A Ideal Diode" H 7000 1750 60  0001 L CNN
+F 4 "1.5A Ideal Diod" H 7000 1650 60  0001 L CNN "Field5"
+	1    6800 1900
+	1    0    0    -1
+$EndComp
+Wire Wire Line
+	7500 2000 8000 2000
+Wire Wire Line
+	8000 2000 8000 2950
+Connection ~ 8000 3300
+Wire Wire Line
+	7800 3500 7800 2300
+Wire Wire Line
+	7800 1900 7500 1900
+Connection ~ 7800 3500
+Wire Wire Line
+	7500 2400 7600 2400
+Wire Wire Line
+	8200 2400 8200 2550
+Wire Wire Line
+	8200 2850 8200 2950
+Wire Wire Line
+	8200 2950 8000 2950
+Connection ~ 8000 2950
+Wire Wire Line
+	8000 2950 8000 3300
+Text HLabel 8750 2400 2    50   Output ~ 0
+P5V
+Wire Wire Line
+	8200 2400 8750 2400
+Connection ~ 8200 2400
+Wire Wire Line
+	7500 2100 7600 2100
+Wire Wire Line
+	7600 2100 7600 2400
+Connection ~ 7600 2400
+Wire Wire Line
+	7600 2400 8200 2400
+Wire Wire Line
+	7500 2300 7800 2300
+Connection ~ 7800 2300
+Wire Wire Line
+	7800 2300 7800 1900
+Text Notes 5900 1650 0    50   ~ 0
+Note:\n1. The capacitor is a radial through hole electrolytic with a diameter\n   of 10mm and lead pitch of 5mm.  The capacitance is 1000µF at 16V.\n2. The ideal diode should keep the 5V rail clean while the P5V rail\n   gets abused.\n
+Text Label 8750 2400 2    50   ~ 0
+P5V
+Wire Wire Line
+	3300 4400 3200 4400
+Wire Wire Line
+	3200 4400 3200 4650
+Wire Wire Line
+	3200 4650 3600 4650
+Wire Wire Line
+	3600 4650 3600 4900
+Text Notes 5550 3550 0    50   ~ 0
+9V for Motors and WOWBus\ngenerated by Pololu Boost regulator.
+Text Notes 8750 2650 0    50   ~ 0
+P5V is a "dirty" 5 volt supply used\nfor lighting LED's etc.
+Text Notes 8600 5000 0    50   ~ 0
+3.3V for miscellanious\ndevices that need it.
+Text Notes 8450 5450 0    50   ~ 0
+Power On LED
 $Comp
 L HR2:USB_B_MINI_POWER_SLAVE CN2
@@
 	1    0    0    -1
 $EndComp
-Wire Wire Line
-	2400 3700 2500 3700
-Wire Wire Line
-	2500 3700 2500 3800
-Wire Wire Line
-	2500 5000 2000 5000
-Connection ~ 2000 5000
-Wire Wire Line
-	2400 3800 2500 3800
-Connection ~ 2500 3800
-Wire Wire Line
-	2500 3800 2500 5000
-Wire Wire Line
-	2400 3300 2950 3300
-Connection ~ 2950 3300
-Text Notes 950  3000 0    50   ~ 0
-Note: When the motors are running full bore\n  up a hill, the current drain becomes significant.\n  Use two USB connectors to maximize current\n  from the USB battery pack.
-$Comp
-L Device:CP1 C?
-U 1 1 5F7AF36B
-P 8200 2700
-AR Path="/5FA4A874/5F7AF36B" Ref="C?"  Part="1"
-AR Path="/5F52F39E/5F7AF36B" Ref="C13"  Part="1"
-F 0 "C13" H 8300 2800 50  0000 L CNN
-F 1 "1000µF@16V;D10P5" H 8250 2600 50  0000 L CNN
-F 2 "" H 8200 2700 50  0001 C CNN
-F 3 "~" H 8200 2700 50  0001 C CNN
-	1    8200 2700
-	1    0    0    -1
-$EndComp
-$Comp
-L HR2:LM66100;SOT363 U4
-U 1 1 5F7B1947
-P 6800 1900
-F 0 "U4" H 7050 2050 60  0000 C CNN
-F 1 "LM66100;SOT363" H 7150 1250 60  0000 C CNN
-F 2 "Package_TO_SOT_SMD:SOT363_SC-70-6" H 7000 1950 60  0001 L CNN
-F 3 "1.5A Ideal Diode" H 7000 1750 60  0001 L CNN
-F 4 "1.5A Ideal Diod" H 7000 1650 60  0001 L CNN "Field5"
-	1    6800 1900
-	1    0    0    -1
-$EndComp
-Wire Wire Line
-	7500 2000 8000 2000
-Wire Wire Line
-	8000 2000 8000 2950
-Connection ~ 8000 3300
-Wire Wire Line
-	7800 3500 7800 2300
-Wire Wire Line
-	7800 1900 7500 1900
-Connection ~ 7800 3500
-Wire Wire Line
-	7500 2400 7600 2400
-Wire Wire Line
-	8200 2400 8200 2550
-Wire Wire Line
-	8200 2850 8200 2950
-Wire Wire Line
-	8200 2950 8000 2950
-Connection ~ 8000 2950
-Wire Wire Line
-	8000 2950 8000 3300
-Text HLabel 8750 2400 2    50   Output ~ 0
-P5V
-Wire Wire Line
-	8200 2400 8750 2400
-Connection ~ 8200 2400
-Wire Wire Line
-	7500 2100 7600 2100
-Wire Wire Line
-	7600 2100 7600 2400
-Connection ~ 7600 2400
-Wire Wire Line
-	7600 2400 8200 2400
-Wire Wire Line
-	7500 2300 7800 2300
-Connection ~ 7800 2300
-Wire Wire Line
-	7800 2300 7800 1900
-Text Notes 5900 1650 0    50   ~ 0
-Note:\n1. The capacitor is a radial through hole electrolytic with a diameter\n   of 10mm and lead pitch of 5mm.  The capacitance is 1000µF at 16V.\n2. The ideal diode should keep the 5V rail clean while the P5V rail\n   gets abused.\n
-Text Label 8750 2400 2    50   ~ 0
-P5V
-Wire Wire Line
-	3300 4400 3200 4400
-Wire Wire Line
-	3200 4400 3200 4650
-Wire Wire Line
-	3200 4650 3600 4650
-Wire Wire Line
-	3600 4650 3600 4900
-Text Notes 5550 3550 0    50   ~ 0
-9V for Motors and WOWBus\ngenerated by Pololu Boost regulator.
-Text Notes 8750 2650 0    50   ~ 0
-P5V is a "dirty" 5 volt supply used\nfor lighting LED's etc.
-Text Notes 8600 5000 0    50   ~ 0
-3.3V for miscellanious\ndevices that need it.
-Text Notes 8450 5450 0    50   ~ 0
-Power On LED
+$Comp
+L HR2:POWER_PFET_GSD Q2
+U 1 1 5F96763E
+P 3300 4300
+F 0 "Q2" H 3700 4590 60  0000 C CNN
+F 1 "POWER_PFET_GSD" H 3700 4484 60  0000 C CNN
+F 2 "HR2:POWER_PFET_GSD" H 3500 4350 60  0001 L CNN
+F 3 "Power PFG (GSD pinout)" H 3500 4150 60  0001 L CNN
+F 4 "Power PFET (GSD pinout)" H 3500 4050 60  0001 L CNN "Field5"
+	1    3300 4300
+	1    0    0    -1
+$EndComp
 $EndSCHEMATC

Commit message: Reannoted. Postioned components are in the 80-99 reference range.
Parts:
- renumbered C4 to C2, C5 to C3, C13 to C4, C6 to C5, C7 to C6, CN2 to CN1, CN1 to CN2, CN42 to CN93, R13 to R5, U4 to U1
Changed lines of the file:
@@
 Connection ~ 4800 5500
 $Comp
-L Connector:USB_B_Mini CN1
+L Connector:USB_B_Mini CN2
 U 1 1 5F4B0748
 P 2000 4500
-F 0 "CN1" H 1900 4850 50  0000 C CNN
+F 0 "CN2" H 1900 4850 50  0000 C CNN
 F 1 "AMP10103594-0001LF;USB1x6H" H 1200 4150 50  0000 C CNN
 F 2 "" H 2150 4450 50  0001 C CNN
@@
 P 6800 3900
 AR Path="/5F5303B1" Ref="CN?"  Part="1"
-AR Path="/5F52F39E/5F5303B1" Ref="CN42"  Part="1"
-F 0 "CN42" H 7100 2950 50  0000 C CNN
+AR Path="/5F52F39E/5F5303B1" Ref="CN93"  Part="1"
+F 0 "CN93" H 7100 2950 50  0000 C CNN
 F 1 "POLOLU_U3V70F9;F1x4+F1x5" H 7200 4050 50  0000 C CNN
 F 2 "HR2:U3V70xMATE_F1x4+F1x5" H 7000 3950 60  0001 L CNN
@@
 	8000 3700 8000 3400
 $Comp
-L Device:C C4
+L Device:C C2
 U 1 1 5F4D49AE
 P 6150 5000
-F 0 "C4" H 6200 5100 50  0000 L CNN
+F 0 "C2" H 6200 5100 50  0000 L CNN
 F 1 "4.7µF;1608" H 5700 4900 50  0000 L CNN
 F 2 "" H 6188 4850 50  0001 C CNN
@@
 $EndComp
 $Comp
-L Device:C C5
+L Device:C C3
 U 1 1 5F4D53A8
 P 7800 5050
-F 0 "C5" H 7650 5150 50  0000 L CNN
+F 0 "C3" H 7650 5150 50  0000 L CNN
 F 1 "4.7µF;1608" H 7350 4950 50  0000 L CNN
 F 2 "" H 7838 4900 50  0001 C CNN
@@
 USB5V
 $Comp
-L Device:CP1 C7
+L Device:CP1 C6
 U 1 1 5F4F1B8B
 P 8400 3450
-F 0 "C7" H 8450 3550 50  0000 L CNN
+F 0 "C6" H 8450 3550 50  0000 L CNN
 F 1 "470µF,25V;D8_P3.5" H 8450 3300 50  0000 L CNN
 F 2 "" H 8400 3450 50  0001 C CNN
@@
 Connection ~ 8200 3200
 $Comp
-L Device:CP1 C6
+L Device:CP1 C5
 U 1 1 5F50C5A8
 P 8200 3950
-F 0 "C6" H 8250 4050 50  0000 L CNN
+F 0 "C5" H 8250 4050 50  0000 L CNN
 F 1 "470µF,25V;D8_P3.5" H 8250 3800 50  0000 L CNN
 F 2 "" H 8200 3950 50  0001 C CNN
@@
 Connection ~ 8400 3200
 $Comp
-L Device:R_US R13
+L Device:R_US R5
 U 1 1 5F4D39A5
 P 8300 5100
-F 0 "R13" H 8150 5200 50  0000 L CNN
+F 0 "R5" H 8150 5200 50  0000 L CNN
 F 1 "470Ω;1608" H 8350 5000 50  0000 L CNN
 F 2 "" V 8340 5090 50  0001 C CNN
@@
 P 8200 2700
 AR Path="/5FA4A874/5F7AF36B" Ref="C?"  Part="1"
-AR Path="/5F52F39E/5F7AF36B" Ref="C13"  Part="1"
-F 0 "C13" H 8250 2800 50  0000 L CNN
+AR Path="/5F52F39E/5F7AF36B" Ref="C4"  Part="1"
+F 0 "C4" H 8250 2800 50  0000 L CNN
 F 1 "1000µF@16V;D10P5" H 8250 2600 50  0000 L CNN
 F 2 "" H 8200 2700 50  0001 C CNN
@@
 $EndComp
 $Comp
-L HR2:LM66100;SOT363 U4
+L HR2:LM66100;SOT363 U1
 U 1 1 5F7B1947
 P 6800 1900
-F 0 "U4" H 7050 2050 60  0000 C CNN
+F 0 "U1" H 7050 2050 60  0000 C CNN
 F 1 "LM66100;SOT363" H 7150 1250 60  0000 C CNN
 F 2 "Package_TO_SOT_SMD:SOT363_SC-70-6" H 7000 1950 60  0001 L CNN
@@
 Power On LED
 $Comp
-L HR2:USB_B_MINI_POWER_SLAVE CN2
+L HR2:USB_B_MINI_POWER_SLAVE CN1
 U 1 1 5F56C48C
 P 1600 3300
-F 0 "CN2" H 1850 3450 50  0000 C CNN
+F 0 "CN1" H 1850 3450 50  0000 C CNN
 F 1 "AMP10103594-0001LF;USB1x6H" H 1200 2650 50  0000 C CNN
 F 2 "Connector:USB_B_Mini" H 1800 3350 60  0001 L CNN

Commit message: Assigned PCB footprints.
Parts:
- C1, C2, C3: footprint (none) -> Capacitor_SMD:C_0603_1608Metric
- C4: footprint (none) -> Capacitor_THT:CP_Radial_D10.0mm_P3.50mm
- C5, C6: footprint (none) -> Capacitor_THT:CP_Radial_D8.0mm_P3.50mm
- CN1: footprint Connector:USB_B_Mini -> Connector_USB:USB_Micro-B_Amphenol_10103594-0001LF_Horizontal
- CN2: footprint (none) -> Connector_USB:USB_Micro-B_Amphenol_10103594-0001LF_Horizontal
- D1: footprint (none) -> LED_SMD:LED_0603_1608Metric
- Q1, Q3: footprint (none) -> Package_TO_SOT_SMD:SOT-23
- Q2: footprint HR2:POWER_PFET_GSD -> Package_TO_SOT_SMD:SOT-23
- R1, R2, R3, R4, R5: footprint (none) -> Resistor_SMD:R_0603_1608Metric
- SW1: footprint (none) -> Button_Switch_SMD:SW_SPST_PTS645
Changed lines of the file:
@@
 F 0 "R1" H 2800 4750 50  0000 L CNN
 F 1 "100KΩ;1608" H 3000 4550 50  0000 L CNN
-F 2 "" V 2990 4640 50  0001 C CNN
+F 2 "Resistor_SMD:R_0603_1608Metric" V 2990 4640 50  0001 C CNN
 F 3 "~" H 2950 4650 50  0001 C CNN
 	1    2950 4650
@@
 F 0 "Q1" H 2950 5350 50  0000 L CNN
 F 1 "2N2222;SOT23" H 2500 5050 50  0000 L CNN
-F 2 "" H 3250 5300 50  0001 C CNN
+F 2 "Package_TO_SOT_SMD:SOT-23" H 3250 5300 50  0001 C CNN
 F 3 "~" H 3050 5200 50  0001 C CNN
 	1    3050 5200
@@
 F 0 "Q3" H 5390 5546 50  0000 L CNN
 F 1 "2N2222;SOT23" H 5390 5455 50  0000 L CNN
-F 2 "" H 5400 5600 50  0001 C CNN
+F 2 "Package_TO_SOT_SMD:SOT-23" H 5400 5600 50  0001 C CNN
 F 3 "~" H 5200 5500 50  0001 C CNN
 	1    5200 5500
@@
 F 0 "R2" H 4050 4850 50  0000 L CNN
 F 1 "100KΩ;1608" H 4250 4650 50  0000 L CNN
-F 2 "" V 4240 4740 50  0001 C CNN
+F 2 "Resistor_SMD:R_0603_1608Metric" V 4240 4740 50  0001 C CNN
 F 3 "~" H 4200 4750 50  0001 C CNN
 	1    4200 4750
@@
 F 0 "R4" H 5150 4850 50  0000 L CNN
 F 1 "100KΩ;1608" H 5350 4650 50  0000 L CNN
-F 2 "" V 5340 4740 50  0001 C CNN
+F 2 "Resistor_SMD:R_0603_1608Metric" V 5340 4740 50  0001 C CNN
 F 3 "~" H 5300 4750 50  0001 C CNN
 	1    5300 4750
@@
 F 0 "R3" H 4650 4850 50  0000 L CNN
 F 1 "1MΩ;1608" H 4850 4650 50  0000 L CNN
-F 2 "" V 4840 4740 50  0001 C CNN
+F 2 "Resistor_SMD:R_0603_1608Metric" V 4840 4740 50  0001 C CNN
 F 3 "~" H 4800 4750 50  0001 C CNN
 	1    4800 4750
@@
 F 0 "SW1" H 4350 5300 50  0000 C CNN
 F 1 "PUSH_BUTTON;6x6x9.5H" H 4300 5150 50  0000 C CNN
-F 2 "" H 4500 5400 50  0001 C CNN
+F 2 "Button_Switch_SMD:SW_SPST_PTS645" H 4500 5400 50  0001 C CNN
 F 3 "~" H 4500 5400 50  0001 C CNN
 	1    4500 5200
@@
 F 0 "C1" H 4650 5850 50  0000 L CNN
 F 1 "22µF;1608" H 4850 5650 50  0000 L CNN
-F 2 "" H 4838 5600 50  0001 C CNN
+F 2 "Capacitor_SMD:C_0603_1608Metric" H 4838 5600 50  0001 C CNN
 F 3 "~" H 4800 5750 50  0001 C CNN
 	1    4800 5750
@@
 F 0 "CN2" H 1900 4850 50  0000 C CNN
 F 1 "AMP10103594-0001LF;USB1x6H" H 1200 4150 50  0000 C CNN
-F 2 "" H 2150 4450 50  0001 C CNN
+F 2 "Connector_USB:USB_Micro-B_Amphenol_10103594-0001LF_Horizontal" H 2150 4450 50  0001 C CNN
 F 3 "~" H 2150 4450 50  0001 C CNN
 	1    2000 4500
@@
 F 0 "C2" H 6200 5100 50  0000 L CNN
 F 1 "4.7µF;1608" H 5700 4900 50  0000 L CNN
-F 2 "" H 6188 4850 50  0001 C CNN
+F 2 "Capacitor_SMD:C_0603_1608Metric" H 6188 4850 50  0001 C CNN
 F 3 "~" H 6150 5000 50  0001 C CNN
 	1    6150 5000
@@
 F 0 "C3" H 7650 5150 50  0000 L CNN
 F 1 "4.7µF;1608" H 7350 4950 50  0000 L CNN
-F 2 "" H 7838 4900 50  0001 C CNN
+F 2 "Capacitor_SMD:C_0603_1608Metric" H 7838 4900 50  0001 C CNN
 F 3 "~" H 7800 5050 50  0001 C CNN
 	1    7800 5050
@@
 F 0 "C6" H 8450 3550 50  0000 L CNN
 F 1 "470µF,25V;D8_P3.5" H 8450 3300 50  0000 L CNN
-F 2 "" H 8400 3450 50  0001 C CNN
+F 2 "Capacitor_THT:CP_Radial_D8.0mm_P3.50mm" H 8400 3450 50  0001 C CNN
 F 3 "~" H 8400 3450 50  0001 C CNN
 	1    8400 3450
@@
 F 0 "C5" H 8250 4050 50  0000 L CNN
 F 1 "470µF,25V;D8_P3.5" H 8250 3800 50  0000 L CNN
-F 2 "" H 8200 3950 50  0001 C CNN
+F 2 "Capacitor_THT:CP_Radial_D8.0mm_P3.50mm" H 8200 3950 50  0001 C CNN
 F 3 "~" H 8200 3950 50  0001 C CNN
 	1    8200 3950
@@
 F 0 "R5" H 8150 5200 50  0000 L CNN
 F 1 "470Ω;1608" H 8350 5000 50  0000 L CNN
-F 2 "" V 8340 5090 50  0001 C CNN
+F 2 "Resistor_SMD:R_0603_1608Metric" V 8340 5090 50  0001 C CNN
 F 3 "~" H 8300 5100 50  0001 C CNN
 	1    8300 5100
@@
 F 0 "D1" V 8400 5700 50  0000 R CNN
 F 1 "LEDGRN;1608" V 8300 5500 50  0000 R CNN
-F 2 "" H 8300 5600 50  0001 C CNN
+F 2 "LED_SMD:LED_0603_1608Metric" H 8300 5600 50  0001 C CNN
 F 3 "~" H 8300 5600 50  0001 C CNN
 	1    8300 5600
@@
 F 0 "C4" H 8250 2800 50  0000 L CNN
 F 1 "1000µF@16V;D10P5" H 8250 2600 50  0000 L CNN
-F 2 "" H 8200 2700 50  0001 C CNN
+F 2 "Capacitor_THT:CP_Radial_D10.0mm_P3.50mm" H 8200 2700 50  0001 C CNN
 F 3 "~" H 8200 2700 50  0001 C CNN
 	1    8200 2700
@@
 F 0 "CN1" H 1850 3450 50  0000 C CNN
 F 1 "AMP10103594-0001LF;USB1x6H" H 1200 2650 50  0000 C CNN
-F 2 "Connector:USB_B_Mini" H 1800 3350 60  0001 L CNN
+F 2 "Connector_USB:USB_Micro-B_Amphenol_10103594-0001LF_Horizontal" H 1800 3350 60  0001 L CNN
 F 3 "USB_Mini Power (Slave)" H 1800 3150 60  0001 L CNN
 F 4 "USB_Mini Power (Slave)" H 1800 3050 60  0001 L CNN "Field5"
@@
 F 0 "Q2" H 3700 4590 60  0000 C CNN
 F 1 "POWER_PFET_GSD" H 3700 4484 60  0000 C CNN
-F 2 "HR2:POWER_PFET_GSD" H 3500 4350 60  0001 L CNN
+F 2 "Package_TO_SOT_SMD:SOT-23" H 3500 4350 60  0001 L CNN
 F 3 "Power PFG (GSD pinout)" H 3500 4150 60  0001 L CNN
 F 4 "Power PFET (GSD pinout)" H 3500 4050 60  0001 L CNN "Field5"
