File: electrical/master_board/rev_a/power.sch (KiCad schematic (older format))
At the start: 21 parts, among them CN1 AMP10103594-0001LF;USB1x6H, CN2 AMP10103594-0001LF;USB1x6H, CN93 POLOLU_U3V70F9;F1x4+F1x5, Q1 2N2222;SOT23, Q2 POWER_PFET_GSD, Q3 2N2222;SOT23, SW1 PUSH_BUTTON;6x6x9.5H, U1 LM66100;SOT363

Commit message: Imported footprints to PCB.
Parts:
- U1: footprint Package_TO_SOT_SMD:SOT363_SC-70-6 -> Package_TO_SOT_SMD:SOT-363_SC-70-6
- VR1: footprint Package_TO_SOT_SMD:SOT_223-3_TabPin2 -> Package_TO_SOT_SMD:SOT-223-3_TabPin2
Changed lines of the file:
@@
 F 0 "VR1" H 6550 4900 50  0000 C CNN
 F 1 "AP2114HA-3.3TRG1_1A;SOT223" H 7350 4900 50  0000 C CNN
-F 2 "Package_TO_SOT_SMD:SOT_223-3_TabPin2" H 6500 4800 60  0001 L CNN
+F 2 "Package_TO_SOT_SMD:SOT-223-3_TabPin2" H 6500 4800 60  0001 L CNN
 F 3 "1A 3.3V LDO Voltage Linear Regulator" H 6500 4600 60  0001 L CNN
 F 4 "1A 3.3V LDO Voltage Linear Regulator" H 6500 4500 60  0001 L CNN "Field5"
@@
 F 0 "U1" H 7050 2050 60  0000 C CNN
 F 1 "LM66100;SOT363" H 7150 1250 60  0000 C CNN
-F 2 "Package_TO_SOT_SMD:SOT363_SC-70-6" H 7000 1950 60  0001 L CNN
+F 2 "Package_TO_SOT_SMD:SOT-363_SC-70-6" H 7000 1950 60  0001 L CNN
 F 3 "1.5A Ideal Diode" H 7000 1750 60  0001 L CNN
 F 4 "1.5A Ideal Diod" H 7000 1650 60  0001 L CNN "Field5"

Commit message: Changing footprints and moving things around on the PCB.
Parts:
- removed CN1: AMP10103594-0001LF;USB1x6H, Connector_USB:USB_Micro-B_Amphenol_10103594-0001LF_Horizontal, symbol HR2:USB_B_MINI_POWER_SLAVE
- removed CN2: AMP10103594-0001LF;USB1x6H, Connector_USB:USB_Micro-B_Amphenol_10103594-0001LF_Horizontal, symbol Connector:USB_B_Mini
- added CN1: USB3140-30-230-1-C;VERT,2.3FLANGE, HR2:USB3140-30-230-1-C;VERT,2.3FLANGE, symbol HR2:USB_B_MICRO_POWER_SLAVE
- added CN2: USB3140-30-230-1-C;VERT,2.3FLANGE, HR2:USB3140-30-230-1-C;VERT,2.3FLANGE, symbol HR2:USB_B_MICRO_POWER_MASTER
- C4: value 1000µF@16V;D10P5 -> 1000µF@10Vmin;D10P5H13max; footprint Capacitor_THT:CP_Radial_D10.0mm_P3.50mm -> Capacitor_THT:CP_Radial_D10.0mm_P5.00mm
- C5, C6: value 470µF,25V;D8_P3.5 -> 470µF,25Vmin;D10P5H13max; footprint Capacitor_THT:CP_Radial_D8.0mm_P3.50mm -> Capacitor_THT:CP_Radial_D10.0mm_P5.00mm
- SW1: value PUSH_BUTTON;6x6x9.5H -> BUTTON;6x3.5; footprint Button_Switch_SMD:SW_SPST_PTS645 -> HR2:BUTTON_6x3.5
Connections:
- wire segments 103 -> 102
- no-connect marks 4 -> 1
Changed lines of the file:
@@
 P 4500 5200
 F 0 "SW1" H 4350 5300 50  0000 C CNN
-F 1 "PUSH_BUTTON;6x6x9.5H" H 4300 5150 50  0000 C CNN
-F 2 "Button_Switch_SMD:SW_SPST_PTS645" H 4500 5400 50  0001 C CNN
+F 1 "BUTTON;6x3.5" H 4450 5100 50  0000 C CNN
+F 2 "HR2:BUTTON_6x3.5" H 4500 5400 50  0001 C CNN
 F 3 "~" H 4500 5400 50  0001 C CNN
 	1    4500 5200
@@
 	4800 5600 4800 5500
 Connection ~ 4800 5500
-$Comp
-L Connector:USB_B_Mini CN2
-U 1 1 5F4B0748
-P 2000 4500
-F 0 "CN2" H 1900 4850 50  0000 C CNN
-F 1 "AMP10103594-0001LF;USB1x6H" H 1200 4150 50  0000 C CNN
-F 2 "Connector_USB:USB_Micro-B_Amphenol_10103594-0001LF_Horizontal" H 2150 4450 50  0001 C CNN
-F 3 "~" H 2150 4450 50  0001 C CNN
-	1    2000 4500
-	1    0    0    -1
-$EndComp
 Wire Wire Line
 	2300 4300 2950 4300
-NoConn ~ 2300 4500
-NoConn ~ 2300 4600
-NoConn ~ 2300 4700
-Wire Wire Line
-	1900 4900 1900 5000
-Wire Wire Line
-	1900 5000 2000 5000
-Wire Wire Line
-	2000 5000 2000 4900
-Wire Wire Line
-	1900 5000 1900 6000
-Wire Wire Line
-	1900 6000 2950 6000
-Connection ~ 1900 5000
 Connection ~ 2950 6000
 Wire Wire Line
@@
 P 8400 3450
 F 0 "C6" H 8450 3550 50  0000 L CNN
-F 1 "470µF,25V;D8_P3.5" H 8450 3300 50  0000 L CNN
-F 2 "Capacitor_THT:CP_Radial_D8.0mm_P3.50mm" H 8400 3450 50  0001 C CNN
+F 1 "470µF,25Vmin;D10P5H13max" H 8450 3300 50  0000 L CNN
+F 2 "Capacitor_THT:CP_Radial_D10.0mm_P5.00mm" H 8400 3450 50  0001 C CNN
 F 3 "~" H 8400 3450 50  0001 C CNN
 	1    8400 3450
@@
 P 8200 3950
 F 0 "C5" H 8250 4050 50  0000 L CNN
-F 1 "470µF,25V;D8_P3.5" H 8250 3800 50  0000 L CNN
-F 2 "Capacitor_THT:CP_Radial_D8.0mm_P3.50mm" H 8200 3950 50  0001 C CNN
+F 1 "470µF,25Vmin;D10P5H13max" H 8250 3800 50  0000 L CNN
+F 2 "Capacitor_THT:CP_Radial_D10.0mm_P5.00mm" H 8200 3950 50  0001 C CNN
 F 3 "~" H 8200 3950 50  0001 C CNN
 	1    8200 3950
@@
 Note: The PFET's in the KiCAD library have passive pins\n  for design rule checks.  A PFET with Power In on the\n  Source and Power Out on the Drain is needed.\n  It was easier to do an ugly box than a pretty PFET.\n  Deal with it.
 Wire Wire Line
-	2400 3700 2500 3700
+	2300 3700 2500 3700
 Wire Wire Line
 	2500 3700 2500 3800
 Wire Wire Line
-	2500 5000 2000 5000
-Connection ~ 2000 5000
-Wire Wire Line
-	2400 3800 2500 3800
+	2300 3800 2500 3800
 Connection ~ 2500 3800
 Wire Wire Line
-	2500 3800 2500 5000
-Wire Wire Line
-	2400 3300 2950 3300
+	2500 3800 2500 4700
+Wire Wire Line
+	2300 3300 2950 3300
 Connection ~ 2950 3300
 Text Notes 950  3000 0    50   ~ 0
@@
 AR Path="/5F52F39E/5F7AF36B" Ref="C4"  Part="1"
 F 0 "C4" H 8250 2800 50  0000 L CNN
-F 1 "1000µF@16V;D10P5" H 8250 2600 50  0000 L CNN
-F 2 "Capacitor_THT:CP_Radial_D10.0mm_P3.50mm" H 8200 2700 50  0001 C CNN
+F 1 "1000µF@10Vmin;D10P5H13max" H 8250 2600 50  0000 L CNN
+F 2 "Capacitor_THT:CP_Radial_D10.0mm_P5.00mm" H 8200 2700 50  0001 C CNN
 F 3 "~" H 8200 2700 50  0001 C CNN
 	1    8200 2700
@@
 Power On LED
 $Comp
-L HR2:USB_B_MINI_POWER_SLAVE CN1
-U 1 1 5F56C48C
-P 1600 3300
-F 0 "CN1" H 1850 3450 50  0000 C CNN
-F 1 "AMP10103594-0001LF;USB1x6H" H 1200 2650 50  0000 C CNN
-F 2 "Connector_USB:USB_Micro-B_Amphenol_10103594-0001LF_Horizontal" H 1800 3350 60  0001 L CNN
-F 3 "USB_Mini Power (Slave)" H 1800 3150 60  0001 L CNN
-F 4 "USB_Mini Power (Slave)" H 1800 3050 60  0001 L CNN "Field5"
-	1    1600 3300
-	1    0    0    -1
-$EndComp
-$Comp
 L HR2:POWER_PFET_GSD Q2
 U 1 1 5F96763E
 P 3300 4300
-F 0 "Q2" H 3700 4590 60  0000 C CNN
-F 1 "POWER_PFET_GSD" H 3700 4484 60  0000 C CNN
+F 0 "Q2" H 3550 4450 50  0000 C CNN
+F 1 "POWER_PFET_GSD" H 3700 4050 50  0000 C CNN
 F 2 "Package_TO_SOT_SMD:SOT-23" H 3500 4350 60  0001 L CNN
 F 3 "Power PFG (GSD pinout)" H 3500 4150 60  0001 L CNN
@@
 	1    0    0    -1
 $EndComp
+Wire Wire Line
+	2300 4700 2500 4700
+Wire Wire Line
+	2500 4800 2500 4700
+Connection ~ 2500 4700
+Wire Wire Line
+	2300 4800 2500 4800
+Wire Wire Line
+	2500 4800 2500 6000
+Connection ~ 2500 4800
+Wire Wire Line
+	2500 6000 2950 6000
+$Comp
+L HR2:USB_B_MICRO_POWER_SLAVE CN1
+U 1 1 5F9D0CA6
+P 1500 3300
+F 0 "CN1" H 1750 3450 50  0000 C CNN
+F 1 "USB3140-30-230-1-C;VERT,2.3FLANGE" H 1700 2650 50  0000 C CNN
+F 2 "HR2:USB3140-30-230-1-C;VERT,2.3FLANGE" H 1700 3350 60  0001 L CNN
+F 3 "2.3FLANGE" H 1700 3150 60  0001 L CNN
+F 4 "USB_Mini Power (Slave)" H 1700 3050 60  0001 L CNN "Field5"
+	1    1500 3300
+	1    0    0    -1
+$EndComp
+$Comp
+L HR2:USB_B_MICRO_POWER_MASTER CN2
+U 1 1 5F9D14A3
+P 1500 4300
+F 0 "CN2" H 1750 4450 50  0000 C CNN
+F 1 "USB3140-30-230-1-C;VERT,2.3FLANGE" H 1700 3650 50  0000 C CNN
+F 2 "HR2:USB3140-30-230-1-C;VERT,2.3FLANGE" H 1700 4350 60  0001 L CNN
+F 3 "2.3FLANGE" H 1700 4150 60  0001 L CNN
+F 4 "USB_Mini Power (Slave)" H 1700 4050 60  0001 L CNN "Field5"
+	1    1500 4300
+	1    0    0    -1
+$EndComp
