File: electrical/master_board/rev_a/power.sch (KiCad schematic (older format))
At the start: 47 parts, among them CN1 USB3140-30-230-1-C;VERT,2.3FL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, CN2 USB3140-30-230-1-C;VERT,2.3FL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, CN93 POLOLU_U3V70F9;F1x4+F1x5, Q1 2N2222;SOT23, Q2 POWER_PFET_GSD, Q3 2N2222;SOT23, SW1 BUTTON;6x3.5, U1 LM66100;SOT363

Commit message: Fixed the schematic DRC errors.
Parts:
- removed Q2: POWER_PFET_GSD, Package_TO_SOT_SMD:SOT-23, symbol HR2:POWER_PFET_GSD
- added Q2: PFET_6A;SOT23, symbol HR2_MISC:Q_PWR_PMOS_GSD
Connections:
- wire segments 183 -> 179
Changed lines of the file:
@@
 Connection ~ 2550 4400
 Wire Wire Line
-	3800 4100 3800 3900
+	3800 4100 3800 3800
 Wire Wire Line
 	2850 4700 3800 4700
@@
 Connection ~ 2550 3800
 Wire Wire Line
-	3800 3900 4400 3900
-Wire Wire Line
-	4400 3900 4400 4100
-Connection ~ 3800 3900
+	3800 3800 4400 3800
+Wire Wire Line
+	4400 3800 4400 4100
+Connection ~ 3800 3800
 Wire Wire Line
 	4300 4700 5100 4700
@@
 	2550 5500 4400 5500
 Connection ~ 4400 5500
-Connection ~ 4400 3900
+Connection ~ 4400 3800
 Wire Wire Line
 	4400 5100 4400 5000
@@
 	2600 7050 2600 7150
 Wire Wire Line
-	2900 3800 2550 3800
-Wire Wire Line
-	2550 3800 2550 2800
-Wire Wire Line
-	3700 3900 3800 3900
+	3000 3800 2550 3800
 Text Notes 2600 3400 0    50   ~ 0
 Note: The PFET's in the KiCAD library have passive pins\n  for design rule checks.  A PFET with Power In on the\n  Source and Power Out on the Drain is needed.\n  It was easier to do an ugly box than a pretty PFET.\n  Deal with it.
@@
 Text Notes 3750 1800 0    50   ~ 0
 Note:\n1. The capacitor is a radial through hole electrolytic with a diameter\n   of 10mm and lead pitch of 5mm.  The capacitance is 1000µF at 16V.\n2. The ideal diode should keep the 5V rail clean while the P5V rail\n   gets abused.\n
-Wire Wire Line
-	2900 3900 2800 3900
-Wire Wire Line
-	2800 3900 2800 4150
-Wire Wire Line
-	2800 4150 3200 4150
-Wire Wire Line
-	3200 4150 3200 4400
 Text Notes 5150 3050 0    50   ~ 0
 9V for Motors and WOWBus\ngenerated by Pololu Boost regulator.
@@
 Text Notes 6200 5000 0    50   ~ 0
 3.3V for miscellanious\ndevices that need it.
-$Comp
-L HR2:POWER_PFET_GSD Q2
-U 1 1 5F96763E
-P 2900 3800
-F 0 "Q2" H 3150 3950 50  0000 C CNN
-F 1 "POWER_PFET_GSD" H 3300 3550 50  0000 C CNN
-F 2 "Package_TO_SOT_SMD:SOT-23" H 3100 3850 60  0001 L CNN
-F 3 "Power PFG (GSD pinout)" H 3100 3650 60  0001 L CNN
-F 4 "Power PFET (GSD pinout)" H 3100 3550 60  0001 L CNN "Field5"
-	1    2900 3800
-	1    0    0    -1
-$EndComp
 Wire Wire Line
 	1900 4200 2100 4200
@@
 Wire Wire Line
 	9200 4900 9700 4900
-Wire Wire Line
-	7900 3800 7900 3900
 Connection ~ 9500 1900
 Wire Wire Line
@@
 	9400 2900 9650 2900
 Wire Wire Line
-	7500 3900 7900 3900
-Connection ~ 7500 3900
-Connection ~ 7900 3900
-Wire Wire Line
-	7900 3900 7900 4100
+	7500 3800 7900 3800
+Connection ~ 7500 3800
+Connection ~ 7900 3800
+Wire Wire Line
+	7900 3800 7900 4100
 Wire Wire Line
 	7400 4600 7900 4600
@@
 Connection ~ 7500 1800
 Wire Wire Line
-	7500 1800 7500 3900
+	7500 1800 7500 3800
 Wire Wire Line
 	7200 3000 7400 3000
@@
 	7900 2600 7900 2900
 Wire Wire Line
-	4400 3900 7500 3900
+	4400 3800 7500 3800
 Wire Wire Line
 	6000 4100 7400 4100
@@
 Wire Wire Line
 	7400 4100 7400 4300
+$Comp
+L HR2_MISC:Q_PWR_PMOS_GSD Q2
+U 1 1 5FCF4323
+P 3200 3900
+F 0 "Q2" V 3100 3800 50  0000 C CNN
+F 1 "PFET_6A;SOT23" V 3450 3900 50  0000 C CNN
+F 2 "" H 3400 4000 50  0001 C CNN
+F 3 "~" H 3200 3900 50  0001 C CNN
+	1    3200 3900
+	0    1    -1   0
+$EndComp
+Wire Wire Line
+	3400 3800 3800 3800
+Wire Wire Line
+	2550 2800 2550 3800
+Wire Wire Line
+	3200 4100 3200 4400
 $EndSCHEMATC

Commit message: Worked on Power supply.
Parts:
- removed CN1: USB3140-30-230-1-C;VERT,2.3FLANGE, HR2:USB3140-30-230-1-C;VERT,2.3FLANGE, symbol HR2:USB_B_MICRO_POWER_SLAVE
- removed CN2: USB3140-30-230-1-C;VERT,2.3FLANGE, HR2:USB3140-30-230-1-C;VERT,2.3FLANGE, symbol HR2:USB_B_MICRO_POWER_MASTER
- removed U1: LM66100;SOT363, Package_TO_SOT_SMD:SOT-363_SC-70-6, symbol HR2:LM66100;SOT363
- added CN1: USB-C;USB-C,POGND, Connector_USB:1USB_C_Receptacle_JAE_DX07S024WJ1R350, symbol HR2:USB-C;USB-C,POGND
- added CN2: USB-C;USB-C, Connector_USB:1USB_C_Receptacle_JAE_DX07S024WJ1R350, symbol HR2:USB-C;USB-C
- added Q26, Q28: 3A_PWR_NMOS_DSG;SOT23, symbol HR2_MISC:Q_PWR_NMOS_DSG
- added Q27: 3A_NMOS_DSG;SOT23, symbol HR2_MISC:Q_PWR_NMOS_DSG
- added R69, R70, R71, R72: 10KΩ;1608, Resistor_SMD:R_0603_1608Metric, symbol Device:R_US
- added U1, U20, U21: LM5050-1;TSOT-23-6, Connector_TO_SOT_SMD:TSOT-23-6, symbol HR2:LM5050-1;TSOT-23-6
Connections:
- net labels removed: USB5V
- wire segments 179 -> 263
- no-connect marks 3 -> 33
Other:
- note added: "Note: Power On/Off circuit is\nfrom David Jones EEVBlog #262"
- note added: "Note: The following URL explains how to get 1.5A@5V from USB-C.\nhttps://www.st.com/resource/en/technical_article/dm00496853-overview-of-usb-type-c-and-power-delivery-technologies-stmicroelectronics.pdf"
- note added: "P5V is a "dirty" 5 volt supply used\nfor lighting LED's, servos, etc."
- note removed: "Note: Power On/Off circuit is from David Jones EEVBlog #262"
- note removed: "Note: The PFET's in the KiCAD library have passive pins\n for design rule checks. A PFET with Power In on the\n Source and Power Out on the Drain is needed.\n It was easier to do an ugly box than a pretty PFET.\n Deal with it."
- note removed: "P5V is a "dirty" 5 volt supply used\nfor lighting LED's etc."
- note removed: "TO DO:\n1. Do power supply review with somebody."
- moved on the sheet: C4, CN93, Q1, R1

Commit message: Moved Power Supply.
Parts:
- removed C1: 22µF;1608, Capacitor_SMD:C_0603_1608Metric, symbol Device:C
- removed Q1, Q3: 2N2222;SOT23, Package_TO_SOT_SMD:SOT-23, symbol Device:Q_NPN_BEC
- removed Q2: PFET_6A;SOT23, symbol HR2_MISC:Q_PWR_PMOS_GSD
- removed Q26: 3A_PWR_NMOS_DSG;SOT23, symbol HR2_MISC:Q_PWR_NMOS_DSG
- removed Q27: 3A_NMOS_DSG;SOT23, symbol HR2_MISC:Q_PWR_NMOS_DSG
- removed R1, R2, R4: 100KΩ;1608, Resistor_SMD:R_0603_1608Metric, symbol Device:R_US
- removed R3: 1MΩ;1608, Resistor_SMD:R_0603_1608Metric, symbol Device:R_US
- removed SW1: BUTTON;6x3.5, HR2:BUTTON_6x3.5, symbol Switch:SW_Push
- added Q1: 3A_PWR_NMOS_DSG;SOT23, Package_TO_SOT_SMD:SOT-23, symbol HR2_MISC:Q_PWR_NMOS_DSG
- added Q27: 3A_PWR_NMOS_DSG;SOT23, Package_TO_SOT_SMD:SOT-23, symbol HR2_MISC:Q_PWR_NMOS_DSG_PI
- CN1, CN2: footprint Connector_USB:1USB_C_Receptacle_JAE_DX07S024WJ1R350 -> Connector_USB:USB_C_Receptacle_JAE_DX07S024WJ3R400
- Q28: footprint (none) -> Package_TO_SOT_SMD:SOT-23
- R20, R21, R22, R63: footprint Resistor_SMD:R_0603_1608Metric -> Resistor_SMD:R_1206_3216Metric
- U1, U20, U21: footprint Connector_TO_SOT_SMD:TSOT-23-6 -> Package_TO_SOT_SMD:TSOT-23-6
Connections:
- net labels added: CN1_5V, CN2_5V
- net labels removed: PWR_FET_G, PWR_QBASE, PWR_SW_A, PWR_SW_B
- wire segments 263 -> 233
Other:
- note removed: "Note: Power On/Off circuit is\nfrom David Jones EEVBlog #262"
- note removed: "Note: The bipolar transtistors are generic\n small signal NPN SOT23 in a BEC (i.e\n pin1 = Base, pin 2 = Emitter,\n pi 3 = Collector) configuration.\n Pretty much any NPN will do, so\n substitutions should be pretty safe."

Commit message: Changed bypass caps and sonar echo outputs
Made following changes:
 - Changed bypass caps to 0.1uF
 - Removed voltage dividers on sonar echo outputs to Nucleo
Connections:
- wire segments 233 -> 232
Changed lines of the file:
@@
 	4000 1400 4400 1400
-Wire Wire Line
-	4400 1400 4400 1000
 Wire Wire Line
 	4400 900  4300 900
@@
 	0    -1   -1   0
 $EndComp
-Connection ~ 4400 1000
-Wire Wire Line
-	4400 1000 4400 900
+Wire Wire Line
+	4400 900  4400 1400
 $EndSCHEMATC

Commit message: JLCPCB BOM is in better shape.
Parts:
- removed Q1, Q28: 3A_PWR_NMOS_DSG;SOT23, Package_TO_SOT_SMD:SOT-23, symbol HR2_MISC:Q_PWR_NMOS_DSG
- removed Q27: 3A_PWR_NMOS_DSG;SOT23, Package_TO_SOT_SMD:SOT-23, symbol HR2_MISC:Q_PWR_NMOS_DSG_PI
- added Q1, Q28: NFET_3A_GSD;SOT23, Package_TO_SOT_SMD:SOT-23, symbol HR2_MISC:Q_PWR_NMOS_GSD
- added Q27: NFET_3A_GSD;SOT23, Package_TO_SOT_SMD:SOT-23, symbol HR2_MISC:Q_PWR_NMOS_GSD_PI
Changed lines of the file:
@@
 	1600 3800 1800 3800
-$Comp
-L HR2_MISC:Q_PWR_NMOS_DSG_PI Q27
-U 1 1 5FDAB4A8
-P 4100 2000
-F 0 "Q27" V 4050 2150 50  0000 C CNN
-F 1 "3A_PWR_NMOS_DSG;SOT23" V 4300 2400 50  0000 C CNN
-F 2 "Package_TO_SOT_SMD:SOT-23" H 4300 2100 50  0001 C CNN
-F 3 "~" H 4100 2000 50  0001 C CNN
-	1    4100 2000
-	0    -1   -1   0
-$EndComp
 $Comp
 L HR2:LM5050-1;TSOT-23-6 U1
@@
 	1    0    0    -1
 $EndComp
-$Comp
-L HR2_MISC:Q_PWR_NMOS_DSG Q28
-U 1 1 5FD516B2
-P 6100 1000
-F 0 "Q28" V 6000 1100 50  0000 C CNN
-F 1 "3A_PWR_NMOS_DSG;SOT23" V 6350 1000 50  0000 C CNN
-F 2 "Package_TO_SOT_SMD:SOT-23" H 6300 1100 50  0001 C CNN
-F 3 "~" H 6100 1000 50  0001 C CNN
-	1    6100 1000
-	0    -1   -1   0
-$EndComp
 Text Label 1700 900  0    50   ~ 0
 CN1_5V
@@
 Wire Wire Line
 	4400 1900 7900 1900
+Wire Wire Line
+	4400 900  4400 1400
 $Comp
-L HR2_MISC:Q_PWR_NMOS_DSG Q1
-U 1 1 5FE080B5
+L HR2_MISC:Q_PWR_NMOS_GSD Q28
+U 1 1 5FE43AF8
+P 6100 1000
+F 0 "Q28" V 6050 1150 50  0000 C CNN
+F 1 "NFET_3A_GSD;SOT23" V 6250 1500 50  0000 C CNN
+F 2 "Package_TO_SOT_SMD:SOT-23" H 6300 1100 50  0001 C CNN
+F 3 "~" H 6100 1000 50  0001 C CNN
+	1    6100 1000
+	0    -1   -1   0
+$EndComp
+$Comp
+L HR2_MISC:Q_PWR_NMOS_GSD_PI Q27
+U 1 1 5FE4EDDB
+P 4100 2000
+F 0 "Q27" V 4050 2200 50  0000 C CNN
+F 1 "NFET_3A_GSD;SOT23" V 4250 2500 50  0000 C CNN
+F 2 "Package_TO_SOT_SMD:SOT-23" H 4300 2100 50  0001 C CNN
+F 3 "~" H 4100 2000 50  0001 C CNN
+	1    4100 2000
+	0    -1   -1   0
+$EndComp
+$Comp
+L HR2_MISC:Q_PWR_NMOS_GSD Q1
+U 1 1 5FE3D28E
 P 4100 1000
 F 0 "Q1" V 4050 1150 50  0000 C CNN
-F 1 "3A_PWR_NMOS_DSG;SOT23" V 4351 1000 50  0000 C CNN
+F 1 "NFET_3A_GSD;SOT23" V 4250 1500 50  0000 C CNN
 F 2 "Package_TO_SOT_SMD:SOT-23" H 4300 1100 50  0001 C CNN
 F 3 "~" H 4100 1000 50  0001 C CNN
@@
 	0    -1   -1   0
 $EndComp
-Wire Wire Line
-	4400 900  4400 1400
 $EndSCHEMATC

Commit message: Made various changes from to_do.md
Parts:
- R15, R17: value 470Ω;1608 -> 180Ω;1005; footprint Resistor_SMD:R_0603_1608Metric -> Resistor_SMD:R_0402_1005Metric
- R16: value 1KΩ;1608 -> 560Ω;1005; footprint Resistor_SMD:R_0603_1608Metric -> Resistor_SMD:R_0402_1005Metric
- R20, R21, R22, R63: value 0Ω;1608 -> 0Ω;3216
- R5: value 330Ω;1608 -> 0Ω;1005; footprint Resistor_SMD:R_0603_1608Metric -> Resistor_SMD:R_0402_1005Metric
Changed lines of the file:
@@
 P 2600 6250
 F 0 "R5" H 2450 6350 50  0000 L CNN
-F 1 "330Ω;1608" H 2650 6150 50  0000 L CNN
-F 2 "Resistor_SMD:R_0603_1608Metric" V 2640 6240 50  0001 C CNN
+F 1 "0Ω;1005" H 2650 6150 50  0000 L CNN
+F 2 "Resistor_SMD:R_0402_1005Metric" V 2640 6240 50  0001 C CNN
 F 3 "~" H 2600 6250 50  0001 C CNN
 	1    2600 6250
@@
 P 3400 6250
 F 0 "R15" H 3250 6350 50  0000 L CNN
-F 1 "470Ω;1608" H 3450 6150 50  0000 L CNN
-F 2 "Resistor_SMD:R_0603_1608Metric" V 3440 6240 50  0001 C CNN
+F 1 "180Ω;1005" H 3450 6150 50  0000 L CNN
+F 2 "Resistor_SMD:R_0402_1005Metric" V 3440 6240 50  0001 C CNN
 F 3 "~" H 3400 6250 50  0001 C CNN
 	1    3400 6250
@@
 P 4200 6250
 F 0 "R16" H 4050 6350 50  0000 L CNN
-F 1 "1KΩ;1608" H 4250 6150 50  0000 L CNN
-F 2 "Resistor_SMD:R_0603_1608Metric" V 4240 6240 50  0001 C CNN
+F 1 "560Ω;1005" H 4250 6150 50  0000 L CNN
+F 2 "Resistor_SMD:R_0402_1005Metric" V 4240 6240 50  0001 C CNN
 F 3 "~" H 4200 6250 50  0001 C CNN
 	1    4200 6250
@@
 P 5000 6250
 F 0 "R17" H 4850 6350 50  0000 L CNN
-F 1 "470Ω;1608" H 5050 6150 50  0000 L CNN
-F 2 "Resistor_SMD:R_0603_1608Metric" V 5040 6240 50  0001 C CNN
+F 1 "180Ω;1005" H 5050 6150 50  0000 L CNN
+F 2 "Resistor_SMD:R_0402_1005Metric" V 5040 6240 50  0001 C CNN
 F 3 "~" H 5000 6250 50  0001 C CNN
 	1    5000 6250
@@
 P 8000 1200
 F 0 "R22" H 8250 1350 50  0000 C CNN
-F 1 "0Ω;1608" H 8450 1050 50  0000 C CNN
+F 1 "0Ω;3216" H 8450 1050 50  0000 C CNN
 F 2 "Resistor_SMD:R_1206_3216Metric" H 8200 1250 60  0001 L CNN
 F 3 "0 Ohm Power Shunt" H 8200 1050 60  0001 L CNN
@@
 P 8000 2900
 F 0 "R63" H 8250 3050 50  0000 C CNN
-F 1 "0Ω;1608" H 8450 2750 50  0000 C CNN
+F 1 "0Ω;3216" H 8450 2750 50  0000 C CNN
 F 2 "Resistor_SMD:R_1206_3216Metric" H 8200 2950 60  0001 L CNN
 F 3 "0 Ohm Power Shunt" H 8200 2750 60  0001 L CNN
@@
 P 8000 2200
 F 0 "R20" H 8250 2350 50  0000 C CNN
-F 1 "0Ω;1608" H 8450 2050 50  0000 C CNN
+F 1 "0Ω;3216" H 8450 2050 50  0000 C CNN
 F 2 "Resistor_SMD:R_1206_3216Metric" H 8200 2250 60  0001 L CNN
 F 3 "0 Ohm Power Shunt" H 8200 2050 60  0001 L CNN
@@
 P 8000 4900
 F 0 "R21" H 8250 5050 50  0000 C CNN
-F 1 "0Ω;1608" H 8450 4750 50  0000 C CNN
+F 1 "0Ω;3216" H 8450 4750 50  0000 C CNN
 F 2 "Resistor_SMD:R_1206_3216Metric" H 8200 4950 60  0001 L CNN
 F 3 "0 Ohm Power Shunt" H 8200 4750 60  0001 L CNN

Commit message: JLCPCB Footprints are both consistent and available.
Parts:
- R15, R17: value 180Ω;1005 -> 220Ω;1005
- R16: value 560Ω;1005 -> 560Ω;1608; footprint Resistor_SMD:R_0402_1005Metric -> Resistor_SMD:R_0603_1608Metric
- R5: value 0Ω;1005 -> 150Ω;1005
Changed lines of the file:
@@
 P 2600 6250
 F 0 "R5" H 2450 6350 50  0000 L CNN
-F 1 "0Ω;1005" H 2650 6150 50  0000 L CNN
+F 1 "150Ω;1005" H 2650 6150 50  0000 L CNN
 F 2 "Resistor_SMD:R_0402_1005Metric" V 2640 6240 50  0001 C CNN
 F 3 "~" H 2600 6250 50  0001 C CNN
@@
 P 3400 6250
 F 0 "R15" H 3250 6350 50  0000 L CNN
-F 1 "180Ω;1005" H 3450 6150 50  0000 L CNN
+F 1 "220Ω;1005" H 3450 6150 50  0000 L CNN
 F 2 "Resistor_SMD:R_0402_1005Metric" V 3440 6240 50  0001 C CNN
 F 3 "~" H 3400 6250 50  0001 C CNN
@@
 P 4200 6250
 F 0 "R16" H 4050 6350 50  0000 L CNN
-F 1 "560Ω;1005" H 4250 6150 50  0000 L CNN
-F 2 "Resistor_SMD:R_0402_1005Metric" V 4240 6240 50  0001 C CNN
+F 1 "560Ω;1608" H 4250 6150 50  0000 L CNN
+F 2 "Resistor_SMD:R_0603_1608Metric" V 4240 6240 50  0001 C CNN
 F 3 "~" H 4200 6250 50  0001 C CNN
 	1    4200 6250
@@
 P 5000 6250
 F 0 "R17" H 4850 6350 50  0000 L CNN
-F 1 "180Ω;1005" H 5050 6150 50  0000 L CNN
+F 1 "220Ω;1005" H 5050 6150 50  0000 L CNN
 F 2 "Resistor_SMD:R_0402_1005Metric" V 5040 6240 50  0001 C CNN
 F 3 "~" H 5000 6250 50  0001 C CNN

Commit message: Changed various resistor sizes and values
Parts:
- R5: value 150Ω;1005 -> 33Ω;1005
- R69, R70, R71, R72: value 10KΩ;1608 -> 10KΩ;1005; footprint Resistor_SMD:R_0603_1608Metric -> Resistor_SMD:R_0402_1005Metric
Changed lines of the file:
@@
 P 2600 6250
 F 0 "R5" H 2450 6350 50  0000 L CNN
-F 1 "150Ω;1005" H 2650 6150 50  0000 L CNN
+F 1 "33Ω;1005" H 2650 6150 50  0000 L CNN
 F 2 "Resistor_SMD:R_0402_1005Metric" V 2640 6240 50  0001 C CNN
 F 3 "~" H 2600 6250 50  0001 C CNN
@@
 P 2150 2700
 F 0 "R72" V 2050 2550 50  0000 L CNN
-F 1 "10KΩ;1608" V 2250 2500 50  0000 L CNN
-F 2 "Resistor_SMD:R_0603_1608Metric" V 2190 2690 50  0001 C CNN
+F 1 "10KΩ;1005" V 2250 2500 50  0000 L CNN
+F 2 "Resistor_SMD:R_0402_1005Metric" V 2190 2690 50  0001 C CNN
 F 3 "~" H 2150 2700 50  0001 C CNN
 	1    2150 2700
@@
 P 2150 2400
 F 0 "R71" V 2050 2250 50  0000 L CNN
-F 1 "10KΩ;1608" V 2250 2200 50  0000 L CNN
-F 2 "Resistor_SMD:R_0603_1608Metric" V 2190 2390 50  0001 C CNN
+F 1 "10KΩ;1005" V 2250 2200 50  0000 L CNN
+F 2 "Resistor_SMD:R_0402_1005Metric" V 2190 2390 50  0001 C CNN
 F 3 "~" H 2150 2400 50  0001 C CNN
 	1    2150 2400
@@
 P 2050 5600
 F 0 "R70" V 1950 5450 50  0000 L CNN
-F 1 "10KΩ;1608" V 2150 5400 50  0000 L CNN
-F 2 "Resistor_SMD:R_0603_1608Metric" V 2090 5590 50  0001 C CNN
+F 1 "10KΩ;1005" V 2150 5400 50  0000 L CNN
+F 2 "Resistor_SMD:R_0402_1005Metric" V 2090 5590 50  0001 C CNN
 F 3 "~" H 2050 5600 50  0001 C CNN
 	1    2050 5600
@@
 P 2050 5300
 F 0 "R69" V 1950 5150 50  0000 L CNN
-F 1 "10KΩ;1608" V 2150 5100 50  0000 L CNN
-F 2 "Resistor_SMD:R_0603_1608Metric" V 2090 5290 50  0001 C CNN
+F 1 "10KΩ;1005" V 2150 5100 50  0000 L CNN
+F 2 "Resistor_SMD:R_0402_1005Metric" V 2090 5290 50  0001 C CNN
 F 3 "~" H 2050 5300 50  0001 C CNN
 	1    2050 5300
