File: electrical/master_board/rev_a/wowbus.sch (KiCad schematic (older format))
At the start: 22 parts, among them CN8 WOW_OUT;M2x6S, Q17 2N7000;SOT23, Q4 2N7000;SOT23, Q5 2N7000;SOT23, Q6 PFET_6A_GSD;SOT23, U13 74LVC1G08;TTSOP8, U14 LTV-827, U15 LTV-827, U16 74LVC1G74;TSSOP8, U17 LTV-827, U18 LTV-827

Commit message: Bound signals to Morpho pins.
Parts:
- removed Q17: 2N7000;SOT23, Package_TO_SOT_SMD:SOT-23, symbol Transistor_FET:2N7000
- removed R39: 100KΩ;1608, symbol Device:R_US
Connections:
- net labels removed: WOW_RXD
- wire segments 169 -> 163
Changed lines of the file:
@@
 $Descr A4 11693 8268
 encoding utf-8
-Sheet 10 10
+Sheet 6 10
 Title "HR2: WOWBus"
 Date "2020-10-17"
@@
 L Transistor_FET:2N7000 Q?
 U 1 1 5F86962A
-P 3400 5400
+P 3400 5600
 AR Path="/5F79BC00/5F86962A" Ref="Q?"  Part="1"
 AR Path="/5FA4A874/5F86962A" Ref="Q?"  Part="1"
 AR Path="/5FAD82EE/5F86962A" Ref="Q?"  Part="1"
 AR Path="/5F8C2F57/5F86962A" Ref="Q5"  Part="1"
-F 0 "Q5" H 3300 5550 50  0000 L CNN
-F 1 "2N7000;SOT23" H 2900 5200 50  0000 L CNN
-F 2 "Package_TO_SOT_SMD:SOT-23" H 3600 5325 50  0001 L CIN
-F 3 "https://www.fairchildsemi.com/datasheets/2N/2N7000.pdf" H 3400 5400 50  0001 L CNN
-	1    3400 5400
+F 0 "Q5" H 3300 5750 50  0000 L CNN
+F 1 "2N7000;SOT23" H 2900 5400 50  0000 L CNN
+F 2 "Package_TO_SOT_SMD:SOT-23" H 3600 5525 50  0001 L CIN
+F 3 "https://www.fairchildsemi.com/datasheets/2N/2N7000.pdf" H 3400 5600 50  0001 L CNN
+	1    3400 5600
 	1    0    0    -1
 $EndComp
@@
 Text HLabel 1000 6800 0    50   Input ~ 0
 GND
-Text HLabel 1000 5400 0    50   Input ~ 0
+Text HLabel 1000 5600 0    50   Input ~ 0
 WOW_EN
 $Comp
@@
 $EndComp
 Wire Wire Line
-	3500 5600 3500 6800
+	3500 5800 3500 6800
 Connection ~ 3500 6800
 Wire Wire Line
-	3500 6800 4100 6800
-Wire Wire Line
 	1000 3900 1700 3900
 Wire Wire Line
 	3500 3900 3500 4000
-Connection ~ 4700 5100
 $Comp
 L Device:R_US R35
@@
 $EndComp
 Wire Wire Line
-	1600 6350 1600 5400
-Wire Wire Line
-	6200 3900 4100 3900
+	1600 6350 1600 5600
 Connection ~ 3500 3900
 Wire Wire Line
@@
 L Transistor_FET:2N7000 Q?
 U 1 1 5F9A0944
-P 2700 5700
+P 2700 4500
 AR Path="/5F79BC00/5F9A0944" Ref="Q?"  Part="1"
 AR Path="/5FA4A874/5F9A0944" Ref="Q?"  Part="1"
 AR Path="/5FAD82EE/5F9A0944" Ref="Q?"  Part="1"
 AR Path="/5F8C2F57/5F9A0944" Ref="Q4"  Part="1"
-F 0 "Q4" H 2600 5850 50  0000 L CNN
-F 1 "2N7000;SOT23" H 2850 5550 50  0000 L CNN
-F 2 "Package_TO_SOT_SMD:SOT-23" H 2900 5625 50  0001 L CIN
-F 3 "https://www.fairchildsemi.com/datasheets/2N/2N7000.pdf" H 2700 5700 50  0001 L CNN
-	1    2700 5700
-	1    0    0    -1
-$EndComp
-Wire Wire Line
-	2800 2350 2800 5500
+F 0 "Q4" H 2600 4650 50  0000 L CNN
+F 1 "2N7000;SOT23" H 2850 4350 50  0000 L CNN
+F 2 "Package_TO_SOT_SMD:SOT-23" H 2900 4425 50  0001 L CIN
+F 3 "https://www.fairchildsemi.com/datasheets/2N/2N7000.pdf" H 2700 4500 50  0001 L CNN
+	1    2700 4500
+	1    0    0    -1
+$EndComp
+Wire Wire Line
+	2800 2350 2800 4300
 Wire Wire Line
 	6300 3500 10200 3500
@@
 $EndComp
 Wire Wire Line
-	4800 4900 4600 4900
-Wire Wire Line
-	4600 4900 4600 5600
-Wire Wire Line
-	4600 5600 6000 5600
-Wire Wire Line
-	6000 5600 6000 6100
-Wire Wire Line
 	6000 6100 5900 6100
 Wire Wire Line
@@
 Wire Wire Line
 	6000 7200 1000 7200
-Connection ~ 6000 6100
 Wire Wire Line
 	5900 6000 6100 6000
@@
 Text HLabel 1000 7200 0    50   Output ~ 0
 ~ESTOP
-$Comp
-L Transistor_FET:2N7000 Q?
-U 1 1 5F9C400A
-P 4000 6500
-AR Path="/5F79BC00/5F9C400A" Ref="Q?"  Part="1"
-AR Path="/5FA4A874/5F9C400A" Ref="Q?"  Part="1"
-AR Path="/5FAD82EE/5F9C400A" Ref="Q?"  Part="1"
-AR Path="/5F8C2F57/5F9C400A" Ref="Q17"  Part="1"
-F 0 "Q17" H 3900 6650 50  0000 L CNN
-F 1 "2N7000;SOT23" H 4150 6350 50  0000 L CNN
-F 2 "Package_TO_SOT_SMD:SOT-23" H 4200 6425 50  0001 L CIN
-F 3 "https://www.fairchildsemi.com/datasheets/2N/2N7000.pdf" H 4000 6500 50  0001 L CNN
-	1    4000 6500
-	1    0    0    -1
-$EndComp
 Wire Wire Line
 	6100 5000 6100 5700
-Wire Wire Line
-	4800 5000 3700 5000
-Wire Wire Line
-	3700 5000 3700 6500
-Wire Wire Line
-	3700 6500 3800 6500
-Wire Wire Line
-	4100 6700 4100 6800
-Connection ~ 4100 6800
-Wire Wire Line
-	4100 6800 6300 6800
-$Comp
-L Device:R_US R39
-U 1 1 5FA11EAD
-P 4100 4150
-F 0 "R39" H 3950 4250 50  0000 L CNN
-F 1 "100KΩ;1608" H 4150 4050 50  0000 L CNN
-F 2 "" V 4140 4140 50  0001 C CNN
-F 3 "~" H 4100 4150 50  0001 C CNN
-	1    4100 4150
-	1    0    0    -1
-$EndComp
-Wire Wire Line
-	3500 4300 3500 5100
-Wire Wire Line
-	4100 4000 4100 3900
-Connection ~ 4100 3900
-Wire Wire Line
-	4100 3900 3500 3900
-Wire Wire Line
-	4700 5100 3500 5100
-Connection ~ 3500 5100
-Wire Wire Line
-	3500 5100 3500 5200
 Text HLabel 1000 6000 0    50   Input ~ 0
 ~ESTOP_CLR
@@
 Wire Wire Line
 	6100 5700 6100 5900
-Wire Wire Line
-	4100 4300 4100 6100
-Wire Wire Line
-	4800 6100 4100 6100
-Connection ~ 4100 6100
-Wire Wire Line
-	4100 6100 4100 6300
 Wire Wire Line
 	4800 5900 4700 5900
@@
 	2200 6800 2800 6800
 Wire Wire Line
-	2800 5900 2800 6800
+	2800 4700 2800 6800
 Connection ~ 2800 6800
 Wire Wire Line
@@
 	1000 6800 1600 6800
 Wire Wire Line
-	1000 5400 1600 5400
-Wire Wire Line
-	2400 5700 2400 5400
-Wire Wire Line
-	2400 5700 2500 5700
-Wire Wire Line
-	2400 5400 3200 5400
+	1000 5600 1600 5600
+Wire Wire Line
+	2400 4500 2400 5600
+Wire Wire Line
+	2400 4500 2500 4500
+Wire Wire Line
+	2400 5600 3200 5600
 $Comp
 L Device:R_US R36
@@
 Text Label 1000 3900 0    50   ~ 0
 3.3V
-Text Label 1000 5400 0    50   ~ 0
+Text Label 1000 5600 0    50   ~ 0
 WOW_EN
 Text Label 1000 6000 0    50   ~ 0
@@
 Text Label 1000 6800 0    50   ~ 0
 GND
-Text Label 4150 6200 0    50   ~ 0
+Text Label 4250 6200 0    50   ~ 0
 ~ESTOP_RESET
-Text Label 4150 6100 0    50   ~ 0
+Text Label 4250 6100 0    50   ~ 0
 ESTOP_TRIG
-Text Label 4150 5000 0    50   ~ 0
-WOW_RXD
-Text Label 4150 5100 0    50   ~ 0
+Text Label 4400 5000 0    50   ~ 0
+~ESTOP
+Text Label 4100 4500 0    50   ~ 0
 WOW_STDBY
 Wire Wire Line
-	2400 5400 1600 5400
-Connection ~ 2400 5400
-Connection ~ 1600 5400
+	2400 5600 1600 5600
+Connection ~ 2400 5600
+Connection ~ 1600 5600
 Text Label 7900 1900 0    50   ~ 0
 WOW_POW_OUT
@@
 Connection ~ 4700 3800
 Wire Wire Line
-	4700 3800 4700 5100
+	4700 3800 4700 4500
 Wire Wire Line
 	9000 4000 9000 3600
@@
 Wire Wire Line
 	6700 6200 6700 6100
+Wire Wire Line
+	4800 6100 4200 6100
+Wire Wire Line
+	4800 4900 4200 4900
+Wire Wire Line
+	4200 4900 4200 6100
+Connection ~ 4700 4500
+Wire Wire Line
+	4700 4500 4700 5100
+Wire Wire Line
+	6000 6100 6000 5500
+Wire Wire Line
+	6000 5500 4300 5500
+Wire Wire Line
+	4300 5500 4300 5000
+Wire Wire Line
+	4300 5000 4800 5000
+Connection ~ 6000 6100
+Wire Wire Line
+	3500 6800 6300 6800
+Wire Wire Line
+	3500 3900 6200 3900
+Wire Wire Line
+	3500 4300 3500 4500
+Connection ~ 3500 4500
+Wire Wire Line
+	3500 4500 3500 5400
+Wire Wire Line
+	3500 4500 4700 4500
 $EndSCHEMATC

Commit message: Schematic is basically complete.
Parts:
- removed U13: 74LVC1G08;TTSOP8, symbol 74xGxx:74LVC1G08
- added C14, C15, C16, C17: 10pF;1608, symbol Device:C
- added R62: 100KΩ;1608, symbol Device:R_US
- added SW3: PUSH_BUTTON;6x6x9.5H, symbol Switch:SW_Push
- added U13: 74LVC1G11, symbol 74xGxx:74LVC1G11
Connections:
- net labels added: ~ESTOP_SET, ~MOTOR_FAULT, ~WOW_EN
- net labels removed: ~ESTOP_RESET
- wire segments 163 -> 190
Other:
- note added: "2\n"
- note added: "3.3 to 9V\nLevel Shift"
- note added: "Bypass Capacitors"
- note added: "Communication CANBus Transceiver"
- note added: "Dual Opto-isolator"
- note added: "E-Stop Set\n3-Input\nAND Gate"
- note added: "E-Stop x74 D Style Flip-Flop"
- note added: "ESTOP CANBus Transceiver"
- note added: "Manual\nE-Stop\nButton"
- note added: "WOW Power P-FET (6A)"
- note added: "WOW Standby\nInverter"
- note removed: "'74 D Flip-Flop"
- note removed: "3"
- note removed: "6 Amp PFET"
- note removed: "CANBus Transceiver"
- moved on the sheet: D2, Q6, R35, R36, R37, R38, R40, R41, R42, R43, R60

Commit message: Fixed corruption of order1.lib file.
Parts:
- Q6: footprint HR2: -> HR2:POWER_PFET_GSD; manf# Power PFG (GSD pinout) -> (none)
Changed lines of the file:
@@
 $Descr A 11000 8500
 encoding utf-8
-Sheet 5 10
+Sheet 10 10
 Title "HR2: WOWBus"
 Date "2020-10-17"
@@
 Wire Wire Line
 	8000 2300 8000 2100
-$Comp
-L HR2:POWER_PFET_GSD Q6
-U 1 1 5F84ED87
-P 4500 900
-F 0 "Q6" H 4750 1050 50  0000 C CNN
-F 1 "PFET_6A_GSD;SOT23" H 4900 650 50  0000 C CNN
-F 2 "HR2:" H 4700 950 60  0001 L CNN
-F 3 "Power PFG (GSD pinout)" H 4700 750 60  0001 L CNN
-F 4 "Power PFG (GSD pinout)" H 4700 850 60  0001 L CNN "manf#"
-F 5 "Power PFET (GSD pinout)" H 4700 650 60  0001 L CNN "Field5"
-	1    4500 900
-	1    0    0    -1
-$EndComp
 $Comp
 L Device:R_US R37
@@
 Wire Wire Line
 	8700 3000 9400 3000
+$Comp
+L HR2:POWER_PFET_GSD Q6
+U 1 1 5F9BEDD5
+P 4500 900
+F 0 "Q6" H 4750 1050 50  0000 C CNN
+F 1 "PFET_6A_GSD;SOT23" H 4900 650 50  0000 C CNN
+F 2 "HR2:POWER_PFET_GSD" H 4700 950 60  0001 L CNN
+F 3 "Power PFG (GSD pinout)" H 4700 750 60  0001 L CNN
+F 4 "Power PFET (GSD pinout)" H 4700 650 60  0001 L CNN "Field5"
+	1    4500 900
+	1    0    0    -1
+$EndComp
 $EndSCHEMATC

Commit message: Reannoted. Postioned components are in the 80-99 reference range.
Parts:
- renumbered C14 to C22, C15 to C23, C16 to C24, C17 to C25, CN8 to CN10, D2 to D3, Q4 to Q20, Q6 to Q21, Q5 to Q22, R36 to R53, R62 to R54, R37 to R55, R35 to R56, R38 to R57, R40 to R58, R41 to R59, R42 to R60, R60 to R61, R43 to R62
Changed lines of the file:
@@
 	7000 1500 7000 1700
 $Comp
-L Device:R_US R41
+L Device:R_US R59
 U 1 1 5F846FDA
 P 8000 1950
-F 0 "R41" H 7850 2050 50  0000 L CNN
+F 0 "R59" H 7850 2050 50  0000 L CNN
 F 1 "120Ω1/4W;1608" H 8050 1850 50  0000 L CNN
 F 2 "" V 8040 1940 50  0001 C CNN
@@
 	8000 2300 8000 2100
 $Comp
-L Device:R_US R37
+L Device:R_US R55
 U 1 1 5F869783
 P 3800 1200
-F 0 "R37" H 3650 1300 50  0000 L CNN
+F 0 "R55" H 3650 1300 50  0000 L CNN
 F 1 "100KΩ;1608" H 3850 1100 50  0000 L CNN
 F 2 "" V 3840 1190 50  0001 C CNN
@@
 WOW_EN
 $Comp
-L Device:R_US R38
+L Device:R_US R57
 U 1 1 5F873ADD
 P 4600 3250
-F 0 "R38" H 4450 3350 50  0000 L CNN
+F 0 "R57" H 4450 3350 50  0000 L CNN
 F 1 "100KΩ;1608" H 4650 3150 50  0000 L CNN
 F 2 "" V 4640 3240 50  0001 C CNN
@@
 $EndComp
 $Comp
-L HR2:WOW_OUT;M2x6S CN8
+L HR2:WOW_OUT;M2x6S CN10
 U 1 1 5F848F57
 P 9600 4600
-F 0 "CN8" H 9800 4750 50  0000 L CNN
+F 0 "CN10" H 9800 4750 50  0000 L CNN
 F 1 "WOW_OUT;M2x6S" H 9750 3350 50  0000 L CNN
 F 2 "Connector_PinHeader_2.54:PinHeader_2x06_P2.54mm_Vertical" H 9800 4650 60  0001 L CNN
@@
 	7000 3200 7000 3400
 $Comp
-L Device:R_US R42
+L Device:R_US R60
 U 1 1 5F84B29E
 P 8000 3650
-F 0 "R42" H 7850 3750 50  0000 L CNN
+F 0 "R60" H 7850 3750 50  0000 L CNN
 F 1 "120Ω1/4W;1608" H 8050 3550 50  0000 L CNN
 F 2 "" V 8040 3640 50  0001 C CNN
@@
 Connection ~ 4600 5900
 $Comp
-L Device:R_US R35
+L Device:R_US R56
 U 1 1 5F98DD9D
 P 4000 5650
-F 0 "R35" H 3850 5750 50  0000 L CNN
+F 0 "R56" H 3850 5750 50  0000 L CNN
 F 1 "100KΩ;1608" H 4000 5500 50  0000 L CNN
 F 2 "" V 4040 5640 50  0001 C CNN
@@
 AR Path="/5FA4A874/5F9A0944" Ref="Q?"  Part="1"
 AR Path="/5FAD82EE/5F9A0944" Ref="Q?"  Part="1"
-AR Path="/5F8C2F57/5F9A0944" Ref="Q4"  Part="1"
-F 0 "Q4" H 3600 4350 50  0000 L CNN
+AR Path="/5F8C2F57/5F9A0944" Ref="Q20"  Part="1"
+F 0 "Q20" H 3600 4350 50  0000 L CNN
 F 1 "2N7000;SOT23" H 3850 4050 50  0000 L CNN
 F 2 "Package_TO_SOT_SMD:SOT-23" H 3900 4125 50  0001 L CIN
@@
 	9400 1300 9400 1400
 $Comp
-L Device:R_US R60
+L Device:R_US R61
 U 1 1 5F8EAE9D
 P 9400 1550
-F 0 "R60" H 9250 1650 50  0000 L CNN
+F 0 "R61" H 9250 1650 50  0000 L CNN
 F 1 "100KΩ;1608" H 8900 1400 50  0000 L CNN
 F 2 "" V 9440 1540 50  0001 C CNN
@@
 	3400 4200 3500 4200
 $Comp
-L Device:R_US R36
+L Device:R_US R53
 U 1 1 5FC61F4D
 P 2300 3250
-F 0 "R36" H 2150 3350 50  0000 L CNN
+F 0 "R53" H 2150 3350 50  0000 L CNN
 F 1 "100KΩ;1608" H 2300 3100 50  0000 L CNN
 F 2 "" V 2340 3240 50  0001 C CNN
@@
 AR Path="/5FA4A874/5FC8C292" Ref="D?"  Part="1"
 AR Path="/5FAD82EE/5FC8C292" Ref="D?"  Part="1"
-AR Path="/5F8C2F57/5FC8C292" Ref="D2"  Part="1"
-F 0 "D2" V 7200 5550 50  0000 R CNN
+AR Path="/5F8C2F57/5FC8C292" Ref="D3"  Part="1"
+F 0 "D3" V 7200 5550 50  0000 R CNN
 F 1 "REDLED;1608" V 7050 5350 50  0000 R CNN
 F 2 "HR2:LED_GRNRA" H 7100 5450 50  0001 C CNN
@@
 $EndComp
 $Comp
-L Device:R_US R40
+L Device:R_US R58
 U 1 1 5FC946D0
 P 7100 5050
-F 0 "R40" H 6950 5150 50  0000 L CNN
+F 0 "R58" H 6950 5150 50  0000 L CNN
 F 1 "470Ω;1608" H 7150 4950 50  0000 L CNN
 F 2 "" V 7140 5040 50  0001 C CNN
@@
 AR Path="/5FA4A874/5F86962A" Ref="Q?"  Part="1"
 AR Path="/5FAD82EE/5F86962A" Ref="Q?"  Part="1"
-AR Path="/5F8C2F57/5F86962A" Ref="Q5"  Part="1"
-F 0 "Q5" H 4400 4650 50  0000 L CNN
+AR Path="/5F8C2F57/5F86962A" Ref="Q22"  Part="1"
+F 0 "Q22" H 4400 4650 50  0000 L CNN
 F 1 "2N7000;SOT23" H 4000 4300 50  0000 L CNN
 F 2 "Package_TO_SOT_SMD:SOT-23" H 4700 4425 50  0001 L CIN
@@
 Connection ~ 3800 5900
 $Comp
-L Device:R_US R62
+L Device:R_US R54
 U 1 1 5FF6B902
 P 2800 3250
-F 0 "R62" H 2650 3350 50  0000 L CNN
+F 0 "R54" H 2650 3350 50  0000 L CNN
 F 1 "100KΩ;1608" H 2800 3100 50  0000 L CNN
 F 2 "" V 2840 3240 50  0001 C CNN
@@
 P 1550 4000
 AR Path="/5F48CAAD/6036DBC8" Ref="C?"  Part="1"
-AR Path="/5F8C2F57/6036DBC8" Ref="C16"  Part="1"
-F 0 "C16" V 1450 3800 50  0000 L CNN
+AR Path="/5F8C2F57/6036DBC8" Ref="C24"  Part="1"
+F 0 "C24" V 1450 3800 50  0000 L CNN
 F 1 "10pF;1608" V 1650 4050 50  0000 L CNN
 F 2 "" H 1588 3850 50  0001 C CNN
@@
 P 1550 4300
 AR Path="/5F48CAAD/60430375" Ref="C?"  Part="1"
-AR Path="/5F8C2F57/60430375" Ref="C17"  Part="1"
-F 0 "C17" V 1450 4100 50  0000 L CNN
+AR Path="/5F8C2F57/60430375" Ref="C25"  Part="1"
+F 0 "C25" V 1450 4100 50  0000 L CNN
 F 1 "10pF;1608" V 1600 4350 50  0000 L CNN
 F 2 "" H 1588 4150 50  0001 C CNN
@@
 P 1550 3700
 AR Path="/5F48CAAD/6043088F" Ref="C?"  Part="1"
-AR Path="/5F8C2F57/6043088F" Ref="C15"  Part="1"
-F 0 "C15" V 1450 3500 50  0000 L CNN
+AR Path="/5F8C2F57/6043088F" Ref="C23"  Part="1"
+F 0 "C23" V 1450 3500 50  0000 L CNN
 F 1 "10pF;1608" V 1600 3750 50  0000 L CNN
 F 2 "" H 1588 3550 50  0001 C CNN
@@
 P 1550 3400
 AR Path="/5F48CAAD/6057FE20" Ref="C?"  Part="1"
-AR Path="/5F8C2F57/6057FE20" Ref="C14"  Part="1"
-F 0 "C14" V 1450 3200 50  0000 L CNN
+AR Path="/5F8C2F57/6057FE20" Ref="C22"  Part="1"
+F 0 "C22" V 1450 3200 50  0000 L CNN
 F 1 "10pF;1608" V 1600 3450 50  0000 L CNN
 F 2 "" H 1588 3250 50  0001 C CNN
@@
 	9400 3000 9400 2850
 $Comp
-L Device:R_US R43
+L Device:R_US R62
 U 1 1 5F8E9E6C
 P 9400 2700
-F 0 "R43" H 9250 2800 50  0000 L CNN
+F 0 "R62" H 9250 2800 50  0000 L CNN
 F 1 "100KΩ;1608" H 8900 2550 50  0000 L CNN
 F 2 "" V 9440 2690 50  0001 C CNN
@@
 	8700 3000 9400 3000
 $Comp
-L HR2:POWER_PFET_GSD Q6
+L HR2:POWER_PFET_GSD Q21
 U 1 1 5F9BEDD5
 P 4500 900
-F 0 "Q6" H 4750 1050 50  0000 C CNN
+F 0 "Q21" H 4750 1050 50  0000 C CNN
 F 1 "PFET_6A_GSD;SOT23" H 4900 650 50  0000 C CNN
 F 2 "HR2:POWER_PFET_GSD" H 4700 950 60  0001 L CNN

Commit message: Assigned PCB footprints.
Parts:
- C22, C23, C24, C25: footprint (none) -> Capacitor_SMD:C_0603_1608Metric
- D3: footprint HR2:LED_GRNRA -> LED_SMD:LED_0603_1608Metric
- Q21: footprint HR2:POWER_PFET_GSD -> Package_TO_SOT_SMD:SOT-23
- R53, R54, R55, R56, R57, R58, R59, R60, R61, R62: footprint (none) -> Resistor_SMD:R_0603_1608Metric
- SW3: footprint (none) -> Button_Switch_SMD:SW_SPST_PTS645
- U13: value 74LVC1G11 -> 74LVC1G11;6TSSOP; footprint (none) -> Package_SO:TSOP-6_1.65x3.05mm_P0.95mm
Connections:
- wire segments 190 -> 191
Changed lines of the file:
@@
 F 0 "R59" H 7850 2050 50  0000 L CNN
 F 1 "120Ω1/4W;1608" H 8050 1850 50  0000 L CNN
-F 2 "" V 8040 1940 50  0001 C CNN
+F 2 "Resistor_SMD:R_0603_1608Metric" V 8040 1940 50  0001 C CNN
 F 3 "~" H 8000 1950 50  0001 C CNN
 	1    8000 1950
@@
 F 0 "R55" H 3650 1300 50  0000 L CNN
 F 1 "100KΩ;1608" H 3850 1100 50  0000 L CNN
-F 2 "" V 3840 1190 50  0001 C CNN
+F 2 "Resistor_SMD:R_0603_1608Metric" V 3840 1190 50  0001 C CNN
 F 3 "~" H 3800 1200 50  0001 C CNN
 	1    3800 1200
@@
 F 0 "R57" H 4450 3350 50  0000 L CNN
 F 1 "100KΩ;1608" H 4650 3150 50  0000 L CNN
-F 2 "" V 4640 3240 50  0001 C CNN
+F 2 "Resistor_SMD:R_0603_1608Metric" V 4640 3240 50  0001 C CNN
 F 3 "~" H 4600 3250 50  0001 C CNN
 	1    4600 3250
@@
 F 0 "R60" H 7850 3750 50  0000 L CNN
 F 1 "120Ω1/4W;1608" H 8050 3550 50  0000 L CNN
-F 2 "" V 8040 3640 50  0001 C CNN
+F 2 "Resistor_SMD:R_0603_1608Metric" V 8040 3640 50  0001 C CNN
 F 3 "~" H 8000 3650 50  0001 C CNN
 	1    8000 3650
@@
 F 0 "R56" H 3850 5750 50  0000 L CNN
 F 1 "100KΩ;1608" H 4000 5500 50  0000 L CNN
-F 2 "" V 4040 5640 50  0001 C CNN
+F 2 "Resistor_SMD:R_0603_1608Metric" V 4040 5640 50  0001 C CNN
 F 3 "~" H 4000 5650 50  0001 C CNN
 	1    4000 5650
@@
 F 0 "R61" H 9250 1650 50  0000 L CNN
 F 1 "100KΩ;1608" H 8900 1400 50  0000 L CNN
-F 2 "" V 9440 1540 50  0001 C CNN
+F 2 "Resistor_SMD:R_0603_1608Metric" V 9440 1540 50  0001 C CNN
 F 3 "~" H 9400 1550 50  0001 C CNN
 	1    9400 1550
@@
 F 0 "R53" H 2150 3350 50  0000 L CNN
 F 1 "100KΩ;1608" H 2300 3100 50  0000 L CNN
-F 2 "" V 2340 3240 50  0001 C CNN
+F 2 "Resistor_SMD:R_0603_1608Metric" V 2340 3240 50  0001 C CNN
 F 3 "~" H 2300 3250 50  0001 C CNN
 	1    2300 3250
@@
 F 0 "D3" V 7200 5550 50  0000 R CNN
 F 1 "REDLED;1608" V 7050 5350 50  0000 R CNN
-F 2 "HR2:LED_GRNRA" H 7100 5450 50  0001 C CNN
+F 2 "LED_SMD:LED_0603_1608Metric" H 7100 5450 50  0001 C CNN
 F 3 "~" H 7100 5450 50  0001 C CNN
 	1    7100 5450
@@
 F 0 "R58" H 6950 5150 50  0000 L CNN
 F 1 "470Ω;1608" H 7150 4950 50  0000 L CNN
-F 2 "" V 7140 5040 50  0001 C CNN
+F 2 "Resistor_SMD:R_0603_1608Metric" V 7140 5040 50  0001 C CNN
 F 3 "~" H 7100 5050 50  0001 C CNN
 	1    7100 5050
@@
 Wire Wire Line
 	3400 4500 4000 4500
-Wire Wire Line
-	4600 4700 4600 5900
 $Comp
 L Transistor_FET:2N7000 Q?
@@
 F 0 "SW3" H 2350 5800 50  0000 C CNN
 F 1 "PUSH_BUTTON;6x6x9.5H" H 2650 5600 50  0000 C CNN
-F 2 "" H 2500 5900 50  0001 C CNN
+F 2 "Button_Switch_SMD:SW_SPST_PTS645" H 2500 5900 50  0001 C CNN
 F 3 "~" H 2500 5900 50  0001 C CNN
 	1    2500 5700
@@
 	4800 4000 4800 5200
 Wire Wire Line
-	3800 4400 3800 5900
+	3800 4400 3800 5200
 Connection ~ 3800 5900
 $Comp
@@
 F 0 "R54" H 2650 3350 50  0000 L CNN
 F 1 "100KΩ;1608" H 2800 3100 50  0000 L CNN
-F 2 "" V 2840 3240 50  0001 C CNN
+F 2 "Resistor_SMD:R_0603_1608Metric" V 2840 3240 50  0001 C CNN
 F 3 "~" H 2800 3250 50  0001 C CNN
 	1    2800 3250
@@
 P 3300 5000
 F 0 "U13" H 3200 5200 50  0000 C CNN
-F 1 "74LVC1G11" H 3550 4800 50  0000 C CNN
-F 2 "" H 3300 5000 50  0001 C CNN
+F 1 "74LVC1G11;6TSSOP" H 3350 4750 50  0000 C CNN
+F 2 "Package_SO:TSOP-6_1.65x3.05mm_P0.95mm" H 3300 5000 50  0001 C CNN
 F 3 "http://www.ti.com/lit/sg/scyt129e/scyt129e.pdf" H 3300 5000 50  0001 C CNN
 	1    3300 5000
@@
 Text Notes 3250 5200 0    40   ~ 0
 2\n
-Wire Wire Line
-	4000 5500 4000 4500
 Connection ~ 4000 4500
 Wire Wire Line
@@
 Connection ~ 2100 5900
 Wire Wire Line
-	2100 5900 3300 5900
-Wire Wire Line
-	3300 5125 3300 5900
-Connection ~ 3300 5900
-Wire Wire Line
-	3300 5900 3800 5900
+	3300 5125 3300 5200
 Wire Wire Line
 	2800 3000 3300 3000
@@
 F 0 "C24" V 1450 3800 50  0000 L CNN
 F 1 "10pF;1608" V 1650 4050 50  0000 L CNN
-F 2 "" H 1588 3850 50  0001 C CNN
+F 2 "Capacitor_SMD:C_0603_1608Metric" H 1588 3850 50  0001 C CNN
 F 3 "~" H 1550 4000 50  0001 C CNN
 	1    1550 4000
@@
 F 0 "C25" V 1450 4100 50  0000 L CNN
 F 1 "10pF;1608" V 1600 4350 50  0000 L CNN
-F 2 "" H 1588 4150 50  0001 C CNN
+F 2 "Capacitor_SMD:C_0603_1608Metric" H 1588 4150 50  0001 C CNN
 F 3 "~" H 1550 4300 50  0001 C CNN
 	1    1550 4300
@@
 F 0 "C23" V 1450 3500 50  0000 L CNN
 F 1 "10pF;1608" V 1600 3750 50  0000 L CNN
-F 2 "" H 1588 3550 50  0001 C CNN
+F 2 "Capacitor_SMD:C_0603_1608Metric" H 1588 3550 50  0001 C CNN
 F 3 "~" H 1550 3700 50  0001 C CNN
 	1    1550 3700
@@
 F 0 "C22" V 1450 3200 50  0000 L CNN
 F 1 "10pF;1608" V 1600 3450 50  0000 L CNN
-F 2 "" H 1588 3250 50  0001 C CNN
+F 2 "Capacitor_SMD:C_0603_1608Metric" H 1588 3250 50  0001 C CNN
 F 3 "~" H 1550 3400 50  0001 C CNN
 	1    1550 3400
@@
 F 0 "R62" H 9250 2800 50  0000 L CNN
 F 1 "100KΩ;1608" H 8900 2550 50  0000 L CNN
-F 2 "" V 9440 2690 50  0001 C CNN
+F 2 "Resistor_SMD:R_0603_1608Metric" V 9440 2690 50  0001 C CNN
 F 3 "~" H 9400 2700 50  0001 C CNN
 	1    9400 2700
@@
 F 0 "Q21" H 4750 1050 50  0000 C CNN
 F 1 "PFET_6A_GSD;SOT23" H 4900 650 50  0000 C CNN
-F 2 "HR2:POWER_PFET_GSD" H 4700 950 60  0001 L CNN
+F 2 "Package_TO_SOT_SMD:SOT-23" H 4700 950 60  0001 L CNN
 F 3 "Power PFG (GSD pinout)" H 4700 750 60  0001 L CNN
 F 4 "Power PFET (GSD pinout)" H 4700 650 60  0001 L CNN "Field5"
@@
 	1    0    0    -1
 $EndComp
+Wire Wire Line
+	4000 5500 4000 4500
+Wire Wire Line
+	4600 4700 4600 5900
+Wire Wire Line
+	3300 5200 3800 5200
+Connection ~ 3800 5200
+Wire Wire Line
+	3800 5200 3800 5900
+Wire Wire Line
+	2100 5900 3800 5900
 $EndSCHEMATC

Commit message: Imported footprints to PCB.
Parts:
- CN10: footprint Connector_PinHeader_2.54:PinHeader_2x06_P2.54mm_Vertical -> Connector_PinHeader_2.54mm:PinHeader_2x06_P2.54mm_Vertical
Changed lines of the file:
@@
 F 0 "CN10" H 9800 4750 50  0000 L CNN
 F 1 "WOW_OUT;M2x6S" H 9750 3350 50  0000 L CNN
-F 2 "Connector_PinHeader_2.54:PinHeader_2x06_P2.54mm_Vertical" H 9800 4650 60  0001 L CNN
+F 2 "Connector_PinHeader_2.54mm:PinHeader_2x06_P2.54mm_Vertical" H 9800 4650 60  0001 L CNN
 F 3 "WOW Output Connector" H 9800 4450 60  0001 L CNN
 F 4 "WOW Output Connector" H 9800 4350 60  0001 L CNN "Field5"
