File: electrical/master_board/rev_a/wowbus.sch (KiCad schematic (older format))
At the start: 26 parts, among them CN10 WOW_OUT;M2x6S, Q20 2N7000;SOT23, Q21 PFET_6A_GSD;SOT23, Q22 2N7000;SOT23, SW3 PUSH_BUTTON;6x6x9.5H, U13 74LVC1G11;6TSSOP, U14 LTV-827, U15 LTV-827, U16 74LVC1G74;TSSOP8, U17 LTV-827, U18 LTV-827

Commit message: Flipped Grove and Mikrobus connectors to the back side.
Parts:
- U14, U15: value LTV-827 -> MCP2542;SOIC8; footprint Package_DIP:DIP-8_W7.62mm -> Package_SO:SOIC-8_3.9x4.9mm_P1.27mm
- U17, U18: value LTV-827 -> LTV-827;SOIC8
Changed lines of the file:
@@
 $EndDescr
-$Comp
-L HR2:MCP2542;SOIC8 U14
-U 1 1 5F846C97
-P 5400 2200
-F 0 "U14" H 5650 2350 50  0000 C CNN
-F 1 "LTV-827" H 5950 1650 50  0000 C CNN
-F 2 "Package_DIP:DIP-8_W7.62mm" H 5600 2250 60  0001 L CNN
-F 3 "http://optoelectronics.liteon.com/upload/download/DS-70-96-0016/LTV-8X7%20series%20201610%20.pdf" H 5600 2050 60  0001 L CNN
-F 4 "MCP2542" H 5600 1950 60  0001 L CNN "Field5"
-	1    5400 2200
-	1    0    0    -1
-$EndComp
 $Comp
 L Isolator:LTV-827 U17
@@
 P 7400 1400
 F 0 "U17" H 7250 1600 50  0000 C CNN
-F 1 "LTV-827" H 7400 1200 50  0000 C CNN
+F 1 "LTV-827;SOIC8" H 7400 1200 50  0000 C CNN
 F 2 "Package_DIP:DIP-8_W7.62mm" H 7200 1200 50  0001 L CIN
 F 3 "http://optoelectronics.liteon.com/upload/download/DS-70-96-0016/LTV-8X7%20series%20201610%20.pdf" H 7400 1400 50  0001 L CNN
@@
 P 8400 1400
 F 0 "U18" H 8550 1200 50  0000 C CNN
-F 1 "LTV-827" H 8400 1600 50  0000 C CNN
+F 1 "LTV-827;SOIC8" H 8400 1600 50  0000 C CNN
 F 2 "Package_DIP:DIP-8_W7.62mm" H 8200 1200 50  0001 L CIN
 F 3 "http://optoelectronics.liteon.com/upload/download/DS-70-96-0016/LTV-8X7%20series%20201610%20.pdf" H 8400 1400 50  0001 L CNN
@@
 	1    0    0    -1
 $EndComp
-$Comp
-L HR2:MCP2542;SOIC8 U15
-U 1 1 5F8496E2
-P 5400 3900
-F 0 "U15" H 5650 4050 50  0000 C CNN
-F 1 "LTV-827" H 5950 3350 50  0000 C CNN
-F 2 "Package_DIP:DIP-8_W7.62mm" H 5600 3950 60  0001 L CNN
-F 3 "http://optoelectronics.liteon.com/upload/download/DS-70-96-0016/LTV-8X7%20series%20201610%20.pdf" H 5600 3750 60  0001 L CNN
-F 4 "MCP2542" H 5600 3650 60  0001 L CNN "Field5"
-	1    5400 3900
-	1    0    0    -1
-$EndComp
 Wire Wire Line
 	5300 2500 5300 2900
@@
 P 7400 3100
 F 0 "U17" H 7250 3300 50  0000 C CNN
-F 1 "LTV-827" H 7400 2900 50  0000 C CNN
+F 1 "LTV-827;SOIC8" H 7400 2900 50  0000 C CNN
 F 2 "Package_DIP:DIP-8_W7.62mm" H 7200 2900 50  0001 L CIN
 F 3 "http://optoelectronics.liteon.com/upload/download/DS-70-96-0016/LTV-8X7%20series%20201610%20.pdf" H 7400 3100 50  0001 L CNN
@@
 P 8400 3100
 F 0 "U18" H 8550 2900 50  0000 C CNN
-F 1 "LTV-827" H 8400 3300 50  0000 C CNN
+F 1 "LTV-827;SOIC8" H 8400 3300 50  0000 C CNN
 F 2 "Package_DIP:DIP-8_W7.62mm" H 8200 2900 50  0001 L CIN
 F 3 "http://optoelectronics.liteon.com/upload/download/DS-70-96-0016/LTV-8X7%20series%20201610%20.pdf" H 8400 3100 50  0001 L CNN
@@
 Wire Wire Line
 	2100 5900 3800 5900
+$Comp
+L HR2:MCP2542;SOIC8 U14
+U 1 1 5F9A7EB1
+P 5400 2200
+F 0 "U14" H 5650 2350 50  0000 C CNN
+F 1 "MCP2542;SOIC8" H 5950 1650 50  0000 C CNN
+F 2 "Package_SO:SOIC-8_3.9x4.9mm_P1.27mm" H 5600 2250 60  0001 L CNN
+F 3 "MCP2542 CAN Transceiver" H 5600 2050 60  0001 L CNN
+F 4 "MCP2542" H 5600 1950 60  0001 L CNN "Field5"
+	1    5400 2200
+	1    0    0    -1
+$EndComp
+$Comp
+L HR2:MCP2542;SOIC8 U15
+U 1 1 5F9AA16D
+P 5400 3900
+F 0 "U15" H 5650 4050 50  0000 C CNN
+F 1 "MCP2542;SOIC8" H 5950 3350 50  0000 C CNN
+F 2 "Package_SO:SOIC-8_3.9x4.9mm_P1.27mm" H 5600 3950 60  0001 L CNN
+F 3 "MCP2542 CAN Transceiver" H 5600 3750 60  0001 L CNN
+F 4 "MCP2542" H 5600 3650 60  0001 L CNN "Field5"
+	1    5400 3900
+	1    0    0    -1
+$EndComp
 $EndSCHEMATC

Commit message: Changing footprints and moving things around on the PCB.
Parts:
- removed U17, U18: LTV-827;SOIC8, Package_DIP:DIP-8_W7.62mm, symbol Isolator:LTV-827
- added U17, U18: CPC1017N;SOP4W3.8L4.1, Package_SO:SOP-4_3.8x4.1mm_P2.54mm, symbol HR2:CPC1017N;SOP4W3.8WL4.1
- CN10: footprint Connector_PinHeader_2.54mm:PinHeader_2x06_P2.54mm_Vertical -> HR2:PinHeader_2x06_P2.54mm_Vertical_Shrouded
- SW3: value PUSH_BUTTON;6x6x9.5H -> BUTTON;6x3.5; footprint Button_Switch_SMD:SW_SPST_PTS645 -> HR2:BUTTON_6x3.5
Connections:
- net labels removed: WOW_COM_TERM, WOW_ESTOP_TERM
- wire segments 191 -> 178
Other:
- note added: "Solid State Relay"
- note added: "https://www.ti.com/lit/ug/tiducf3/tiducf3.pdf"
- note removed: "Dual Opto-isolator"
- moved on the sheet: R59, R60, R61, R62
