File: electrical/master_board/rev_a/wowbus.sch (KiCad schematic (older format))
At the start: 33 parts, among them CN10 WOW_OUT;M2x6S, Q20 2N7000;SOT23, Q21 PFET_6A_GSD;SOT23, Q22 2N7000;SOT23, SW3 BUTTON;6x3.5, U13 74LVC1G11;SOT363, U14 MCP2542;SOIC8, U15 MCP2542;SOIC8, U16 74LVC1G74;TSSOP8, U17 CPC1017N;SOP4W3.8L4.1, U18 CPC1017N;SOP4W3.8L4.1

Commit message: Fixed the schematic DRC errors.
Parts:
- removed Q21: PFET_6A_GSD;SOT23, Package_TO_SOT_SMD:SOT-23, symbol HR2:POWER_PFET_GSD
- added Q21: PFET_6A;SOT23, symbol HR2_MISC:Q_PWR_PMOS_GSD
Connections:
- wire segments 199 -> 198
Changed lines of the file:
@@
 $Descr A 11000 8500
 encoding utf-8
-Sheet 8 10
+Sheet 7 10
 Title "HR2: WOWBus"
 Date "2020-11-22"
@@
 $EndComp
 Wire Wire Line
-	4500 1100 3800 1100
+	4200 1100 3800 1100
 Wire Wire Line
 	3800 1100 3800 1250
 Wire Wire Line
-	3800 1650 4400 1650
+	3800 1700 4400 1700
 Wire Wire Line
 	6900 2800 6500 2800
@@
 Connection ~ 7100 2400
 Wire Wire Line
-	4500 1200 4400 1200
-Wire Wire Line
-	4400 1200 4400 1650
+	4400 1400 4400 1700
 Text HLabel 1100 3200 0    50   Input ~ 0
 3.3V
@@
 $EndComp
 Wire Wire Line
-	3800 1650 3800 4000
+	3800 1700 3800 4000
 Text HLabel 1100 2500 0    50   Input ~ 0
 WOW_TX
@@
 Text Notes 5550 3900 0    50   ~ 0
 ESTOP CANBus Transceiver
-Text Notes 4550 900  0    50   ~ 0
+Text Notes 3700 850  0    50   ~ 0
 WOW Power P-FET (6A)
 Text Notes 5400 5000 0    50   ~ 0
@@
 WOW_STDBY
 Connection ~ 3400 4700
-Text Label 7900 1200 0    50   ~ 0
+Text Label 6800 1100 0    50   ~ 0
 WOW_POW_OUT
 Text Label 8700 3500 0    50   ~ 0
@@
 Connection ~ 2700 3200
 Wire Wire Line
-	3800 1650 3800 1550
-Connection ~ 3800 1650
+	3800 1700 3800 1550
+Connection ~ 3800 1700
 Connection ~ 4000 4700
 Wire Wire Line
@@
 Text Notes 4050 5100 0    50   ~ 0
 WOW Standby\nInverter
-Text Label 3800 1650 0    50   ~ 0
+Text Label 3800 1700 0    50   ~ 0
 ~WOW_EN
 $Comp
@@
 Wire Wire Line
 	9400 2900 9400 3000
-$Comp
-L HR2:POWER_PFET_GSD Q21
-U 1 1 5F9BEDD5
-P 4500 1100
-F 0 "Q21" H 4750 1250 50  0000 C CNN
-F 1 "PFET_6A_GSD;SOT23" H 4900 850 50  0000 C CNN
-F 2 "Package_TO_SOT_SMD:SOT-23" H 4700 1150 60  0001 L CNN
-F 3 "Power PFG (GSD pinout)" H 4700 950 60  0001 L CNN
-F 4 "Power PFET (GSD pinout)" H 4700 850 60  0001 L CNN "Field5"
-	1    4500 1100
-	1    0    0    -1
-$EndComp
 Wire Wire Line
 	4000 5700 4000 4700
@@
 TO DO:\n1. Add Test Points.\n
 Wire Wire Line
-	5600 800  5600 1200
-Wire Wire Line
-	5900 800  5600 800
-Wire Wire Line
-	6700 1200 6600 1200
-Wire Wire Line
-	6700 800  6700 1200
-Wire Wire Line
-	6300 800  6700 800
+	5600 700  5600 1100
+Wire Wire Line
+	5900 700  5600 700
+Wire Wire Line
+	6700 1100 6600 1100
+Wire Wire Line
+	6700 700  6700 1100
+Wire Wire Line
+	6300 700  6700 700
 $Comp
 L Jumper:Jumper_2_Open JP?
 U 1 1 5FB530EF
-P 6100 800
+P 6100 700
 AR Path="/5F52F39E/5FB530EF" Ref="JP?"  Part="1"
 AR Path="/5F8C2F57/5FB530EF" Ref="JP8"  Part="1"
-F 0 "JP8" H 5900 850 50  0000 C CNN
-F 1 "SHUNT;M1x2" H 6100 700 50  0000 C CNN
-F 2 "Connector_PinHeader_2.54mm:PinHeader_1x02_P2.54mm_Vertical" H 6100 800 50  0001 C CNN
-F 3 "~" H 6100 800 50  0001 C CNN
-	1    6100 800
-	1    0    0    -1
-$EndComp
-Wire Wire Line
-	5700 1200 5600 1200
-Connection ~ 5600 1200
-Wire Wire Line
-	6700 1200 9800 1200
-Connection ~ 6700 1200
-Wire Wire Line
-	5300 1200 5600 1200
-Wire Wire Line
-	9800 1200 9800 4400
+F 0 "JP8" H 5900 750 50  0000 C CNN
+F 1 "SHUNT;M1x2" H 6100 600 50  0000 C CNN
+F 2 "Connector_PinHeader_2.54mm:PinHeader_1x02_P2.54mm_Vertical" H 6100 700 50  0001 C CNN
+F 3 "~" H 6100 700 50  0001 C CNN
+	1    6100 700
+	1    0    0    -1
+$EndComp
+Wire Wire Line
+	5700 1100 5600 1100
+Connection ~ 5600 1100
+Wire Wire Line
+	6700 1100 9800 1100
+Connection ~ 6700 1100
+Wire Wire Line
+	9800 1100 9800 4400
 $Comp
 L Jumper:Jumper_2_Open JP7
@@
 L HR2:SHUNT R64
 U 1 1 5FD3322D
-P 5700 1200
-F 0 "R64" H 5950 1350 50  0000 C CNN
-F 1 "0Ω;1608" H 6150 1050 50  0000 C CNN
-F 2 "Resistor_SMD:R_0603_1608Metric" H 5900 1250 60  0001 L CNN
-F 3 "0 Ohm Power Shunt" H 5900 1050 60  0001 L CNN
-F 4 "0 Ohm Power Shunt" H 5900 950 60  0001 L CNN "Field5"
-	1    5700 1200
-	1    0    0    -1
-$EndComp
+P 5700 1100
+F 0 "R64" H 5950 1250 50  0000 C CNN
+F 1 "0Ω;1608" H 6150 950 50  0000 C CNN
+F 2 "Resistor_SMD:R_0603_1608Metric" H 5900 1150 60  0001 L CNN
+F 3 "0 Ohm Power Shunt" H 5900 950 60  0001 L CNN
+F 4 "0 Ohm Power Shunt" H 5900 850 60  0001 L CNN "Field5"
+	1    5700 1100
+	1    0    0    -1
+$EndComp
+$Comp
+L HR2_MISC:Q_PWR_PMOS_GSD Q21
+U 1 1 5FD48C48
+P 4400 1200
+F 0 "Q21" V 4300 1100 50  0000 C CNN
+F 1 "PFET_6A;SOT23" V 4651 1200 50  0000 C CNN
+F 2 "" H 4600 1300 50  0001 C CNN
+F 3 "~" H 4400 1200 50  0001 C CNN
+	1    4400 1200
+	0    1    -1   0
+$EndComp
+Wire Wire Line
+	4600 1100 5600 1100
 $EndSCHEMATC

Commit message: Moved Power Supply.
Parts:
- Q21: footprint (none) -> Package_TO_SOT_SMD:SOT-23
Changed lines of the file:
@@
 F 0 "Q21" V 4300 1100 50  0000 C CNN
 F 1 "PFET_6A;SOT23" V 4651 1200 50  0000 C CNN
-F 2 "" H 4600 1300 50  0001 C CNN
+F 2 "Package_TO_SOT_SMD:SOT-23" H 4600 1300 50  0001 C CNN
 F 3 "~" H 4400 1200 50  0001 C CNN
 	1    4400 1200

Commit message: Changed bypass caps and sonar echo outputs
Made following changes:
 - Changed bypass caps to 0.1uF
 - Removed voltage dividers on sonar echo outputs to Nucleo
Parts:
- C22, C23, C24, C25: value 10pF;1608 -> 0.1µF;1608
Changed lines of the file:
@@
 AR Path="/5F8C2F57/6036DBC8" Ref="C24"  Part="1"
 F 0 "C24" V 1450 4000 50  0000 L CNN
-F 1 "10pF;1608" V 1650 4250 50  0000 L CNN
+F 1 "0.1µF;1608" V 1650 4250 50  0000 L CNN
 F 2 "Capacitor_SMD:C_0603_1608Metric" H 1588 4050 50  0001 C CNN
 F 3 "~" H 1550 4200 50  0001 C CNN
@@
 AR Path="/5F8C2F57/60430375" Ref="C25"  Part="1"
 F 0 "C25" V 1450 4300 50  0000 L CNN
-F 1 "10pF;1608" V 1600 4550 50  0000 L CNN
+F 1 "0.1µF;1608" V 1600 4550 50  0000 L CNN
 F 2 "Capacitor_SMD:C_0603_1608Metric" H 1588 4350 50  0001 C CNN
 F 3 "~" H 1550 4500 50  0001 C CNN
@@
 AR Path="/5F8C2F57/6043088F" Ref="C23"  Part="1"
 F 0 "C23" V 1450 3700 50  0000 L CNN
-F 1 "10pF;1608" V 1600 3950 50  0000 L CNN
+F 1 "0.1µF;1608" V 1600 3950 50  0000 L CNN
 F 2 "Capacitor_SMD:C_0603_1608Metric" H 1588 3750 50  0001 C CNN
 F 3 "~" H 1550 3900 50  0001 C CNN
@@
 AR Path="/5F8C2F57/6057FE20" Ref="C22"  Part="1"
 F 0 "C22" V 1450 3400 50  0000 L CNN
-F 1 "10pF;1608" V 1600 3650 50  0000 L CNN
+F 1 "0.1µF;1608" V 1600 3650 50  0000 L CNN
 F 2 "Capacitor_SMD:C_0603_1608Metric" H 1588 3450 50  0001 C CNN
 F 3 "~" H 1550 3600 50  0001 C CNN

Commit message: Changed bypass caps size from 1608 to 1005
Parts:
- C22, C23, C24, C25: value 0.1µF;1608 -> 0.1µF;1005; footprint Capacitor_SMD:C_0603_1608Metric -> Capacitor_SMD:C_0402_1005Metric
Changed lines of the file:
@@
 AR Path="/5F8C2F57/6036DBC8" Ref="C24"  Part="1"
 F 0 "C24" V 1450 4000 50  0000 L CNN
-F 1 "0.1µF;1608" V 1650 4250 50  0000 L CNN
-F 2 "Capacitor_SMD:C_0603_1608Metric" H 1588 4050 50  0001 C CNN
+F 1 "0.1µF;1005" V 1650 4250 50  0000 L CNN
+F 2 "Capacitor_SMD:C_0402_1005Metric" H 1588 4050 50  0001 C CNN
 F 3 "~" H 1550 4200 50  0001 C CNN
 	1    1550 4200
@@
 AR Path="/5F8C2F57/60430375" Ref="C25"  Part="1"
 F 0 "C25" V 1450 4300 50  0000 L CNN
-F 1 "0.1µF;1608" V 1600 4550 50  0000 L CNN
-F 2 "Capacitor_SMD:C_0603_1608Metric" H 1588 4350 50  0001 C CNN
+F 1 "0.1µF;1005" V 1600 4550 50  0000 L CNN
+F 2 "Capacitor_SMD:C_0402_1005Metric" H 1588 4350 50  0001 C CNN
 F 3 "~" H 1550 4500 50  0001 C CNN
 	1    1550 4500
@@
 AR Path="/5F8C2F57/6043088F" Ref="C23"  Part="1"
 F 0 "C23" V 1450 3700 50  0000 L CNN
-F 1 "0.1µF;1608" V 1600 3950 50  0000 L CNN
-F 2 "Capacitor_SMD:C_0603_1608Metric" H 1588 3750 50  0001 C CNN
+F 1 "0.1µF;1005" V 1600 3950 50  0000 L CNN
+F 2 "Capacitor_SMD:C_0402_1005Metric" H 1588 3750 50  0001 C CNN
 F 3 "~" H 1550 3900 50  0001 C CNN
 	1    1550 3900
@@
 AR Path="/5F8C2F57/6057FE20" Ref="C22"  Part="1"
 F 0 "C22" V 1450 3400 50  0000 L CNN
-F 1 "0.1µF;1608" V 1600 3650 50  0000 L CNN
-F 2 "Capacitor_SMD:C_0603_1608Metric" H 1588 3450 50  0001 C CNN
+F 1 "0.1µF;1005" V 1600 3650 50  0000 L CNN
+F 2 "Capacitor_SMD:C_0402_1005Metric" H 1588 3450 50  0001 C CNN
 F 3 "~" H 1550 3600 50  0001 C CNN
 	1    1550 3600

Commit message: Changed more parts to 1005 size and R9 value
Parts:
- R53, R54, R55, R56: value 100KΩ;1608 -> 100KΩ;1005; footprint Resistor_SMD:R_0603_1608Metric -> Resistor_SMD:R_0402_1005Metric
Changed lines of the file:
@@
 P 3800 1400
 F 0 "R55" H 3650 1500 50  0000 L CNN
-F 1 "100KΩ;1608" H 3850 1300 50  0000 L CNN
-F 2 "Resistor_SMD:R_0603_1608Metric" V 3840 1390 50  0001 C CNN
+F 1 "100KΩ;1005" H 3850 1300 50  0000 L CNN
+F 2 "Resistor_SMD:R_0402_1005Metric" V 3840 1390 50  0001 C CNN
 F 3 "~" H 3800 1400 50  0001 C CNN
 	1    3800 1400
@@
 P 4000 5850
 F 0 "R56" H 3850 5950 50  0000 L CNN
-F 1 "100KΩ;1608" H 4000 5700 50  0000 L CNN
-F 2 "Resistor_SMD:R_0603_1608Metric" V 4040 5840 50  0001 C CNN
+F 1 "100KΩ;1005" H 4000 5700 50  0000 L CNN
+F 2 "Resistor_SMD:R_0402_1005Metric" V 4040 5840 50  0001 C CNN
 F 3 "~" H 4000 5850 50  0001 C CNN
 	1    4000 5850
@@
 P 2200 3450
 F 0 "R53" H 2050 3550 50  0000 L CNN
-F 1 "100KΩ;1608" H 2200 3300 50  0000 L CNN
-F 2 "Resistor_SMD:R_0603_1608Metric" V 2240 3440 50  0001 C CNN
+F 1 "100KΩ;1005" H 2200 3300 50  0000 L CNN
+F 2 "Resistor_SMD:R_0402_1005Metric" V 2240 3440 50  0001 C CNN
 F 3 "~" H 2200 3450 50  0001 C CNN
 	1    2200 3450
@@
 P 2700 3450
 F 0 "R54" H 2550 3550 50  0000 L CNN
-F 1 "100KΩ;1608" H 2700 3300 50  0000 L CNN
-F 2 "Resistor_SMD:R_0603_1608Metric" V 2740 3440 50  0001 C CNN
+F 1 "100KΩ;1005" H 2700 3300 50  0000 L CNN
+F 2 "Resistor_SMD:R_0402_1005Metric" V 2740 3440 50  0001 C CNN
 F 3 "~" H 2700 3450 50  0001 C CNN
 	1    2700 3450

Commit message: Updated WOWBus portion of schematic.
Parts:
- removed U13: 74LVC1G11;SOT363, Package_TO_SOT_SMD:SOT-363_SC-70-6, symbol HR2:74LVC1G11;SOT363
- added U13, U22: 74x11G1, symbol HR2_MISC:74x11G1
- R59, R60: value 120Ω1/4W;1608 -> 120Ω.25W;1608
- TP14: value ~ESTOP_CLR -> ~nESTOP_SET
- TP15: value ESTOP_TRIG;M1x1 -> ~nWOW_ESTOP;M1x1
Connections:
- net labels added: ESTOP_CLR, ~NBTN_ESTOP, ~NESTOP, ~NESTOP_SET, ~NHBTN_ESTOP, ~NHR2_ESTOP, ~NMOTOR_FAULT, ~NWOW_EN, ~NWOW_ESTOP
- net labels removed: ESTOP, ESTOP_TRIG, ~ESTOP, ~ESTOP_CLR, ~ESTOP_SET, ~MOTOR_FAULT, ~WOW_EN
- wire segments 198 -> 214
- no-connect marks 0 -> 1
Other:
- note added: "AND Gate\nPower Pins"
- note added: "E-Stop AND Gate"
- note added: "External\nE-Stop\nButton"
- note added: "Filter Capacitors"
- note removed: "Bypass Capacitors"
- moved on the sheet: C22, C23, C24, C25, D3, R53, R54, R55, R56, R57, R58, R59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

Commit message: Got Schematic and PCB syncronized again.
Parts:
- U13, U22: value 74x11G1 -> 74x11G1;TSOP6; footprint (none) -> Package_SO:TSOP-6_1.65x3.05mm_P0.95mm
Changed lines of the file:
@@
 U 1 1 5FC61F4D
 P 2800 4350
-F 0 "R53" H 2650 4450 50  0000 L CNN
+F 0 "R53" H 2650 4500 50  0000 L CNN
 F 1 "100KΩ;1005" H 2300 4200 50  0000 L CNN
 F 2 "Resistor_SMD:R_0402_1005Metric" V 2840 4340 50  0001 C CNN
@@
 P 3500 5300
 F 0 "U13" H 3500 5625 50  0000 C CNN
-F 1 "74x11G1" H 3500 5534 50  0000 C CNN
-F 2 "" H 3500 5300 50  0001 C CNN
+F 1 "74x11G1;TSOP6" H 3500 5534 50  0000 C CNN
+F 2 "Package_SO:TSOP-6_1.65x3.05mm_P0.95mm" H 3500 5300 50  0001 C CNN
 F 3 "http://www.ti.com/lit/gpn/sn74LS11" H 3500 5300 50  0001 C CNN
 	1    3500 5300
@@
 U 4 2 5FD5FD90
 P 1900 3800
-F 0 "U13" H 1800 3950 50  0000 C CNN
-F 1 "74x11G1" H 1900 3650 50  0000 C CNN
-F 2 "" H 1900 3800 50  0001 C CNN
+F 0 "U13" H 2000 3950 50  0000 C CNN
+F 1 "74x11G1;TSOP6" H 1850 3650 50  0000 C CNN
+F 2 "Package_SO:TSOP-6_1.65x3.05mm_P0.95mm" H 1900 3800 50  0001 C CNN
 F 3 "http://www.ti.com/lit/gpn/sn74LS11" H 1900 3800 50  0001 C CNN
 	4    1900 3800
-	1    0    0    -1
+	-1   0    0    -1
 $EndComp
 Wire Wire Line
@@
 P 2600 2800
 F 0 "U22" H 2800 2700 50  0000 C CNN
-F 1 "74x11G1" H 2600 3000 50  0000 C CNN
-F 2 "" H 2600 2800 50  0001 C CNN
+F 1 "74x11G1;TSOP6" H 2600 3000 50  0000 C CNN
+F 2 "Package_SO:TSOP-6_1.65x3.05mm_P0.95mm" H 2600 2800 50  0001 C CNN
 F 3 "http://www.ti.com/lit/gpn/sn74LS11" H 2600 2800 50  0001 C CNN
 	1    2600 2800
@@
 	3000 4100 3000 3200
 Wire Wire Line
-	1400 3200 2400 3200
-Wire Wire Line
 	1500 3800 1400 3800
 Connection ~ 1400 3800
@@
 Wire Wire Line
 	2400 3800 2400 3400
-Connection ~ 2400 3200
-Wire Wire Line
-	2400 3200 3000 3200
 Wire Wire Line
 	2300 3400 2400 3400
-Connection ~ 2400 3400
-Wire Wire Line
-	2400 3400 2400 3200
 $Comp
 L HR2_MISC:74x11G1 U22
@@
 P 1900 3400
 F 0 "U22" H 2000 3250 50  0000 C CNN
-F 1 "74x11G1" H 1900 3550 50  0000 C CNN
-F 2 "" H 1900 3400 50  0001 C CNN
+F 1 "74x11G1;TSOP6" H 1850 3550 50  0000 C CNN
+F 2 "Package_SO:TSOP-6_1.65x3.05mm_P0.95mm" H 1900 3400 50  0001 C CNN
 F 3 "http://www.ti.com/lit/gpn/sn74LS11" H 1900 3400 50  0001 C CNN
 	4    1900 3400
@@
 Text Notes 3050 5750 0    50   ~ 0
 External\nE-Stop\nButton
+Wire Wire Line
+	1400 3200 3000 3200
+Wire Wire Line
+	2200 4100 2400 4100
+Wire Wire Line
+	2400 4100 2400 3800
+Connection ~ 2200 4100
+Connection ~ 2400 3800
 $EndSCHEMATC

Commit message: JLCPCB BOM is in better shape.
Parts:
- removed Q20, Q22: 2N7000;SOT23, Package_TO_SOT_SMD:SOT-23, symbol Transistor_FET:2N7000
- added Q20, Q22: 2N7002;SOT23, Package_TO_SOT_SMD:SOT-23, symbol Transistor_FET:2N7002
- Q21: value PFET_6A;SOT23 -> PFET_6A_GSD;SOT23
Changed lines of the file:
@@
-	1    0    0    -1
-$EndComp
-$Comp
-L Transistor_FET:2N7000 Q?
-U 1 1 5F9A0944
-P 3800 4200
-AR Path="/5F79BC00/5F9A0944" Ref="Q?"  Part="1"
-AR Path="/5FA4A874/5F9A0944" Ref="Q?"  Part="1"
-AR Path="/5FAD82EE/5F9A0944" Ref="Q?"  Part="1"
-AR Path="/5F8C2F57/5F9A0944" Ref="Q20"  Part="1"
-F 0 "Q20" H 3700 4350 50  0000 L CNN
-F 1 "2N7000;SOT23" H 3950 4050 50  0000 L CNN
-F 2 "Package_TO_SOT_SMD:SOT-23" H 4000 4125 50  0001 L CIN
-F 3 "https://www.fairchildsemi.com/datasheets/2N/2N7000.pdf" H 3800 4200 50  0001 L CNN
-	1    3800 4200
 	1    0    0    -1
 $EndComp
@@
 Wire Wire Line
 	5400 4300 5500 4300
-Wire Wire Line
-	4700 3600 4700 4400
 Connection ~ 4700 4400
 Wire Wire Line
@@
 Wire Wire Line
 	4700 4400 4700 4500
-$Comp
-L Transistor_FET:2N7000 Q?
-U 1 1 5F86962A
-P 4600 4700
-AR Path="/5F79BC00/5F86962A" Ref="Q?"  Part="1"
-AR Path="/5FA4A874/5F86962A" Ref="Q?"  Part="1"
-AR Path="/5FAD82EE/5F86962A" Ref="Q?"  Part="1"
-AR Path="/5F8C2F57/5F86962A" Ref="Q22"  Part="1"
-F 0 "Q22" H 4500 4850 50  0000 L CNN
-F 1 "2N7000;SOT23" H 4100 4500 50  0000 L CNN
-F 2 "Package_TO_SOT_SMD:SOT-23" H 4800 4625 50  0001 L CIN
-F 3 "https://www.fairchildsemi.com/datasheets/2N/2N7000.pdf" H 4600 4700 50  0001 L CNN
-	1    4600 4700
-	1    0    0    -1
-$EndComp
 Wire Wire Line
 	4700 3200 6900 3200
@@
 Text Notes 3950 4000 0    50   ~ 0
 3.3 to 9V\nLevel Shift
-Text Notes 4750 5000 0    50   ~ 0
+Text Notes 4750 5050 0    50   ~ 0
 WOW Standby\nInverter
 Text Label 3900 2000 0    50   ~ 0
@@
 P 4500 1200
 F 0 "Q21" V 4400 1100 50  0000 C CNN
-F 1 "PFET_6A;SOT23" V 4751 1200 50  0000 C CNN
+F 1 "PFET_6A_GSD;SOT23" V 4751 1200 50  0000 C CNN
 F 2 "Package_TO_SOT_SMD:SOT-23" H 4700 1300 50  0001 C CNN
 F 3 "~" H 4500 1200 50  0001 C CNN
@@
 Connection ~ 2200 4100
 Connection ~ 2400 3800
+$Comp
+L Transistor_FET:2N7002 Q20
+U 1 1 5FE8B140
+P 3800 4200
+F 0 "Q20" H 3650 4350 50  0000 L CNN
+F 1 "2N7002;SOT23" H 3950 4100 50  0000 L CNN
+F 2 "Package_TO_SOT_SMD:SOT-23" H 4000 4125 50  0001 L CIN
+F 3 "https://www.onsemi.com/pub/Collateral/NDS7002A-D.PDF" H 3800 4200 50  0001 L CNN
+	1    3800 4200
+	1    0    0    -1
+$EndComp
+Wire Wire Line
+	4700 3600 4700 4400
+$Comp
+L Transistor_FET:2N7002 Q22
+U 1 1 5FE90DD1
+P 4600 4700
+F 0 "Q22" H 4450 4850 50  0000 L CNN
+F 1 "2N7002;SOT23" H 4750 4600 50  0000 L CNN
+F 2 "Package_TO_SOT_SMD:SOT-23" H 4800 4625 50  0001 L CIN
+F 3 "https://www.onsemi.com/pub/Collateral/NDS7002A-D.PDF" H 4600 4700 50  0001 L CNN
+	1    4600 4700
+	1    0    0    -1
+$EndComp
 $EndSCHEMATC
