File: electrical/master_board/rev_a/connectors.sch (KiCad schematic (older format))
At the start: 9 parts, among them CN5 LIDAR_ADAPTER;2xF1x3+F1x2, CN88 MIKROBUS_MATE;SMALL, CN89 MIKROBUS_MATE;MEDIUM, U5 SN74HCS595;TTSOP16, U6 SN74HCS166;TTSOP16, U7 SN74HCS166;TTSOP16

Commit message: More work thinning rats nest of unconnected wires.
Other:
- note added: "TO DO:\n1. Add test points.\n2. Add edge sense connectors.\n3. Add Grove connectors.\n4. Add a button."
Changed lines of the file:
@@
 	4600 1900 4600 2000
 Entry Wire Line
-	4100 1400 4000 1300
-Entry Wire Line
-	6300 1400 6200 1300
+	6300 1350 6200 1250
 $Comp
 L Device:C C?
@@
 	5200 2000 5800 2000
 Wire Wire Line
-	4400 1500 4400 1400
+	4400 1500 4400 1350
 Wire Wire Line
 	5800 2000 6300 2000
 Wire Wire Line
-	6300 2000 6300 1400
+	6300 2000 6300 1350
 Connection ~ 5800 2000
 Text Notes 4900 1450 0    50   ~ 0
@@
 Wire Wire Line
 	4400 5500 4400 5100
+Text Notes 3900 1150 0    80   ~ 0
+TO DO:\n1. Add test points.\n2. Add edge sense connectors.\n3. Add Grove connectors.\n4. Add a button.
+Entry Wire Line
+	4400 1350 4300 1250
 Wire Wire Line
 	4600 6500 8100 6500
@@
 	7400 6100 7400 6400
 Wire Bus Line
-	2400 1300 10300 1300
+	2400 1250 10300 1250
+Wire Bus Line
+	2400 800  2400 1250
 Wire Bus Line
 	4700 6400 4700 7700
 Wire Bus Line
-	2400 800  2400 1300
-Wire Bus Line
-	10300 1300 10300 6400
+	10300 1250 10300 6400
 Wire Bus Line
 	7250 1700 7250 6600

Commit message: PCB Complete (for now).
Parts:
- added CN11, CN12, CN13, CN14, CN15, CN16, CN17, CN4: SENSE;M1x3, Connector_PinHeader_2.54mm:PinHeader_1x03_P2.54mm_Vertical, symbol HR2:SENSE;M1x3
Connections:
- net labels added: SIG1, SIG2, SIG3, SIG4, SIG5, SIG6, SIG7, SIG8
- wire segments 157 -> 183
Other:
- note added: "Note: The 8 extra input pins on U& that are currently unused."
- note removed: "Note: There are many extra input pins. Most of these will be assigned\nto Grove connectors and edge detectors."
- note removed: "TO DO:\n1. Add test points.\n2. Add edge sense connectors.\n3. Add Grove connectors.\n4. Add a button."
- note removed: "Temporarily\nGround Inputs"
- moved on the sheet: C14, C15, C16
