File: electrical/master_board/rev_a/connectors.sch (KiCad schematic (older format))
At the start: 17 parts, among them CN11 SENSE;M1x3, CN12 SENSE;M1x3, CN13 SENSE;M1x3, CN14 SENSE;M1x3, CN15 SENSE;M1x3, CN16 SENSE;M1x3, CN17 SENSE;M1x3, CN4 SENSE;M1x3, CN5 LIDAR_ADAPTER;2xF1x3+F1x2, CN88 MIKROBUS_MATE;SMALL, CN89 MIKROBUS_MATE;MEDIUM, U5 SN74HCS595;TTSOP16, U6 SN74HCS166;TTSOP16, U7 SN74HCS166;TTSOP16

Commit message: Fixed SPI shift registers (good find by James Nugen\!)
Changed lines of the file:
@@
 INT0
 NoConn ~ 4500 4600
-NoConn ~ 3900 7300
 NoConn ~ 3900 7100
 NoConn ~ 3900 7000
@@
 	10100 3200 10300 3200
 Wire Wire Line
-	3900 7200 4600 7200
-Wire Wire Line
 	8800 3600 8100 3600
 Wire Wire Line
@@
 Text Label 8100 5800 0    50   ~ 0
 ~DIO_NSS
-Text Label 3900 7200 0    50   ~ 0
+Text Label 3900 7300 0    50   ~ 0
 SER_OUT_TO_IN1
 Text Label 9050 4050 0    50   ~ 0
@@
 Text Label 2250 6900 0    50   ~ 0
 ~DIO_NSS
-Wire Wire Line
-	4600 7200 4600 6600
 Wire Wire Line
 	10100 1700 8100 1700
@@
 Text Label 7300 5500 0    50   ~ 0
 SIG8
+Wire Wire Line
+	3900 7300 4600 7300
+Wire Wire Line
+	4600 6600 4600 7300
+NoConn ~ 3900 7200
 Wire Bus Line
 	8100 6100 8100 6400

Commit message: Switched from x166 to x165 shift registers.  Add bin/spi_sim.py.
Parts:
- removed U6, U7: SN74HCS166;TTSOP16, Package_SO:TSSOP-16_4.4x5mm_P0.65mm, symbol HR2:SN74HCS166;TTSOP16
- added U6, U7: SN74HCS165;TTSOP16, Package_SO:TSSOP-16_4.4x5mm_P0.65mm, symbol HR2:SN74HCS165;TTSOP16
Connections:
- net labels added: DIO_IN_BRIDGE, DIO_OUT_TO_IN, DIO_SS
- net labels removed: SER_IN1_TO_IN2, SER_OUT_TO_IN1
- wire segments 183 -> 177
- no-connect marks 44 -> 46
Changed lines of the file:
@@
 $Descr A 11000 8500
 encoding utf-8
-Sheet 6 10
+Sheet 10 10
 Title "HR2 Connectors"
 Date "2020-11-22"
@@
 Entry Wire Line
 	5900 5500 6000 5600
-$Comp
-L HR2:SN74HCS166;TTSOP16 U6
-U 1 1 5F845F8F
-P 8800 2500
-F 0 "U6" H 9050 2650 60  0000 C CNN
-F 1 "SN74HCS166;TTSOP16" H 9400 1150 60  0000 C CNN
-F 2 "Package_SO:TSSOP-16_4.4x5mm_P0.65mm" H 9000 2550 60  0001 L CNN
-F 3 "8-Bit Parallel In Serial Out Shift Register" H 9000 2350 60  0001 L CNN
-F 4 "8-Bit Parallel In Serial Out Shift Register" H 9000 2250 60  0001 L CNN "Field5"
-	1    8800 2500
-	1    0    0    -1
-$EndComp
-$Comp
-L HR2:SN74HCS166;TTSOP16 U7
-U 1 1 5F849624
-P 8800 4700
-F 0 "U7" H 9050 4850 60  0000 C CNN
-F 1 "SN74HCS166;TTSOP16" H 9400 3350 60  0000 C CNN
-F 2 "Package_SO:TSSOP-16_4.4x5mm_P0.65mm" H 9000 4750 60  0001 L CNN
-F 3 "8-Bit Parallel In Serial Out Shift Register" H 9000 4550 60  0001 L CNN
-F 4 "8-Bit Parallel In Serial Out Shift Register" H 9000 4450 60  0001 L CNN "Field5"
-	1    8800 4700
-	1    0    0    -1
-$EndComp
-Wire Wire Line
-	8600 5500 8800 5500
-Wire Wire Line
-	10000 5300 10100 5300
-Wire Wire Line
-	10100 5300 10100 4050
-Wire Wire Line
-	10100 4050 8600 4050
-Wire Wire Line
-	8600 4050 8600 3300
-Wire Wire Line
-	8600 3300 8800 3300
-Wire Wire Line
-	10000 3100 10100 3100
-Wire Wire Line
-	10100 3100 10100 1700
-Wire Wire Line
-	8800 4700 8500 4700
+Wire Wire Line
+	9900 5200 10100 5200
+Wire Wire Line
+	10100 5200 10100 4050
+Wire Wire Line
+	10100 4050 8700 4050
+Wire Wire Line
+	8700 4050 8700 3300
+Wire Wire Line
+	8700 3300 8900 3300
+Wire Wire Line
+	9900 3000 10100 3000
+Wire Wire Line
+	10100 3000 10100 1700
+Wire Wire Line
+	8900 4700 8500 4700
 Wire Wire Line
 	8500 4700 8500 4800
 Wire Wire Line
-	8500 5400 8800 5400
-Wire Wire Line
-	8800 5300 8500 5300
+	8500 5400 8900 5400
+Wire Wire Line
+	8900 5300 8500 5300
 Connection ~ 8500 5300
 Wire Wire Line
 	8500 5300 8500 5400
 Wire Wire Line
-	8800 5200 8500 5200
+	8900 5200 8500 5200
 Connection ~ 8500 5200
 Wire Wire Line
 	8500 5200 8500 5300
 Wire Wire Line
-	8800 5100 8500 5100
+	8900 5100 8500 5100
 Connection ~ 8500 5100
 Wire Wire Line
 	8500 5100 8500 5200
 Wire Wire Line
-	8800 5000 8500 5000
+	8900 5000 8500 5000
 Connection ~ 8500 5000
 Wire Wire Line
 	8500 5000 8500 5100
 Wire Wire Line
-	8800 4900 8500 4900
+	8900 4900 8500 4900
 Connection ~ 8500 4900
 Wire Wire Line
 	8500 4900 8500 5000
 Wire Wire Line
-	8800 4800 8500 4800
+	8900 4800 8500 4800
 Connection ~ 8500 4800
 Wire Wire Line
 	8500 4800 8500 4900
-Text Label 8200 6100 0    50   ~ 0
-~NRST
-Entry Wire Line
-	8200 6100 8100 6200
-Wire Wire Line
-	8200 6100 8500 6100
-Entry Wire Line
-	10300 3000 10400 3100
+Entry Wire Line
+	10300 2900 10400 3000
 Entry Wire Line
 	10300 3200 10400 3300
 Entry Wire Line
-	10300 5200 10400 5300
+	10300 5100 10400 5200
 Entry Wire Line
 	10300 5400 10400 5500
 Wire Wire Line
-	10000 5200 10300 5200
-Wire Wire Line
-	10000 5400 10100 5400
-Wire Wire Line
-	10000 3200 10100 3200
-Wire Wire Line
-	10000 3000 10300 3000
+	9900 5100 10300 5100
+Wire Wire Line
+	9900 5400 10100 5400
+Wire Wire Line
+	9900 2900 10300 2900
 Text Label 10300 3200 2    50   ~ 0
 GND
-Text Label 10300 3000 2    50   ~ 0
+Text Label 10300 2900 2    50   ~ 0
 3.3V
 Text Label 10300 5400 2    50   ~ 0
 GND
-Text Label 10300 5200 2    50   ~ 0
-3.3V
-Wire Wire Line
-	8400 3700 8800 3700
-Connection ~ 8100 6400
-Wire Bus Line
-	8100 6400 10400 6400
-Wire Wire Line
-	8400 3700 8400 5500
-Wire Wire Line
-	8800 5900 8500 5900
-Wire Wire Line
-	8500 5900 8500 6100
+Text Label 10300 5100 2    50   ~ 0
+3.3V
 Connection ~ 8500 4700
 Entry Wire Line
-	8100 5800 8000 5900
-Entry Wire Line
 	8100 5700 8000 5800
-Wire Wire Line
-	8700 6200 10100 6200
-Wire Wire Line
-	10100 6200 10100 5400
+Entry Wire Line
+	8100 5600 8000 5700
+Wire Wire Line
+	8800 6100 10100 6100
+Wire Wire Line
+	10100 6100 10100 5400
 Connection ~ 10100 5400
 Wire Wire Line
 	10100 5400 10300 5400
 Wire Wire Line
-	8100 5800 8800 5800
-Wire Wire Line
-	8100 5700 8800 5700
-Wire Wire Line
-	8800 5600 8700 5600
-Wire Wire Line
-	8700 5600 8700 6200
-Wire Wire Line
-	8800 3400 8700 3400
-Wire Wire Line
-	8700 3400 8700 3950
-Wire Wire Line
-	8700 3950 10100 3950
+	8100 5700 8900 5700
+Wire Wire Line
+	8900 3600 8800 3600
+Wire Wire Line
+	8800 3600 8800 3950
+Wire Wire Line
+	8800 3950 10100 3950
 Wire Wire Line
 	10100 3950 10100 3200
@@
 	10100 3200 10300 3200
 Wire Wire Line
-	8800 3600 8100 3600
-Wire Wire Line
-	8100 3500 8800 3500
+	8900 3400 8100 3400
+Wire Wire Line
+	8100 3500 8900 3500
 Entry Wire Line
 	8000 3600 8100 3500
 Entry Wire Line
-	8000 3700 8100 3600
+	8000 3500 8100 3400
 Text Label 8100 3500 0    50   ~ 0
 DIO_SCK
+Text Label 8100 5600 0    50   ~ 0
+DIO_SCK
+Text Label 8100 3400 0    50   ~ 0
+DIO_SS
 Text Label 8100 5700 0    50   ~ 0
-DIO_SCK
-Text Label 8100 3600 0    50   ~ 0
-~DIO_NSS
-Text Label 8100 5800 0    50   ~ 0
-~DIO_NSS
-Text Label 3900 7300 0    50   ~ 0
-SER_OUT_TO_IN1
+DIO_SS
 Text Label 9050 4050 0    50   ~ 0
-SER_IN1_TO_IN2
+DIO_IN_BRIDGE
 Wire Wire Line
 	8500 4250 10300 4250
@@
 Text Notes 8600 2250 0    50   ~ 0
 8-Bit Parallel to\nSerial Shift Register
-Text Notes 8650 4450 0    50   ~ 0
+Text Notes 8550 4450 0    50   ~ 0
 8-Bit Parallel to\nSerial Shift Register
 Wire Wire Line
@@
 Entry Wire Line
 	3900 1350 3800 1250
-Wire Wire Line
-	8400 5500 8500 5500
-Wire Wire Line
-	8500 5500 8500 5900
-Connection ~ 8500 5900
 $Comp
 L HR2:SENSE;M1x3 CN4
@@
 	7900 5500 7900 3200
 Wire Wire Line
-	7900 3200 8800 3200
-Wire Wire Line
 	7300 5000 7800 5000
 Wire Wire Line
 	7800 5000 7800 3100
 Wire Wire Line
-	7800 3100 8800 3100
-Wire Wire Line
 	7300 4500 7700 4500
 Wire Wire Line
 	7700 4500 7700 3000
 Wire Wire Line
-	7700 3000 8800 3000
+	7700 3000 8900 3000
 Wire Wire Line
 	7300 4000 7600 4000
@@
 	7600 4000 7600 2900
 Wire Wire Line
-	7600 2900 8800 2900
+	7600 2900 8900 2900
 Wire Wire Line
 	7300 3500 7500 3500
@@
 	7500 3500 7500 2800
 Wire Wire Line
-	7500 2800 8800 2800
+	7500 2800 8900 2800
 Wire Bus Line
 	4850 6700 8000 6700
-Wire Bus Line
-	6000 6400 8100 6400
 Connection ~ 6000 6400
 Wire Bus Line
@@
 	7400 3000 7400 2700
 Wire Wire Line
-	7400 2700 8800 2700
+	7400 2700 8900 2700
 Wire Wire Line
 	7400 2600 7400 2500
@@
 	7400 2500 7300 2500
 Wire Wire Line
-	7400 2600 8800 2600
+	7400 2600 8900 2600
 Wire Wire Line
 	7500 2500 7500 2000
@@
 	7500 2000 7300 2000
 Wire Wire Line
-	7500 2500 8800 2500
-Wire Wire Line
-	4600 6600 8600 6600
-Wire Wire Line
-	8600 5500 8600 6600
+	7500 2500 8900 2500
 Text Label 7300 2000 0    50   ~ 0
 SIG1
@@
 Text Label 7300 5500 0    50   ~ 0
 SIG8
+NoConn ~ 3900 7200
+Text HLabel 1500 7650 0    50   Input ~ 0
+DIO_SS
+Entry Wire Line
+	2050 7650 2150 7750
+Wire Wire Line
+	1500 7650 2050 7650
+Text Label 1500 7650 0    50   ~ 0
+DIO_SS
+$Comp
+L HR2:SN74HCS165;TTSOP16 U7
+U 1 1 5FC4FA21
+P 8900 4700
+F 0 "U7" H 9150 4850 50  0000 C CNN
+F 1 "SN74HCS165;TTSOP16" H 9400 3450 50  0000 C CNN
+F 2 "Package_SO:TSSOP-16_4.4x5mm_P0.65mm" H 9100 4750 60  0001 L CNN
+F 3 "8-Bit Parallel In Serial Out Shift Register" H 9100 4550 60  0001 L CNN
+F 4 "8-Bit Parallel In Serial Out Shift Register" H 9100 4450 60  0001 L CNN "desc"
+	1    8900 4700
+	1    0    0    -1
+$EndComp
+Wire Wire Line
+	9900 3200 10100 3200
+Wire Wire Line
+	7900 3200 8900 3200
+Wire Wire Line
+	7800 3100 8900 3100
+NoConn ~ 9900 3100
+Wire Bus Line
+	6000 6400 10400 6400
+Text Label 3900 7300 0    50   ~ 0
+DIO_OUT_TO_IN
 Wire Wire Line
 	3900 7300 4600 7300
 Wire Wire Line
 	4600 6600 4600 7300
-NoConn ~ 3900 7200
-Wire Bus Line
-	8100 6100 8100 6400
+Wire Wire Line
+	4600 6600 8600 6600
+Wire Wire Line
+	8600 5500 8900 5500
+Wire Wire Line
+	8600 5500 8600 6600
+Wire Wire Line
+	8100 5600 8900 5600
+Wire Wire Line
+	8900 5800 8800 5800
+Wire Wire Line
+	8800 5800 8800 6100
+NoConn ~ 9900 5300
 Wire Bus Line
 	2400 1250 6000 1250
 Wire Bus Line
+	4700 6400 4700 7700
+Wire Bus Line
 	2400 800  2400 1250
 Wire Bus Line
-	4700 6400 4700 7700
-Wire Bus Line
 	10400 1250 10400 6400
 Wire Bus Line
@@
 Wire Bus Line
 	6000 1250 6000 6400
+$Comp
+L HR2:SN74HCS165;TTSOP16 U6
+U 1 1 5FC4EDF6
+P 8900 2500
+F 0 "U6" H 9150 2650 50  0000 C CNN
+F 1 "SN74HCS165;TTSOP16" H 9400 1250 50  0000 C CNN
+F 2 "Package_SO:TSSOP-16_4.4x5mm_P0.65mm" H 9100 2550 60  0001 L CNN
+F 3 "8-Bit Parallel In Serial Out Shift Register" H 9100 2350 60  0001 L CNN
+F 4 "8-Bit Parallel In Serial Out Shift Register" H 9100 2250 60  0001 L CNN "desc"
+	1    8900 2500
+	1    0    0    -1
+$EndComp
 $EndSCHEMATC

Commit message: Change to sch and pcb
    Made following changes:
     - Remove Mikrobus connectors from sch and pcb
     - Change board to 4 layers
     - Add GND layer
     - Add 5V layer
     - Add 3.3V zone to 5V layer (experiment)
Parts:
- removed CN88: MIKROBUS_MATE;SMALL, HR2:MIKROBUS_SMALL_MATE, symbol HR2:MIKROBUS_MATE;SMALL
- removed CN89: MIKROBUS_MATE;MEDIUM, HR2:MIKROBUS_MEDIUM_MATE, symbol HR2:MIKROBUS_MATE;MEDIUM
- added Q?: 2N7000;SOT23, Package_TO_SOT_SMD:SOT-23, symbol Transistor_FET:2N7000
- added R?: 100KΩ;1608, Resistor_SMD:R_0603_1608Metric, symbol Device:R_US
Connections:
- net labels removed: A0, A1, A4_SDA, A5_SCL, D0_RX, D10_PWM_NSS, D11_PWM_MOSI, D12_MISO, D13_SCK, D1_TX, DIO_OUT_TO_IN, INT0, INT1
- wire segments 177 -> 140
- no-connect marks 46 -> 9
Other:
- note removed: "Arduino Connector Pins Bus"
- note removed: "MikroBus\nClick\nConnector"
- note removed: "Note\n1. D0_TX transmits from Nucleo to Arduiono pins.\n2. D1_RX recevies form Arduino pins t Nucleo."

Commit message: Fixed the schematic DRC errors.
Parts:
- gave numbers to parts that had none: 2
Other:
- note added: "~DIO_NSS~ to DIOS_SS Inverter"
- moved on the sheet: R68
Changed lines of the file:
@@
 	2250 6900 2150 7000
 Wire Bus Line
-	4850 7900 4850 6700
-Wire Bus Line
-	2150 7900 4850 7900
+	4900 7900 4900 6600
+Wire Bus Line
+	2150 7900 4900 7900
 Text Label 2250 6800 0    50   ~ 0
 DIO_SCK
@@
 Text Notes 2900 7850 0    50   ~ 0
 Digitial I/O Bus
-Text Notes 5350 6800 0    50   ~ 0
+Text Notes 5400 6700 0    50   ~ 0
 Digitial I/O Bus
 Text Notes 8050 1950 0    50   ~ 0
@@
 Text Label 3900 1400 0    50   ~ 0
 3.3V
-Text Label 5800 1400 0    50   ~ 0
+Text Label 3600 1400 0    50   ~ 0
 GND
 $Comp
@@
 	4100 1900 4100 2000
 Entry Wire Line
-	5800 1350 5700 1250
+	3600 1400 3500 1300
 $Comp
 L Device:C C?
@@
 	4700 2000 5300 2000
 Wire Wire Line
-	3900 1500 3900 1350
-Wire Wire Line
-	5300 2000 5800 2000
-Wire Wire Line
-	5800 2000 5800 1350
-Connection ~ 5300 2000
+	3900 1500 3900 1400
+Wire Wire Line
+	4100 2000 3600 2000
+Wire Wire Line
+	3600 2000 3600 1400
 Text Notes 4400 1450 0    50   ~ 0
 ByPass Capacitors
@@
 Note: The 8 extra input pins on U& that are currently unused.
 Entry Wire Line
-	3900 1350 3800 1250
+	3900 1400 3800 1300
 $Comp
 L HR2:SENSE;M1x3 CN4
@@
 	7500 2800 8900 2800
 Wire Bus Line
-	4850 6700 8000 6700
+	4900 6600 8000 6600
 Connection ~ 6000 6400
 Wire Bus Line
-	6000 1250 10400 1250
-Connection ~ 6000 1250
+	6000 1300 10400 1300
+Connection ~ 6000 1300
 Wire Wire Line
 	7300 3000 7400 3000
@@
 L Transistor_FET:2N7000 Q?
 U 1 1 5FDEB033
-P 3250 4500
+P 3200 4400
 AR Path="/5F79BC00/5FDEB033" Ref="Q?"  Part="1"
 AR Path="/5FA4A874/5FDEB033" Ref="Q?"  Part="1"
@@
 AR Path="/5F8C2F57/5FDEB033" Ref="Q?"  Part="1"
 AR Path="/5F3221A2/5FDEB033" Ref="Q?"  Part="1"
-AR Path="/5F4CEE66/5FDEB033" Ref="Q?"  Part="1"
-F 0 "Q?" H 3150 4650 50  0000 L CNN
-F 1 "2N7000;SOT23" H 3400 4350 50  0000 L CNN
-F 2 "Package_TO_SOT_SMD:SOT-23" H 3450 4425 50  0001 L CIN
-F 3 "https://www.fairchildsemi.com/datasheets/2N/2N7000.pdf" H 3250 4500 50  0001 L CNN
-	1    3250 4500
-	1    0    0    -1
-$EndComp
-Wire Wire Line
-	2700 4500 3050 4500
+AR Path="/5F4CEE66/5FDEB033" Ref="Q25"  Part="1"
+F 0 "Q25" H 3050 4550 50  0000 L CNN
+F 1 "2N7000;SOT23" H 3350 4250 50  0000 L CNN
+F 2 "Package_TO_SOT_SMD:SOT-23" H 3400 4325 50  0001 L CIN
+F 3 "https://www.fairchildsemi.com/datasheets/2N/2N7000.pdf" H 3200 4400 50  0001 L CNN
+	1    3200 4400
+	1    0    0    -1
+$EndComp
 $Comp
 L Device:R_US R?
 U 1 1 5FDEB03A
-P 3350 3950
+P 3300 3850
 AR Path="/5F52F39E/5FDEB03A" Ref="R?"  Part="1"
 AR Path="/5F3221A2/5FDEB03A" Ref="R?"  Part="1"
-AR Path="/5F4CEE66/5FDEB03A" Ref="R?"  Part="1"
-F 0 "R?" H 3200 4050 50  0000 L CNN
-F 1 "100KΩ;1608" H 3400 3850 50  0000 L CNN
-F 2 "Resistor_SMD:R_0603_1608Metric" V 3390 3940 50  0001 C CNN
-F 3 "~" H 3350 3950 50  0001 C CNN
-	1    3350 3950
-	1    0    0    -1
-$EndComp
-Wire Wire Line
-	3350 4300 3350 4200
-Wire Wire Line
-	3350 4700 3350 5100
-Text HLabel 3100 3700 0    50   Input ~ 0
-3.3V
-Wire Wire Line
-	3100 3700 3350 3700
-Wire Wire Line
-	3350 3700 3350 3800
-Text HLabel 3600 4200 2    50   Output ~ 0
+AR Path="/5F4CEE66/5FDEB03A" Ref="R68"  Part="1"
+F 0 "R68" H 3150 3950 50  0000 L CNN
+F 1 "100KΩ;1608" H 3350 3750 50  0000 L CNN
+F 2 "Resistor_SMD:R_0603_1608Metric" V 3340 3840 50  0001 C CNN
+F 3 "~" H 3300 3850 50  0001 C CNN
+	1    3300 3850
+	1    0    0    -1
+$EndComp
+Wire Wire Line
+	3300 4200 3300 4100
+Wire Wire Line
+	3300 4600 3300 4700
+Wire Wire Line
+	2800 3600 3300 3600
+Wire Wire Line
+	3300 3600 3300 3700
+Connection ~ 3300 4100
+Wire Wire Line
+	3300 4100 3300 4000
+Wire Wire Line
+	3300 4700 2800 4700
+Entry Wire Line
+	2150 4500 2250 4400
+Text Label 2250 4400 0    50   ~ 0
+~DIO_NSS
+Entry Wire Line
+	2800 3600 2700 3500
+Text Label 2800 3600 0    50   ~ 0
+3.3V
+Wire Wire Line
+	2250 4400 3000 4400
+Entry Wire Line
+	2800 4700 2700 4600
+Text Label 2800 4700 0    50   ~ 0
+GND
+Wire Bus Line
+	2400 1300 2700 1300
+Connection ~ 2700 1300
+Wire Wire Line
+	3300 4100 2250 4100
+Text Label 2250 4100 0    50   ~ 0
 DIO_SS
-Wire Wire Line
-	3600 4200 3350 4200
-Connection ~ 3350 4200
-Wire Wire Line
-	3350 4200 3350 4100
-Text HLabel 3100 5100 0    50   Input ~ 0
-GND
-Wire Wire Line
-	3350 5100 3100 5100
-Text HLabel 2700 4500 0    50   Input ~ 0
-~DIO_NSS
-Wire Bus Line
-	2400 1250 6000 1250
+Entry Wire Line
+	2250 4100 2150 4200
+Text Notes 2800 3450 0    50   ~ 0
+~DIO_NSS~ to DIOS_SS Inverter
+Connection ~ 4100 2000
+Wire Bus Line
+	2700 1300 6000 1300
+Wire Bus Line
+	2700 1300 2700 4750
 Wire Bus Line
 	4700 6400 4700 7700
 Wire Bus Line
-	2400 800  2400 1250
-Wire Bus Line
-	10400 1250 10400 6400
-Wire Bus Line
-	8000 1700 8000 6700
-Wire Bus Line
-	2150 6800 2150 7900
-Wire Bus Line
-	6000 1250 6000 6400
+	2400 800  2400 1300
+Wire Bus Line
+	10400 1300 10400 6400
+Wire Bus Line
+	8000 1700 8000 6600
+Wire Bus Line
+	2150 4000 2150 7900
+Wire Bus Line
+	6000 1300 6000 6400
 $EndSCHEMATC

Commit message: Changed bypass caps and sonar echo outputs
Made following changes:
 - Changed bypass caps to 0.1uF
 - Removed voltage dividers on sonar echo outputs to Nucleo
Parts:
- C14, C15, C16: value 10pF;1608 -> 0.1µF;1608
Changed lines of the file:
@@
 AR Path="/5F4CEE66/5F97D822" Ref="C14"  Part="1"
 F 0 "C14" H 3900 1850 50  0000 L CNN
-F 1 "10pF;1608" H 4150 1650 50  0000 L CNN
+F 1 "0.1µF;1608" H 4150 1650 50  0000 L CNN
 F 2 "Capacitor_SMD:C_0603_1608Metric" H 4138 1600 50  0001 C CNN
 F 3 "~" H 4100 1750 50  0001 C CNN
@@
 AR Path="/5F4CEE66/5F97D82E" Ref="C15"  Part="1"
 F 0 "C15" H 4500 1850 50  0000 L CNN
-F 1 "10pF;1608" H 4750 1650 50  0000 L CNN
+F 1 "0.1µF;1608" H 4750 1650 50  0000 L CNN
 F 2 "Capacitor_SMD:C_0603_1608Metric" H 4738 1600 50  0001 C CNN
 F 3 "~" H 4700 1750 50  0001 C CNN
@@
 AR Path="/5F4CEE66/5F97D834" Ref="C16"  Part="1"
 F 0 "C16" H 5100 1850 50  0000 L CNN
-F 1 "10pF;1608" H 5350 1650 50  0000 L CNN
+F 1 "0.1µF;1608" H 5350 1650 50  0000 L CNN
 F 2 "Capacitor_SMD:C_0603_1608Metric" H 5338 1600 50  0001 C CNN
 F 3 "~" H 5300 1750 50  0001 C CNN

Commit message: Changed bypass caps size from 1608 to 1005
Parts:
- C14, C15, C16: value 0.1µF;1608 -> 0.1µF;1005; footprint Capacitor_SMD:C_0603_1608Metric -> Capacitor_SMD:C_0402_1005Metric
Changed lines of the file:
@@
 AR Path="/5F4CEE66/5F97D822" Ref="C14"  Part="1"
 F 0 "C14" H 3900 1850 50  0000 L CNN
-F 1 "0.1µF;1608" H 4150 1650 50  0000 L CNN
-F 2 "Capacitor_SMD:C_0603_1608Metric" H 4138 1600 50  0001 C CNN
+F 1 "0.1µF;1005" H 4150 1650 50  0000 L CNN
+F 2 "Capacitor_SMD:C_0402_1005Metric" H 4138 1600 50  0001 C CNN
 F 3 "~" H 4100 1750 50  0001 C CNN
 	1    4100 1750
@@
 AR Path="/5F4CEE66/5F97D82E" Ref="C15"  Part="1"
 F 0 "C15" H 4500 1850 50  0000 L CNN
-F 1 "0.1µF;1608" H 4750 1650 50  0000 L CNN
-F 2 "Capacitor_SMD:C_0603_1608Metric" H 4738 1600 50  0001 C CNN
+F 1 "0.1µF;1005" H 4750 1650 50  0000 L CNN
+F 2 "Capacitor_SMD:C_0402_1005Metric" H 4738 1600 50  0001 C CNN
 F 3 "~" H 4700 1750 50  0001 C CNN
 	1    4700 1750
@@
 AR Path="/5F4CEE66/5F97D834" Ref="C16"  Part="1"
 F 0 "C16" H 5100 1850 50  0000 L CNN
-F 1 "0.1µF;1608" H 5350 1650 50  0000 L CNN
-F 2 "Capacitor_SMD:C_0603_1608Metric" H 5338 1600 50  0001 C CNN
+F 1 "0.1µF;1005" H 5350 1650 50  0000 L CNN
+F 2 "Capacitor_SMD:C_0402_1005Metric" H 5338 1600 50  0001 C CNN
 F 3 "~" H 5300 1750 50  0001 C CNN
 	1    5300 1750

Commit message: Changed more parts to 1005 size and R9 value
Parts:
- R68: value 100KΩ;1608 -> 100KΩ;1005; footprint Resistor_SMD:R_0603_1608Metric -> Resistor_SMD:R_0402_1005Metric
- U5: value SN74HCS595;TTSOP16 -> SN74HC595;TTSOP16
- U6, U7: value SN74HCS165;TTSOP16 -> SN74HC165;TTSOP16
Changed lines of the file:
@@
 P 2800 6400
 F 0 "U5" H 3050 6550 50  0000 C CNN
-F 1 "SN74HCS595;TTSOP16" H 3300 5250 50  0000 C CNN
+F 1 "SN74HC595;TTSOP16" H 3300 5250 50  0000 C CNN
 F 2 "Package_SO:TSSOP-16_4.4x5mm_P0.65mm" H 3000 6450 60  0001 L CNN
 F 3 "Tri-state 8-Bit Shift Register" H 3000 6250 60  0001 L CNN
@@
 P 8900 4700
 F 0 "U7" H 9150 4850 50  0000 C CNN
-F 1 "SN74HCS165;TTSOP16" H 9400 3450 50  0000 C CNN
+F 1 "SN74HC165;TTSOP16" H 9400 3450 50  0000 C CNN
 F 2 "Package_SO:TSSOP-16_4.4x5mm_P0.65mm" H 9100 4750 60  0001 L CNN
 F 3 "8-Bit Parallel In Serial Out Shift Register" H 9100 4550 60  0001 L CNN
@@
 P 8900 2500
 F 0 "U6" H 9150 2650 50  0000 C CNN
-F 1 "SN74HCS165;TTSOP16" H 9400 1250 50  0000 C CNN
+F 1 "SN74HC165;TTSOP16" H 9400 1250 50  0000 C CNN
 F 2 "Package_SO:TSSOP-16_4.4x5mm_P0.65mm" H 9100 2550 60  0001 L CNN
 F 3 "8-Bit Parallel In Serial Out Shift Register" H 9100 2350 60  0001 L CNN
@@
 AR Path="/5F4CEE66/5FDEB03A" Ref="R68"  Part="1"
 F 0 "R68" H 3150 3950 50  0000 L CNN
-F 1 "100KΩ;1608" H 3350 3750 50  0000 L CNN
-F 2 "Resistor_SMD:R_0603_1608Metric" V 3340 3840 50  0001 C CNN
+F 1 "100KΩ;1005" H 3350 3750 50  0000 L CNN
+F 2 "Resistor_SMD:R_0402_1005Metric" V 3340 3840 50  0001 C CNN
 F 3 "~" H 3300 3850 50  0001 C CNN
 	1    3300 3850
