File: electrical/master_board/rev_a/leds.sch (KiCad schematic (older format))
At the start: 52 parts, among them Q10 2N7000;SOT23, Q11 2N7000;SOT23, Q12 2N7000;SOT23, Q13 2N7000;SOT23, Q14 2N7000;SOT23, Q15 2N7000;SOT23, Q16 2N7000;SOT23, Q17 2N7000;SOT23, Q18 2N7000;SOT23, Q19 2N7000;SOT23, Q4 2N7000;SOT23, Q5 2N7000;SOT23, Q6 2N7000;SOT23, Q7 2N7000;SOT23, Q8 2N7000;SOT23, Q9 2N7000;SOT23, U11 SN74HCS595;TTSOP16, U12 SN74HCS595;TTSOP16

Commit message: Fixed SPI shift registers (good find by James Nugen\!)
Connections:
- net labels added: LED8_SER
- no-connect marks 4 -> 3
Changed lines of the file:
@@
 	1    0    0    -1
 $EndComp
-Wire Wire Line
-	3000 5900 3100 5900
 Entry Wire Line
 	3400 2200 3500 2100
@@
 Text Label 3400 6400 2    50   ~ 0
 GND
-NoConn ~ 3000 6000
 Text Label 1000 5400 0    50   ~ 0
 LED_MOSI
@@
 NoConn ~ 3000 3100
 Wire Wire Line
-	3100 5900 3100 3700
-Wire Wire Line
 	3100 3700 1400 3700
 Wire Wire Line
@@
 Wire Wire Line
 	1400 2500 1900 2500
-Connection ~ 3100 5900
-Wire Wire Line
-	3100 5900 4100 5900
 Text Label 2100 3700 0    50   ~ 0
-LED8
+LED8_SER
 Text Label 3400 2500 2    50   ~ 0
 LED11
@@
 NoConn ~ 3050 -850
 NoConn ~ 11600 -650
+Wire Wire Line
+	3000 6000 3100 6000
 Wire Bus Line
 	3500 1300 3500 7200
+Wire Wire Line
+	3000 5900 4100 5900
+Wire Wire Line
+	3100 3700 3100 6000
 $EndSCHEMATC

Commit message: Changed bypass caps and sonar echo outputs
Made following changes:
 - Changed bypass caps to 0.1uF
 - Removed voltage dividers on sonar echo outputs to Nucleo
Parts:
- C20, C21: value 10pF;1608 -> 0.1µF;1608
Changed lines of the file:
@@
 $Descr A4 11693 8268
 encoding utf-8
-Sheet 7 10
+Sheet 6 10
 Title "HR2 LED's"
 Date "2020-11-22"
@@
 AR Path="/5FA4A874/5FA78555" Ref="C20"  Part="1"
 F 0 "C20" H 3600 7050 50  0000 L CNN
-F 1 "10pF;1608" H 3850 6850 50  0000 L CNN
+F 1 "0.1µF;1608" H 3850 6850 50  0000 L CNN
 F 2 "Capacitor_SMD:C_0603_1608Metric" H 3838 6800 50  0001 C CNN
 F 3 "~" H 3800 6950 50  0001 C CNN
@@
 AR Path="/5FA4A874/5FA78560" Ref="C21"  Part="1"
 F 0 "C21" H 4200 7050 50  0000 L CNN
-F 1 "10pF;1608" H 4450 6850 50  0000 L CNN
+F 1 "0.1µF;1608" H 4450 6850 50  0000 L CNN
 F 2 "Capacitor_SMD:C_0603_1608Metric" H 4438 6800 50  0001 C CNN
 F 3 "~" H 4400 6950 50  0001 C CNN
@@
 Wire Wire Line
 	3000 6000 3100 6000
+Wire Wire Line
+	3000 5900 4100 5900
+Wire Wire Line
+	3100 3700 3100 6000
 Wire Bus Line
 	3500 1300 3500 7200
-Wire Wire Line
-	3000 5900 4100 5900
-Wire Wire Line
-	3100 3700 3100 6000
 $EndSCHEMATC

Commit message: Changed bypass caps size from 1608 to 1005
Parts:
- C20, C21: value 0.1µF;1608 -> 0.1µF;1005; footprint Capacitor_SMD:C_0603_1608Metric -> Capacitor_SMD:C_0402_1005Metric
Changed lines of the file:
@@
 AR Path="/5FA4A874/5FA78555" Ref="C20"  Part="1"
 F 0 "C20" H 3600 7050 50  0000 L CNN
-F 1 "0.1µF;1608" H 3850 6850 50  0000 L CNN
-F 2 "Capacitor_SMD:C_0603_1608Metric" H 3838 6800 50  0001 C CNN
+F 1 "0.1µF;1005" H 3850 6850 50  0000 L CNN
+F 2 "Capacitor_SMD:C_0402_1005Metric" H 3838 6800 50  0001 C CNN
 F 3 "~" H 3800 6950 50  0001 C CNN
 	1    3800 6950
@@
 AR Path="/5FA4A874/5FA78560" Ref="C21"  Part="1"
 F 0 "C21" H 4200 7050 50  0000 L CNN
-F 1 "0.1µF;1608" H 4450 6850 50  0000 L CNN
-F 2 "Capacitor_SMD:C_0603_1608Metric" H 4438 6800 50  0001 C CNN
+F 1 "0.1µF;1005" H 4450 6850 50  0000 L CNN
+F 2 "Capacitor_SMD:C_0402_1005Metric" H 4438 6800 50  0001 C CNN
 F 3 "~" H 4400 6950 50  0001 C CNN
 	1    4400 6950

Commit message: Changed more parts to 1005 size and R9 value
Parts:
- U11, U12: value SN74HCS595;TTSOP16 -> SN74HC595;TTSOP16
Changed lines of the file:
@@
 AR Path="/5FA4A874/5FB58AAF" Ref="U12"  Part="1"
 F 0 "U12" H 2150 5250 50  0000 C CNN
-F 1 "SN74HCS595;TTSOP16" H 2450 3950 50  0000 C CNN
+F 1 "SN74HC595;TTSOP16" H 2450 3950 50  0000 C CNN
 F 2 "Package_SO:TSSOP-16_4.4x5mm_P0.65mm" H 2100 5150 60  0001 L CNN
 F 3 "Tri-state 8-Bit Shift Register" H 2100 4950 60  0001 L CNN
@@
 AR Path="/5FA4A874/5FB58AA4" Ref="U11"  Part="1"
 F 0 "U11" H 2150 2350 50  0000 C CNN
-F 1 "SN74HCS595;TTSOP16" H 2450 1050 50  0000 C CNN
+F 1 "SN74HC595;TTSOP16" H 2450 1050 50  0000 C CNN
 F 2 "Package_SO:TSSOP-16_4.4x5mm_P0.65mm" H 2100 2250 60  0001 L CNN
 F 3 "Tri-state 8-Bit Shift Register" H 2100 2050 60  0001 L CNN

Commit message: JLCPCB BOM is in better shape.
Parts:
- removed Q10, Q11, Q12, Q13, Q14, Q15, Q16, Q17, Q18, Q19, Q4, Q5, Q6, Q7, Q8, Q9: 2N7000;SOT23, Package_TO_SOT_SMD:SOT-23, symbol Transistor_FET:2N7000
- added Q10, Q11, Q12, Q13, Q14, Q15, Q16, Q17, Q18, Q19, Q4, Q5, Q6, Q7, Q8, Q9: 2N7002;SOT23, Package_TO_SOT_SMD:SOT-23, symbol Transistor_FET:2N7002

Commit message: Made various changes from to_do.md
Parts:
- R37, R38, R39, R40, R42, R43, R44, R46, R47, R48, R49, R50, R51, R52: value 470Ω.25W;1608 -> 270Ω;1005; footprint Resistor_SMD:R_0603_1608Metric -> Resistor_SMD:R_0402_1005Metric
- R41, R45: value 470Ω.25W;1608 -> 270Ω.;1005; footprint Resistor_SMD:R_0603_1608Metric -> Resistor_SMD:R_0402_1005Metric
Changed lines of the file:
@@
 AR Path="/5FA4A874/5FAB2D76" Ref="R52"  Part="1"
 F 0 "R52" H 9950 4600 50  0000 L CNN
-F 1 "470Ω.25W;1608" H 10100 4350 50  0000 L CNN
-F 2 "Resistor_SMD:R_0603_1608Metric" V 10140 4440 50  0001 C CNN
+F 1 "270Ω;1005" H 10100 4350 50  0000 L CNN
+F 2 "Resistor_SMD:R_0402_1005Metric" V 10140 4440 50  0001 C CNN
 F 3 "~" H 10100 4450 50  0001 C CNN
 	1    10100 4450
@@
 AR Path="/5FA4A874/5FAB2D55" Ref="R50"  Part="1"
 F 0 "R50" H 9150 4600 50  0000 L CNN
-F 1 "470Ω.25W;1608" H 9300 4350 50  0000 L CNN
-F 2 "Resistor_SMD:R_0603_1608Metric" V 9340 4440 50  0001 C CNN
+F 1 "270Ω;1005" H 9300 4350 50  0000 L CNN
+F 2 "Resistor_SMD:R_0402_1005Metric" V 9340 4440 50  0001 C CNN
 F 3 "~" H 9300 4450 50  0001 C CNN
 	1    9300 4450
@@
 AR Path="/5FA4A874/5FAB2D34" Ref="R48"  Part="1"
 F 0 "R48" H 8350 4600 50  0000 L CNN
-F 1 "470Ω.25W;1608" H 8500 4350 50  0000 L CNN
-F 2 "Resistor_SMD:R_0603_1608Metric" V 8540 4440 50  0001 C CNN
+F 1 "270Ω;1005" H 8500 4350 50  0000 L CNN
+F 2 "Resistor_SMD:R_0402_1005Metric" V 8540 4440 50  0001 C CNN
 F 3 "~" H 8500 4450 50  0001 C CNN
 	1    8500 4450
@@
 AR Path="/5FA4A874/5FAB2D13" Ref="R46"  Part="1"
 F 0 "R46" H 7550 4600 50  0000 L CNN
-F 1 "470Ω.25W;1608" H 7700 4350 50  0000 L CNN
-F 2 "Resistor_SMD:R_0603_1608Metric" V 7740 4440 50  0001 C CNN
+F 1 "270Ω;1005" H 7700 4350 50  0000 L CNN
+F 2 "Resistor_SMD:R_0402_1005Metric" V 7740 4440 50  0001 C CNN
 F 3 "~" H 7700 4450 50  0001 C CNN
 	1    7700 4450
@@
 AR Path="/5FA4A874/5FA9CF6C" Ref="R44"  Part="1"
 F 0 "R44" H 6750 4600 50  0000 L CNN
-F 1 "470Ω.25W;1608" H 6900 4350 50  0000 L CNN
-F 2 "Resistor_SMD:R_0603_1608Metric" V 6940 4440 50  0001 C CNN
+F 1 "270Ω;1005" H 6900 4350 50  0000 L CNN
+F 2 "Resistor_SMD:R_0402_1005Metric" V 6940 4440 50  0001 C CNN
 F 3 "~" H 6900 4450 50  0001 C CNN
 	1    6900 4450
@@
 AR Path="/5FA4A874/5FA9CF4A" Ref="R42"  Part="1"
 F 0 "R42" H 5950 4600 50  0000 L CNN
-F 1 "470Ω.25W;1608" H 6100 4350 50  0000 L CNN
-F 2 "Resistor_SMD:R_0603_1608Metric" V 6140 4440 50  0001 C CNN
+F 1 "270Ω;1005" H 6100 4350 50  0000 L CNN
+F 2 "Resistor_SMD:R_0402_1005Metric" V 6140 4440 50  0001 C CNN
 F 3 "~" H 6100 4450 50  0001 C CNN
 	1    6100 4450
@@
 AR Path="/5FA4A874/5FA992FD" Ref="R40"  Part="1"
 F 0 "R40" H 5150 4600 50  0000 L CNN
-F 1 "470Ω.25W;1608" H 5300 4350 50  0000 L CNN
-F 2 "Resistor_SMD:R_0603_1608Metric" V 5340 4440 50  0001 C CNN
+F 1 "270Ω;1005" H 5300 4350 50  0000 L CNN
+F 2 "Resistor_SMD:R_0402_1005Metric" V 5340 4440 50  0001 C CNN
 F 3 "~" H 5300 4450 50  0001 C CNN
 	1    5300 4450
@@
 AR Path="/5FA4A874/5FA5B814" Ref="R38"  Part="1"
 F 0 "R38" H 4350 4600 50  0000 L CNN
-F 1 "470Ω.25W;1608" H 4500 4350 50  0000 L CNN
-F 2 "Resistor_SMD:R_0603_1608Metric" V 4540 4440 50  0001 C CNN
+F 1 "270Ω;1005" H 4500 4350 50  0000 L CNN
+F 2 "Resistor_SMD:R_0402_1005Metric" V 4540 4440 50  0001 C CNN
 F 3 "~" H 4500 4450 50  0001 C CNN
 	1    4500 4450
@@
 AR Path="/5FA4A874/5FB18978" Ref="R51"  Part="1"
 F 0 "R51" H 9950 1700 50  0000 L CNN
-F 1 "470Ω.25W;1608" H 10100 1450 50  0000 L CNN
-F 2 "Resistor_SMD:R_0603_1608Metric" V 10140 1540 50  0001 C CNN
+F 1 "270Ω;1005" H 10100 1450 50  0000 L CNN
+F 2 "Resistor_SMD:R_0402_1005Metric" V 10140 1540 50  0001 C CNN
 F 3 "~" H 10100 1550 50  0001 C CNN
 	1    10100 1550
@@
 AR Path="/5FA4A874/5FB18999" Ref="R49"  Part="1"
 F 0 "R49" H 9150 1700 50  0000 L CNN
-F 1 "470Ω.25W;1608" H 9300 1450 50  0000 L CNN
-F 2 "Resistor_SMD:R_0603_1608Metric" V 9340 1540 50  0001 C CNN
+F 1 "270Ω;1005" H 9300 1450 50  0000 L CNN
+F 2 "Resistor_SMD:R_0402_1005Metric" V 9340 1540 50  0001 C CNN
 F 3 "~" H 9300 1550 50  0001 C CNN
 	1    9300 1550
@@
 AR Path="/5FA4A874/5FB189BA" Ref="R47"  Part="1"
 F 0 "R47" H 8350 1700 50  0000 L CNN
-F 1 "470Ω.25W;1608" H 8500 1450 50  0000 L CNN
-F 2 "Resistor_SMD:R_0603_1608Metric" V 8540 1540 50  0001 C CNN
+F 1 "270Ω;1005" H 8500 1450 50  0000 L CNN
+F 2 "Resistor_SMD:R_0402_1005Metric" V 8540 1540 50  0001 C CNN
 F 3 "~" H 8500 1550 50  0001 C CNN
 	1    8500 1550
@@
 AR Path="/5FA4A874/5FB189DB" Ref="R45"  Part="1"
 F 0 "R45" H 7550 1700 50  0000 L CNN
-F 1 "470Ω.25W;1608" H 7700 1450 50  0000 L CNN
-F 2 "Resistor_SMD:R_0603_1608Metric" V 7740 1540 50  0001 C CNN
+F 1 "270Ω.;1005" H 7700 1450 50  0000 L CNN
+F 2 "Resistor_SMD:R_0402_1005Metric" V 7740 1540 50  0001 C CNN
 F 3 "~" H 7700 1550 50  0001 C CNN
 	1    7700 1550
@@
 AR Path="/5FA4A874/5FB189FC" Ref="R43"  Part="1"
 F 0 "R43" H 6750 1700 50  0000 L CNN
-F 1 "470Ω.25W;1608" H 6900 1450 50  0000 L CNN
-F 2 "Resistor_SMD:R_0603_1608Metric" V 6940 1540 50  0001 C CNN
+F 1 "270Ω;1005" H 6900 1450 50  0000 L CNN
+F 2 "Resistor_SMD:R_0402_1005Metric" V 6940 1540 50  0001 C CNN
 F 3 "~" H 6900 1550 50  0001 C CNN
 	1    6900 1550
@@
 AR Path="/5FA4A874/5FB18A1E" Ref="R41"  Part="1"
 F 0 "R41" H 5950 1700 50  0000 L CNN
-F 1 "470Ω.25W;1608" H 6100 1450 50  0000 L CNN
-F 2 "Resistor_SMD:R_0603_1608Metric" V 6140 1540 50  0001 C CNN
+F 1 "270Ω.;1005" H 6100 1450 50  0000 L CNN
+F 2 "Resistor_SMD:R_0402_1005Metric" V 6140 1540 50  0001 C CNN
 F 3 "~" H 6100 1550 50  0001 C CNN
 	1    6100 1550
@@
 AR Path="/5FA4A874/5FB18A40" Ref="R39"  Part="1"
 F 0 "R39" H 5150 1700 50  0000 L CNN
-F 1 "470Ω.25W;1608" H 5300 1450 50  0000 L CNN
-F 2 "Resistor_SMD:R_0603_1608Metric" V 5340 1540 50  0001 C CNN
+F 1 "270Ω;1005" H 5300 1450 50  0000 L CNN
+F 2 "Resistor_SMD:R_0402_1005Metric" V 5340 1540 50  0001 C CNN
 F 3 "~" H 5300 1550 50  0001 C CNN
 	1    5300 1550
@@
 AR Path="/5FA4A874/5FB18A62" Ref="R37"  Part="1"
 F 0 "R37" H 4350 1700 50  0000 L CNN
-F 1 "470Ω.25W;1608" H 4500 1450 50  0000 L CNN
-F 2 "Resistor_SMD:R_0603_1608Metric" V 4540 1540 50  0001 C CNN
+F 1 "270Ω;1005" H 4500 1450 50  0000 L CNN
+F 2 "Resistor_SMD:R_0402_1005Metric" V 4540 1540 50  0001 C CNN
 F 3 "~" H 4500 1550 50  0001 C CNN
 	1    4500 1550
@@
 	1    0    0    -1
 $EndComp
-Wire Bus Line
-	3500 1300 3500 7200
 $Comp
 L Transistor_FET:2N7002 Q6
@@
 	1    0    0    -1
 $EndComp
+Wire Bus Line
+	3500 1300 3500 7200
 $EndSCHEMATC

Commit message: JLCPCB Footprints are both consistent and available.
Parts:
- removed U11, U12: SN74HC595;TTSOP16, Package_SO:TSSOP-16_4.4x5mm_P0.65mm, symbol HR2:SN74HCS595;TTSOP16
- added U11, U12: SN74HC595;HTSSOP16EP3.4x5, Package_SO:HTSSOP-16-1EP_4.4x5mm_P0.65mm_EP3.4x5mm, symbol HR2:SN74HC595;HTSSOP16EP3.4x5
- R37, R38, R39, R40, R42, R43, R44, R46, R47, R48, R49, R50, R51, R52: value 270Ω;1005 -> 270Ω;1608; footprint Resistor_SMD:R_0402_1005Metric -> Resistor_SMD:R_0603_1608Metric
- R41, R45: value 270Ω.;1005 -> 270Ω;1608; footprint Resistor_SMD:R_0402_1005Metric -> Resistor_SMD:R_0603_1608Metric
Changed lines of the file:
@@
 AR Path="/5FA4A874/5FAB2D76" Ref="R52"  Part="1"
 F 0 "R52" H 9950 4600 50  0000 L CNN
-F 1 "270Ω;1005" H 10100 4350 50  0000 L CNN
-F 2 "Resistor_SMD:R_0402_1005Metric" V 10140 4440 50  0001 C CNN
+F 1 "270Ω;1608" H 10100 4350 50  0000 L CNN
+F 2 "Resistor_SMD:R_0603_1608Metric" V 10140 4440 50  0001 C CNN
 F 3 "~" H 10100 4450 50  0001 C CNN
 	1    10100 4450
@@
 AR Path="/5FA4A874/5FAB2D55" Ref="R50"  Part="1"
 F 0 "R50" H 9150 4600 50  0000 L CNN
-F 1 "270Ω;1005" H 9300 4350 50  0000 L CNN
-F 2 "Resistor_SMD:R_0402_1005Metric" V 9340 4440 50  0001 C CNN
+F 1 "270Ω;1608" H 9300 4350 50  0000 L CNN
+F 2 "Resistor_SMD:R_0603_1608Metric" V 9340 4440 50  0001 C CNN
 F 3 "~" H 9300 4450 50  0001 C CNN
 	1    9300 4450
@@
 AR Path="/5FA4A874/5FAB2D34" Ref="R48"  Part="1"
 F 0 "R48" H 8350 4600 50  0000 L CNN
-F 1 "270Ω;1005" H 8500 4350 50  0000 L CNN
-F 2 "Resistor_SMD:R_0402_1005Metric" V 8540 4440 50  0001 C CNN
+F 1 "270Ω;1608" H 8500 4350 50  0000 L CNN
+F 2 "Resistor_SMD:R_0603_1608Metric" V 8540 4440 50  0001 C CNN
 F 3 "~" H 8500 4450 50  0001 C CNN
 	1    8500 4450
@@
 AR Path="/5FA4A874/5FAB2D13" Ref="R46"  Part="1"
 F 0 "R46" H 7550 4600 50  0000 L CNN
-F 1 "270Ω;1005" H 7700 4350 50  0000 L CNN
-F 2 "Resistor_SMD:R_0402_1005Metric" V 7740 4440 50  0001 C CNN
+F 1 "270Ω;1608" H 7700 4350 50  0000 L CNN
+F 2 "Resistor_SMD:R_0603_1608Metric" V 7740 4440 50  0001 C CNN
 F 3 "~" H 7700 4450 50  0001 C CNN
 	1    7700 4450
@@
 AR Path="/5FA4A874/5FA9CF6C" Ref="R44"  Part="1"
 F 0 "R44" H 6750 4600 50  0000 L CNN
-F 1 "270Ω;1005" H 6900 4350 50  0000 L CNN
-F 2 "Resistor_SMD:R_0402_1005Metric" V 6940 4440 50  0001 C CNN
+F 1 "270Ω;1608" H 6900 4350 50  0000 L CNN
+F 2 "Resistor_SMD:R_0603_1608Metric" V 6940 4440 50  0001 C CNN
 F 3 "~" H 6900 4450 50  0001 C CNN
 	1    6900 4450
@@
 AR Path="/5FA4A874/5FA9CF4A" Ref="R42"  Part="1"
 F 0 "R42" H 5950 4600 50  0000 L CNN
-F 1 "270Ω;1005" H 6100 4350 50  0000 L CNN
-F 2 "Resistor_SMD:R_0402_1005Metric" V 6140 4440 50  0001 C CNN
+F 1 "270Ω;1608" H 6100 4350 50  0000 L CNN
+F 2 "Resistor_SMD:R_0603_1608Metric" V 6140 4440 50  0001 C CNN
 F 3 "~" H 6100 4450 50  0001 C CNN
 	1    6100 4450
@@
 AR Path="/5FA4A874/5FA992FD" Ref="R40"  Part="1"
 F 0 "R40" H 5150 4600 50  0000 L CNN
-F 1 "270Ω;1005" H 5300 4350 50  0000 L CNN
-F 2 "Resistor_SMD:R_0402_1005Metric" V 5340 4440 50  0001 C CNN
+F 1 "270Ω;1608" H 5300 4350 50  0000 L CNN
+F 2 "Resistor_SMD:R_0603_1608Metric" V 5340 4440 50  0001 C CNN
 F 3 "~" H 5300 4450 50  0001 C CNN
 	1    5300 4450
@@
 AR Path="/5FA4A874/5FA5B814" Ref="R38"  Part="1"
 F 0 "R38" H 4350 4600 50  0000 L CNN
-F 1 "270Ω;1005" H 4500 4350 50  0000 L CNN
-F 2 "Resistor_SMD:R_0402_1005Metric" V 4540 4440 50  0001 C CNN
+F 1 "270Ω;1608" H 4500 4350 50  0000 L CNN
+F 2 "Resistor_SMD:R_0603_1608Metric" V 4540 4440 50  0001 C CNN
 F 3 "~" H 4500 4450 50  0001 C CNN
 	1    4500 4450
@@
 AR Path="/5FA4A874/5FB18978" Ref="R51"  Part="1"
 F 0 "R51" H 9950 1700 50  0000 L CNN
-F 1 "270Ω;1005" H 10100 1450 50  0000 L CNN
-F 2 "Resistor_SMD:R_0402_1005Metric" V 10140 1540 50  0001 C CNN
+F 1 "270Ω;1608" H 10100 1450 50  0000 L CNN
+F 2 "Resistor_SMD:R_0603_1608Metric" V 10140 1540 50  0001 C CNN
 F 3 "~" H 10100 1550 50  0001 C CNN
 	1    10100 1550
@@
 AR Path="/5FA4A874/5FB18999" Ref="R49"  Part="1"
 F 0 "R49" H 9150 1700 50  0000 L CNN
-F 1 "270Ω;1005" H 9300 1450 50  0000 L CNN
-F 2 "Resistor_SMD:R_0402_1005Metric" V 9340 1540 50  0001 C CNN
+F 1 "270Ω;1608" H 9300 1450 50  0000 L CNN
+F 2 "Resistor_SMD:R_0603_1608Metric" V 9340 1540 50  0001 C CNN
 F 3 "~" H 9300 1550 50  0001 C CNN
 	1    9300 1550
@@
 AR Path="/5FA4A874/5FB189BA" Ref="R47"  Part="1"
 F 0 "R47" H 8350 1700 50  0000 L CNN
-F 1 "270Ω;1005" H 8500 1450 50  0000 L CNN
-F 2 "Resistor_SMD:R_0402_1005Metric" V 8540 1540 50  0001 C CNN
+F 1 "270Ω;1608" H 8500 1450 50  0000 L CNN
+F 2 "Resistor_SMD:R_0603_1608Metric" V 8540 1540 50  0001 C CNN
 F 3 "~" H 8500 1550 50  0001 C CNN
 	1    8500 1550
@@
 AR Path="/5FA4A874/5FB189DB" Ref="R45"  Part="1"
 F 0 "R45" H 7550 1700 50  0000 L CNN
-F 1 "270Ω.;1005" H 7700 1450 50  0000 L CNN
-F 2 "Resistor_SMD:R_0402_1005Metric" V 7740 1540 50  0001 C CNN
+F 1 "270Ω;1608" H 7700 1450 50  0000 L CNN
+F 2 "Resistor_SMD:R_0603_1608Metric" V 7740 1540 50  0001 C CNN
 F 3 "~" H 7700 1550 50  0001 C CNN
 	1    7700 1550
@@
 AR Path="/5FA4A874/5FB189FC" Ref="R43"  Part="1"
 F 0 "R43" H 6750 1700 50  0000 L CNN
-F 1 "270Ω;1005" H 6900 1450 50  0000 L CNN
-F 2 "Resistor_SMD:R_0402_1005Metric" V 6940 1540 50  0001 C CNN
+F 1 "270Ω;1608" H 6900 1450 50  0000 L CNN
+F 2 "Resistor_SMD:R_0603_1608Metric" V 6940 1540 50  0001 C CNN
 F 3 "~" H 6900 1550 50  0001 C CNN
 	1    6900 1550
@@
 AR Path="/5FA4A874/5FB18A1E" Ref="R41"  Part="1"
 F 0 "R41" H 5950 1700 50  0000 L CNN
-F 1 "270Ω.;1005" H 6100 1450 50  0000 L CNN
-F 2 "Resistor_SMD:R_0402_1005Metric" V 6140 1540 50  0001 C CNN
+F 1 "270Ω;1608" H 6100 1450 50  0000 L CNN
+F 2 "Resistor_SMD:R_0603_1608Metric" V 6140 1540 50  0001 C CNN
 F 3 "~" H 6100 1550 50  0001 C CNN
 	1    6100 1550
@@
 AR Path="/5FA4A874/5FB18A40" Ref="R39"  Part="1"
 F 0 "R39" H 5150 1700 50  0000 L CNN
-F 1 "270Ω;1005" H 5300 1450 50  0000 L CNN
-F 2 "Resistor_SMD:R_0402_1005Metric" V 5340 1540 50  0001 C CNN
+F 1 "270Ω;1608" H 5300 1450 50  0000 L CNN
+F 2 "Resistor_SMD:R_0603_1608Metric" V 5340 1540 50  0001 C CNN
 F 3 "~" H 5300 1550 50  0001 C CNN
 	1    5300 1550
@@
 AR Path="/5FA4A874/5FB18A62" Ref="R37"  Part="1"
 F 0 "R37" H 4350 1700 50  0000 L CNN
-F 1 "270Ω;1005" H 4500 1450 50  0000 L CNN
-F 2 "Resistor_SMD:R_0402_1005Metric" V 4540 1540 50  0001 C CNN
+F 1 "270Ω;1608" H 4500 1450 50  0000 L CNN
+F 2 "Resistor_SMD:R_0603_1608Metric" V 4540 1540 50  0001 C CNN
 F 3 "~" H 4500 1550 50  0001 C CNN
 	1    4500 1550
@@
 Text HLabel 1000 5500 0    50   Input ~ 0
 LEDS_SCLK
-$Comp
-L HR2:SN74HCS595;TTSOP16 U?
-U 1 1 5FB58AAF
-P 1900 5100
-AR Path="/5F48CAAD/5FB58AAF" Ref="U?"  Part="1"
-AR Path="/5FA4A874/5FB58AAF" Ref="U12"  Part="1"
-F 0 "U12" H 2150 5250 50  0000 C CNN
-F 1 "SN74HC595;TTSOP16" H 2450 3950 50  0000 C CNN
-F 2 "Package_SO:TSSOP-16_4.4x5mm_P0.65mm" H 2100 5150 60  0001 L CNN
-F 3 "Tri-state 8-Bit Shift Register" H 2100 4950 60  0001 L CNN
-F 4 "Tri-State 8-Bit Shift Register" H 2100 4850 60  0001 L CNN "Field5"
-	1    1900 5100
-	1    0    0    -1
-$EndComp
 Text Label 3400 5900 2    50   ~ 0
 LED8
@@
 Wire Wire Line
 	3000 5200 9700 5200
-$Comp
-L HR2:SN74HCS595;TTSOP16 U?
-U 1 1 5FB58AA4
-P 1900 2200
-AR Path="/5F48CAAD/5FB58AA4" Ref="U?"  Part="1"
-AR Path="/5FA4A874/5FB58AA4" Ref="U11"  Part="1"
-F 0 "U11" H 2150 2350 50  0000 C CNN
-F 1 "SN74HC595;TTSOP16" H 2450 1050 50  0000 C CNN
-F 2 "Package_SO:TSSOP-16_4.4x5mm_P0.65mm" H 2100 2250 60  0001 L CNN
-F 3 "Tri-state 8-Bit Shift Register" H 2100 2050 60  0001 L CNN
-F 4 "Tri-State 8-Bit Shift Register" H 2100 1950 60  0001 L CNN "Field5"
-	1    1900 2200
-	1    0    0    -1
-$EndComp
 Entry Wire Line
 	3400 2200 3500 2100
@@
 	1    0    0    -1
 $EndComp
+$Comp
+L HR2:SN74HC595;HTSSOP16EP3.4x5 U?
+U 1 1 5FE3B49B
+P 1900 2200
+AR Path="/5F4CEE66/5FE3B49B" Ref="U?"  Part="1"
+AR Path="/5FA4A874/5FE3B49B" Ref="U11"  Part="1"
+F 0 "U11" H 2150 2350 50  0000 C CNN
+F 1 "SN74HC595;HTSSOP16EP3.4x5" H 2500 1050 50  0000 C CNN
+F 2 "Package_SO:HTSSOP-16-1EP_4.4x5mm_P0.65mm_EP3.4x5mm" H 2100 2250 60  0001 L CNN
+F 3 "Tri-state 8-Bit Shift Register" H 2100 2050 60  0001 L CNN
+F 4 "Tri-State 8-Bit Shift Register" H 2100 1950 60  0001 L CNN "desc"
+	1    1900 2200
+	1    0    0    -1
+$EndComp
 Wire Bus Line
 	3500 1300 3500 7200
+$Comp
+L HR2:SN74HC595;HTSSOP16EP3.4x5 U?
+U 1 1 5FE48EC9
+P 1900 5100
+AR Path="/5F4CEE66/5FE48EC9" Ref="U?"  Part="1"
+AR Path="/5FA4A874/5FE48EC9" Ref="U12"  Part="1"
+F 0 "U12" H 2150 5250 50  0000 C CNN
+F 1 "SN74HC595;HTSSOP16EP3.4x5" H 2500 3950 50  0000 C CNN
+F 2 "Package_SO:HTSSOP-16-1EP_4.4x5mm_P0.65mm_EP3.4x5mm" H 2100 5150 60  0001 L CNN
+F 3 "Tri-state 8-Bit Shift Register" H 2100 4950 60  0001 L CNN
+F 4 "Tri-State 8-Bit Shift Register" H 2100 4850 60  0001 L CNN "desc"
+	1    1900 5100
+	1    0    0    -1
+$EndComp
 $EndSCHEMATC
